File: Hardware/rev1/croptop_rev1/croptop_rev1.sch (KiCad schematic (older format))
At the start: 93 parts

Commit message: November 1st edit1
Parts:
- removed C?: 10uF, symbol Device:CP1
- removed C? (x7): 0.1uF, symbol Device:C
- removed C?: 100uF, symbol Device:C
- removed D? (x2): D_Zener, symbol Device:D_Zener
- removed J?: RPI I2C Header, symbol Connector:Conn_01x02_Male
- removed Q? (x2): BS250, Package_TO_SOT_THT:TO-92_Inline, symbol Transistor_FET:BS250
- removed R? (x4): 10k, symbol Device:R
- removed R?: R, symbol Device:R
- removed U?: IFX9201SG, symbol croptop:IFX9201SG
- added C?: 0.1uF, symbol Device:C
- added C? (x2): 10uF, symbol Device:C
- added J?: Power Test, symbol Connector:Conn_01x09_Male
- added J?: GPS Test, symbol Connector:Conn_01x03_Male
- added J?: Conn_01x04_Male, symbol Connector:Conn_01x04_Male
- added J?: ROT Test, symbol Connector:Conn_01x02_Male
- added J?: DRV Test, symbol Connector:Conn_01x03_Male
- added J?: ADC Test, symbol Connector:Conn_01x04_Male
- added J?: I2C Test, symbol Connector:Conn_01x02_Male
- added J?: BTN Test, symbol Connector:Conn_01x04_Male
- added J?: LED Test, symbol Connector:Conn_01x04_Male
- added J?: SPI2 Test, symbol Connector:Conn_01x04_Male
- added J?: SPI1 Test, symbol Connector:Conn_01x04_Male
- added U?: DRV8872, symbol croptop:DRV8872
- J?: value Battery 2 -> 12V Motor Battery
Connections:
- net labels added: ADC_CS, BTN_A, BTN_B, BTN_C, BTN_D, DRV_FLT, DRV_IN1, DRV_IN2, GPS_ONOFF, GPS_RST, GPS_TM, LED_A, LED_B, LED_C, LED_D, PKT_MCLR, PKT_PGEC, PKT_PGED, ROT_A, ROT_B, RPI_CS, TP_3V3_INT, TP_3V_BAT, TP_5V5_PUMP, TP_5V_USB, TP_ADC_CS, TP_ADC_DIN, TP_ADC_DOUT, TP_ADC_SCLK, TP_AGND, TP_AVDD, TP_DGND, TP_DVDD
- net labels removed: AD_CS, BN_A, BN_B, BN_C, BN_D, BTN_1, BTN_2, BTN_3, BTN_4, GP_ONOFF, GP_RST, GP_TM, LD_A, LD_B, LD_C, LD_D, LED_1, LED_2, LED_3, LED_4, MD_CS, PK_MCLR, PK_PGEC, PK_PGED, RE_A, RE_B, SCL_2, SDA_2
- wire segments 467 -> 507
- no-connect marks 26 -> 47
Other:
- note added: "RaspberryPI SPI Header"
- note added: "Test Point Headers"
- note removed: "FDS pg38\nadd C/R?"
- note removed: "GPIO Net Prefix Key:\nGP - GPS\nAC - Accelerometer\nTH - Temperature Sensor\nMD - Motor Driver\nPK - PICKit\nAD - Force Sensor\nBN - Buttons\nLD - LEDs\nRE - Rotary Encoder\n\n"
- note removed: "Place close\nto MCU"
- note removed: "RaspberryPI I2C Header"
- note removed: "To Do List:\n-Coin battery for GPS\n-On LED\n-External Oscillator\n-Redo Microcontroller Pinout\n-Testpoints\n-Power Switch\n-Pick a resistor notation"
- note removed: "USB Not\nUsed"
- moved on the sheet: C?, J?, JP?, R?

Commit message: Created BOM
Parts:
- added J?: Micro_SD_Card_Det, symbol croptop_rev1-rescue:Micro_SD_Card_Det
- added R? (x2): 10k, symbol Device:R
- J?: value Conn_01x04_Male -> Linear Encoder
- U?: symbol croptop:LIS3DH -> croptop_rev1-rescue:LIS3DH-croptop
- U?: symbol croptop:A2235-H -> croptop_rev1-rescue:A2235-H-croptop
- U?: symbol croptop:AD7799 -> croptop_rev1-rescue:AD7799-croptop
- U?: symbol croptop:HDC2010 -> croptop_rev1-rescue:HDC2010-croptop
- U?: symbol croptop:AZ1117 -> croptop_rev1-rescue:AZ1117-croptop
- U? (x2): symbol croptop:MC74HC125A -> croptop_rev1-rescue:MC74HC125A-croptop
- U?: symbol croptop:TPS2115A -> croptop_rev1-rescue:TPS2115A-croptop
- U?: symbol croptop:REG71055 -> croptop_rev1-rescue:REG71055-croptop
- U?: symbol croptop:TC1014 -> croptop_rev1-rescue:TC1014-croptop
- U?: symbol croptop:DRV8872 -> croptop_rev1-rescue:DRV8872-croptop
- U?: symbol croptop:PIC32MX575F512H -> croptop_rev1-rescue:PIC32MX575F512H-croptop
Connections:
- net labels added: LIN_VOLT, SD_CD, SD_CLK, SD_CS, SD_MISO, SD_MOSI
- wire segments 507 -> 529
Other:
- moved on the sheet: J?

Commit message: Added screen power supply
Parts:
- removed BT?: Coin, symbol Device:Battery_Cell
- removed C? (x2): 1uF, symbol Device:C
- removed C? (x2): 0.1uF, symbol Device:C
- removed J?: Rotary Encoder, symbol Connector:Conn_01x04_Male
- removed J?: Force Sensor, symbol Connector:Conn_01x04_Male
- removed J?: Micro_SD_Card_Det, symbol croptop_rev1-rescue:Micro_SD_Card_Det
- removed J?: Linear Actuator, symbol Connector:Conn_01x04_Male
- removed J?: 12V Motor Battery, symbol Connector:Conn_01x04_Male
- removed J?: Linear Encoder, symbol Connector:Conn_01x04_Male
- removed R? (x6): 2.2k, symbol Device:R
- removed R? (x4): 10k, symbol Device:R
- removed U?: A2235-H, symbol croptop_rev1-rescue:A2235-H-croptop
- removed U?: HDC2010, symbol croptop_rev1-rescue:HDC2010-croptop
- removed U?: AZ1117, symbol croptop_rev1-rescue:AZ1117-croptop
- removed U?: TPS2115A, symbol croptop_rev1-rescue:TPS2115A-croptop
- removed U?: PIC32MX575F512H, symbol croptop_rev1-rescue:PIC32MX575F512H-croptop
- added C? (x8): 0.1uF, symbol Device:C
- added C?: 10uF, symbol Device:C
- added C? (x2): 1uF, symbol Device:C
- added C? (x2): 27pF, symbol Device:C
- added C? (x3): 4.7uF, symbol Device:C
- added C?: 560pF, symbol Device:C
- added C? (x2): 18pF, symbol Device:C
- added D?: MBR0540, symbol Device:D
- added D?: 3SMAJ5935B, symbol Device:D_Schottky
- added D? (x4): D, symbol Device:D
- added J?: 54104-4031, symbol croptop_rev1-rescue:54104-4031
- added J?: Terminal Block, symbol Connector:Screw_Terminal_01x15
- added J?: USB_A, symbol Connector:USB_A
- added L?: 10uH, symbol Device:L
- added L?: 1uH, symbol Device:L
- added R? (x3): 10k, symbol Device:R
- added R?: R, symbol Device:R
- added R? (x3): 0, symbol Device:R
- added R? (x4): 220, symbol Device:R
- added R? (x4): 10, symbol Device:R
- added U?: PIC32MX795F512L, MODULE, symbol croptop_rev1-rescue:PIC32MX795F512L
- added U?: FAN5333BSX, symbol croptop_rev1-rescue:FAN5333BSX
- added U?: IS66WV51216EBLL, symbol croptop_rev1-rescue:IS66WV51216EBLL
- added U?: MIC23050, symbol croptop_rev1-rescue:MIC23050
- added U?: W25N01GV, symbol croptop_rev1-rescue:W25N01GV
- added U?: Si7006-A20, symbol croptop_rev1-rescue:Si7006-A20
- added U?: BU21026MUV-E2, symbol croptop_rev1-rescue:BU21026MUV-E2
- added U?: UCAM-M8Q, symbol croptop_rev1-rescue:UCAM-M8Q
- added Y?: CXO, symbol Device:Crystal
Connections:
- net labels added: ADC_A1+, ADC_A1-, ADC_GND, ADC_VDD, BLK_PWM, DRV_BAT, DRV_GND, DRV_OUT1, DRV_OUT2, GPS_RX, GPS_TX, LCD_B1, LCD_B2, LCD_B3, LCD_B4, LCD_B5, LCD_CS, LCD_DEN, LCD_G1, LCD_G2, LCD_G3, LCD_G4, LCD_G5, LCD_G6, LCD_HSYNC, LCD_LED+, LCD_LED-, LCD_R1, LCD_R2, LCD_R3, LCD_R4, LCD_R5, LCD_RESET, LCD_SHIFT, LCD_VSYNC, LIN_GND, LIN_IN, LIN_VDD, NAND_CS, NAND_HOLD, NAND_WP, PMPWR, RES_INT, ROT_A1, ROT_A2, ROT_GND, ROT_VDD, ROT_Y1, ROT_Y2, SCL_2, SDA_2, SRAM_CS, TCH_DOWN, TCH_LEFT, TCH_RIGHT, TCH_UP, USB_D+, USB_D-, VBUS
- net labels removed: SD_CD, SD_CLK, SD_CS, SD_MISO, SD_MOSI
- wire segments 529 -> 766
- no-connect marks 47 -> 41
Other:
- note added: "12V"
- note added: "3V3"
- note added: "A"
- note added: "A1+"
- note added: "A1-"
- note added: "Asynchronous SRAM"
- note added: "B"
- note added: "BAT"
- note added: "Ceramic, 10-20V Low ESR\nRun power to caps before pins"
- note added: "GND"
- note added: "IN"
- note added: "Load Cell"
- note added: "Motor"
- note added: "NAND Flash Memory\n"
- note added: "PIC32 Microcontroller"
- note added: "PICKit3 Header"
- note added: "POT"
- note added: "Peripheral Terminal Block"
- note added: "Peripheral USB Port"
- note added: "Pin 15"
- note added: "Pin 16"
- note added: "Pin 2"
- note added: "Pin 30"
- note added: "Pin 31\n"
- note added: "Pin 36"
- note added: "Pin 37"
- note added: "Pin 45"
- note added: "Pin 46"
- note added: "Pin 62"
- note added: "Pin 65"
- note added: "Pin 75"
- note added: "Possibly\nD.N.P."
- note added: "Resistive Touch Driver"
- note added: "Rot Encoder"
- note added: "TFT LCD Header"
- note removed: "(This area will contain the RaspberryPi SO-DIMM\nand Peripherals in later revisions of this board)\n"
- note removed: "3V\n"
- note removed: "AVDD & AVSS\nDecoupling"
- note removed: "Ceramic, 10-20V Low ESR\nRun power caps then pins"
- note removed: "Check: R Values"
- note removed: "Check: Resistor Values"
- note removed: "External\nAntenna"
- note removed: "Microcontroller Decoupling Capacitors"
- note removed: "PIC32MX Microcontroller"
- note removed: "PICKit Programming Header"
- note removed: "Pin 10"
- note removed: "Pin 19"
- note removed: "Pin 20"
- note removed: "Pin 25"
- note removed: "Pin 26"
- note removed: "Pin 38"
- note removed: "Pin 41"
- note removed: "Pin 57"
- note removed: "Pin 9"
- note removed: "RS232"
- note removed: "RaspberryPI SPI Header"
- note removed: "Self Start"
- note removed: "Test Point Headers"
- note removed: "VDD & VSS\nDecoupling"
- moved on the sheet: C?, D?, J?, JP?, L?, R?, SW?, U?
