File: KiCAD/mcucap.sch (KiCad schematic (older format))
At the start: 7 parts

Commit message: Decoupling caps & more
Parts:
- removed C? (x7): 0.1uF, symbol Device:C
Other:
- note removed: "Ceramic, 10-20V Low ESR\nRun power to caps before pins"
- note removed: "No Pin"
- note removed: "Pin 15"
- note removed: "Pin 16"
- note removed: "Pin 2"
- note removed: "Pin 30"
- note removed: "Pin 31\n"
- note removed: "Pin 36"
- note removed: "Pin 37"
- note removed: "Pin 45"
- note removed: "Pin 46"
- note removed: "Pin 62"
- note removed: "Pin 65"
- note removed: "Pin 75"
