File: KiCAD/croptop_rev1.sch (KiCad schematic (older format))
At the start: 0 parts

Commit message: Decoupling caps & more
Other:
- note added: "List of tasks:\n-Pick all caps and inductors\n-Shorten symbol leads\n-Fiducials\n-Move ground pin to sides\n-Test points\n-Delete 2 btns and 2 leds\n-Consistant blue text labels"
Changed lines of the file:
@@
 $Descr USLetter 11000 8500
 encoding utf-8
-Sheet 1 8
+Sheet 1 7
 Title "CropTop"
-Date "2018-11-18"
-Rev "Revision 1"
+Date "2018-11-20"
+Rev "Revision 8"
 Comp "University of Idaho"
-Comment1 "Designer 1: Kennedy Caisley"
-Comment2 "Designer 2: Ryan Donahue"
+Comment1 "Kennedy Caisley, Ryan Donahue"
+Comment2 ""
 Comment3 ""
 Comment4 ""
@@
 $EndSheet
 $Sheet
-S 5500 4500 1200 900
-U 66A12209
-F0 "Microcontroller Decoupling" 50
-F1 "mcucap.sch" 50
-$EndSheet
-$Sheet
 S 4100 3300 1200 900
 U 66A12230
@@
 $EndSheet
 $Sheet
-S 4100 5700 1200 900
+S 5500 4500 1200 900
 U 66A201BE
 F0 "Temporary Debugging" 50
@@
 Text Notes 4100 1750 0    138  ~ 28
 List of Schematic Sheets
+Text Notes 7350 3350 0    79   ~ 0
+List of tasks:\n-Pick all caps and inductors\n-Shorten symbol leads\n-Fiducials\n-Move ground pin to sides\n-Test points\n-Delete 2 btns and 2 leds\n-Consistant blue text labels
 $EndSCHEMATC

Commit message: Before changing files
Other:
- note removed: "List of tasks:\n-Pick all caps and inductors\n-Shorten symbol leads\n-Fiducials\n-Move ground pin to sides\n-Test points\n-Delete 2 btns and 2 leds\n-Consistant blue text labels"
Changed lines of the file:
@@
 $Descr USLetter 11000 8500
 encoding utf-8
-Sheet 1 7
+Sheet 1 6
 Title "CropTop"
 Date "2018-11-20"
@@
 F1 "onboard.sch" 50
 $EndSheet
-$Sheet
-S 5500 4500 1200 900
-U 66A201BE
-F0 "Temporary Debugging" 50
-F1 "debug.sch" 50
-$EndSheet
 Text Notes 4100 1750 0    138  ~ 28
 List of Schematic Sheets
-Text Notes 7350 3350 0    79   ~ 0
-List of tasks:\n-Pick all caps and inductors\n-Shorten symbol leads\n-Fiducials\n-Move ground pin to sides\n-Test points\n-Delete 2 btns and 2 leds\n-Consistant blue text labels
 $EndSCHEMATC
