File: KiCAD/lcd.sch (KiCad schematic (older format))
At the start: 24 parts

Commit message: Decoupling caps & more
Parts:
- removed C? (x3): 0.1uF, symbol Device:C
- removed C? (x3): 1uF, symbol Device:C
- removed C? (x3): 10uF, symbol Device:C
- added C? (x3): 0.1uF, symbol Device:C
- added C? (x3): 1uF, symbol Device:C
- added C? (x3): 10uF, symbol Device:C
Connections:
- net DGND: now also C?.2, C?.2, C?.2, C?.2, C?.2, C?.2, C?.2, C?.2, C?.2
- net DVDD: now also C?.1, C?.1, C?.1, C?.1, C?.1, C?.1, C?.1, C?.1, C?.1
- net LCD_LED+ renamed LCD_ANODE
- net LCD_LED- renamed LCD_CATHODE
Other:
- note added: "Pick Diodes"
- note removed: "-Pick ESD Diodes\n-Change LCD_LED+ and LCD_LED- to PWR Flags"
- moved on the sheet: C?, D?, J?, R?, U?

Commit message: Before changing files
Parts:
- removed C? (x2): 0.1uF, symbol Device:C
- removed C? (x3): 1uF, symbol Device:C
- removed C? (x2): 10uF, symbol Device:C
- removed D? (x4): D, symbol Device:D
- removed J?: 54104-4031, symbol croptop_rev1-rescue:54104-4031
- removed U?: BU21026MUV-E2, symbol croptop_rev1-rescue:BU21026MUV-E2
- removed U?: IS66WV51216EBLL, symbol croptop_rev1-rescue:IS66WV51216EBLL
- added C? (x2): 0.1uF, symbol Device:C
- added C? (x2): 10uF, symbol Device:C
- added D? (x4): BAT42W, symbol Device:D_Schottky
- added J?: 54104-4031, symbol CropTop:54104-4031
- added U?: IS66WV51216EBLL, symbol CropTop:IS66WV51216EBLL
- added U?: BU21026MUV-E2, symbol CropTop:BU21026MUV-E2
Connections:
- net DGND: now also C?.2, C?.2, C?.2, C?.2, D?.2 (A), D?.2 (A), D?.2 (A), D?.2 (A), J?.29 (GND), J?.3 (GND), J?.36 (GND), U?.1 (AD1), U?.12 (GND), U?.18 (GND), U?.34 (GND), U?.39 (~LB), U?.4 (AD0), U?.40 (~UB), U?.7 (AUX)
- net DVDD: now also C?.1, C?.1, C?.1, C?.1, J?.4 (VDD), U?.11 (VDD), U?.33 (VDD), U?.8 (VDD)
- net LCD_ANODE: now also J?.2 (LED+)
- net LCD_B1: now also J?.24 (B3), U?.7 (I/O0)
- net LCD_B2: now also J?.25 (B4), U?.8 (I/O1)
- net LCD_B3: now also J?.26 (B5), U?.9 (I/O2)
- net LCD_B4: now also J?.27 (B6), U?.10 (I/O3)
- net LCD_B5: now also J?.21 (B0), J?.22 (B1), J?.23 (B2), J?.28 (B7), U?.13 (I/O4)
- net LCD_CATHODE: now also J?.1 (LED-)
- net LCD_CS: now also U?.41 (~OE)
- net LCD_DEN: now also J?.34 (DE)
- net LCD_G1: now also J?.15 (G2), U?.14 (I/O5)
- net LCD_G2: now also J?.16 (G3), U?.15 (I/O6)
- net LCD_G3: now also J?.17 (G4), U?.16 (I/O7)
- net LCD_G4: now also J?.18 (G5), U?.29 (I/O8)
- net LCD_G5: now also J?.19 (G6), U?.30 (I/O9)
- net LCD_G6: now also J?.13 (G0), J?.14 (G1), J?.20 (G7), U?.31 (I/O10)
- net LCD_HSYNC: now also J?.32 (HSYNC)
- net LCD_R1: now also J?.8 (R3), U?.32 (I/O11)
- net LCD_R2: now also J?.9 (R4), U?.35 (I/O12)
- net LCD_R3: now also J?.10 (R5), U?.36 (I/O13)
- net LCD_R4: now also J?.11 (R6), U?.37 (I/O14)
- net LCD_R5: now also J?.12 (R7), J?.5 (R0), J?.6 (R1), J?.7 (R2), U?.38 (I/O15)
- net LCD_RESET: now also J?.31 (DISP)
- net LCD_SHIFT: now also J?.30 (CLK)
- net LCD_VSYNC: now also J?.33 (VSYNC)
- net PMPWR: now also U?.17 (~WE)
- net RES_INT: now also U?.5 (INT)
- net SCL_1: now also U?.2 (SCL)
- net SDA_1: now also U?.3 (SDA)
- net SRAM_A0: now also U?.5 (A0)
- net SRAM_A1: now also U?.4 (A1)
- net SRAM_A10: now also U?.25 (A10)
- net SRAM_A11: now also U?.24 (A11)
- net SRAM_A12: now also U?.22 (A12)
- net SRAM_A13: now also U?.21 (A13)
- net SRAM_A14: now also U?.20 (A14)
- net SRAM_A15: now also U?.19 (A15)
- net SRAM_A16: now also U?.18 (A16)
- net SRAM_A17: now also U?.23 (A17)
- net SRAM_A18: now also U?.28 (A18)
- net SRAM_A2: now also U?.3 (A2)
- net SRAM_A3: now also U?.2 (A3)
- net SRAM_A4: now also U?.1 (A4)
- net SRAM_A5: now also U?.44 (A5)
- net SRAM_A6: now also U?.43 (A6)
- net SRAM_A7: now also U?.42 (A7)
- net SRAM_A8: now also U?.27 (A8)
- net SRAM_A9: now also U?.26 (A9)
- net SRAM_CS: now also U?.6 (~CS1)
- net TCH_DOWN: now also D?.1 (K), J?.38 (YD)
- net TCH_LEFT: now also D?.1 (K), J?.39 (XL)
- net TCH_RIGHT: now also D?.1 (K), J?.37 (XR)
- net TCH_UP: now also D?.1 (K), J?.40 (YU)
- net at C?.1, R?.1: now also U?.15 (YN)
- net at C?.1, R?.1: now also U?.14 (XN)
- net at C?.1, R?.1: now also U?.11 (XP)
- net at C?.1, R?.1: now also U?.12 (YP)
Other:
- note removed: "Pick Diodes"
- moved on the sheet: C?, R?
