File: KiCAD/mcu.sch (KiCad schematic (older format))
At the start: 36 parts

Commit message: Decoupling caps & more
Parts:
- added C? (x7): 0.1uF, symbol Device:C
- added C?: 10uF, symbol Device:C
- U?: symbol croptop_rev1-rescue:PIC32MX795F512L -> croptop_rev1-rescue:PIC32MX795F512L-croptop_rev1-rescue
Connections:
- net DGND: now also C?.2, C?.2, C?.2, C?.2, C?.2, C?.2, C?.2, C?.2
- net DVDD: now also C?.1, C?.1, C?.1, C?.1, C?.1, C?.1, C?.1, C?.1
Other:
- note added: "Inductor"
- note added: "Need new caps for GPA PIC"
- note added: "No Pin"
- note added: "Pin 15"
- note added: "Pin 16"
- note added: "Pin 2"
- note added: "Pin 30"
- note added: "Pin 31\n"
- note added: "Pin 36"
- note added: "Pin 37"
- note added: "Pin 45"
- note added: "Pin 46"
- note added: "Pin 62"
- note added: "Pin 65"
- note added: "Pin 75"
- note added: "Replace"
- note added: "Replace\nw/ New"
- note added: "Supply \nmust\nbe 5V\nnot 3V3"
- moved on the sheet: C?, J?, R?

Commit message: Before changing files
Parts:
- removed R?: 0, symbol Device:R
- removed U?: PIC32MX795F512L, MODULE, symbol croptop_rev1-rescue:PIC32MX795F512L-croptop_rev1-rescue
- added C?: 0.1uF, symbol Device:C
- added L?: 10uH, symbol Device:L
- added TP?: TestPoint, symbol Connector:TestPoint
- added U?: PIC32MX795F512L, MODULE, symbol CropTop:PIC32MX795F512L
- C? (x2): value 18pF -> 26pF
- R? (x2): value 2.2k -> 2K
Connections:
- net VBUS is gone; now on net DVDD: J?.1 (VBUS)
- net BLK_PWM: now also U?.78 (OC4)
- net BTN_A: now also U?.20 (RB5)
- net BTN_B: now also U?.21 (RB4)
- net BTN_C: now also U?.22 (RB3)
- net BTN_D: now also U?.23 (RB2)
- net DGND: now also C?.2, U?.15 (VSS), U?.31 (AVSS), U?.36 (VSS), U?.45 (VSS), U?.65 (VSS), U?.75 (VSS)
- net DRV_FLT: now also U?.82 (CN15)
- net DRV_IN1: now also U?.76 (OC2)
- net DRV_IN2: now also U?.77 (OC3)
- net DVDD: now also C?.1, L?.1, U?.16 (VDD), U?.2 (VDD), U?.37 (VDD), U?.46 (VDD), U?.54 (VBUS), U?.55 (VUSB3V3), U?.62 (VDD), U?.86 (VDD)
- net GPS_INT: now also U?.32 (RB8)
- net GPS_RX: now also U?.39 (U5TX/RF13)
- net GPS_TX: now also U?.40 (U5RX/RF12)
- net LED_A: now also U?.6 (RC1)
- net LED_B: now also U?.7 (RC2)
- net LED_C: now also U?.8 (RC3)
- net LED_D: now also U?.9 (RC4)
- net LIN_VOLT: now also U?.33 (AN9)
- net MOSI_1: now also U?.53 (SDO3)
- net NAND_CS: now also U?.47 (SS3)
- net NAND_HOLD: now also U?.61 (RA5)
- net NAND_WP: now also U?.60 (RA4)
- net PKT_MCLR: now also U?.13 (~MCLR)
- net PKT_PGEC: now also U?.26 (PGEC2)
- net PKT_PGED: now also U?.27 (PGED2)
- net PMPWR: now also U?.81 (PMWR)
- net RES_INT: now also U?.18 (INT1/RE8)
- net ROT_Y1: now also U?.68 (IC1)
- net ROT_Y2: now also U?.69 (IC2)
- net SCLK_1: now also U?.48 (SCK3)
- net SCL_1: now also U?.66 (SCL1)
- net SDA_1: now also U?.67 (SDA1)
- net SRAM_A0: now also U?.44 (PMA0)
- net SRAM_A1: now also U?.43 (PMA1)
- net SRAM_A10: now also U?.42 (PMA10)
- net SRAM_A11: now also U?.41 (PMA11)
- net SRAM_A12: now also U?.35 (PMA12)
- net SRAM_A13: now also U?.34 (PMA13)
- net SRAM_A14: now also U?.71 (PMA14)
- net SRAM_A15: now also U?.70 (PMA15)
- net SRAM_A16: now also U?.97 (RG13)
- net SRAM_A17: now also U?.96 (RG12)
- net SRAM_A18: now also U?.95 (RG14)
- net SRAM_A2: now also U?.14 (PMA2)
- net SRAM_A3: now also U?.12 (PMA3)
- net SRAM_A4: now also U?.11 (PMA4)
- net SRAM_A5: now also U?.10 (PMA5)
- net SRAM_A6: now also U?.29 (PMA6)
- net SRAM_A7: now also U?.28 (PMA7)
- net SRAM_A8: now also U?.50 (PMA8)
- net SRAM_A9: now also U?.49 (PMA9)
- net SRAM_CS: now also U?.1 (RG15)
- net USB_D+: now also U?.57 (D+)
- net USB_D-: now also U?.56 (D-)
- net at C?.1: now also U?.85 (V_CAP)
- net at R?.1: now also U?.100 (PMD4)
- net at R?.1: now also U?.3 (PMD5)
- net at R?.2: now also U?.38 (RA1)
- net at R?.1: now also U?.4 (PMD6)
- net at R?.1: now also U?.5 (PMD7)
- net at R?.2: now also U?.52 (SDI3)
- net at C?.1, Y?.2: now also U?.63 (OSC1)
- net at R?.2: now also U?.64 (OSC2)
- net at R?.2: now also U?.72 (RD0)
- net at R?.2: now also U?.73 (RC13)
- net at R?.2: now also U?.74 (RC14)
- net at R?.1: now also U?.79 (PMD12)
- net at R?.1: now also U?.80 (PMD13)
- net at R?.1: now also U?.83 (PMD14)
- net at R?.1: now also U?.84 (PMD15)
- net at R?.1: now also U?.87 (PMD11)
- net at R?.1: now also U?.88 (PMD10)
- net at R?.1: now also U?.89 (PMD9)
- net at R?.1: now also U?.90 (PMD8)
- net at R?.2: now also U?.91 (RA6)
- net at R?.2: now also U?.92 (RA7)
- net at R?.1: now also U?.93 (PMD0)
- net at R?.1: now also U?.94 (PMD1)
- net at R?.1: now also U?.98 (PMD2)
- net at R?.1: now also U?.99 (PMD3)
- new net: L?.2, U?.30 (AVDD)
Other:
- note added: "Bulk"
- note removed: "Consider increasing caps\nto compensate for \nstray capacitance"
- note removed: "Inductor"
- note removed: "Need new caps for GPA PIC"
- note removed: "Replace"
- note removed: "Replace\nw/ New"
- moved on the sheet: C?, J?, R?, Y?
