File: KiCAD/onboard.sch (KiCad schematic (older format))
At the start: 9 parts

Commit message: Decoupling caps & more
Parts:
- added C? (x3): 0.1uF, symbol Device:C
- added C? (x3): 1uF, symbol Device:C
- added C? (x3): 10uF, symbol Device:C
Connections:
- net DGND: now also C?.2, C?.2, C?.2, C?.2, C?.2, C?.2, C?.2, C?.2, C?.2
- net DVDD: now also C?.1, C?.1, C?.1, C?.1, C?.1, C?.1, C?.1, C?.1, C?.1
Other:
- note added: "Make less ugly"
- note added: "Replace\nw/ New"
- moved on the sheet: C?, R?, U?

Commit message: Before changing files
Parts:
- removed C? (x3): 0.1uF, symbol Device:C
- removed C? (x3): 1uF, symbol Device:C
- removed C? (x3): 10uF, symbol Device:C
- removed C?: 4.7uF, symbol Device:C
- removed R? (x2): 10, symbol Device:R
- removed U?: LIS3DH, symbol croptop_rev1-rescue:LIS3DH-croptop
- removed U?: W25N01GV, symbol croptop_rev1-rescue:W25N01GV
- removed U?: UCAM-M8Q, symbol croptop_rev1-rescue:UCAM-M8Q
- removed U?: Si7006-A20, symbol croptop_rev1-rescue:Si7006-A20
- added C? (x4): 0.1uF, symbol Device:C
- added C? (x4): 10uF, symbol Device:C
- added D?: LED4, symbol Device:LED
- added D?: LED3, symbol Device:LED
- added D?: LED2, symbol Device:LED
- added D?: LED1, symbol Device:LED
- added R? (x2): 10, symbol Device:R
- added R? (x8): 10k, symbol Device:R
- added R? (x4): 100, symbol Device:R
- added SW?: BTNA, symbol Switch:SW_Push
- added SW?: BTNB, symbol Switch:SW_Push
- added SW?: BTNC, symbol Switch:SW_Push
- added SW?: BTND, symbol Switch:SW_Push
- added U?: UCAM-M8Q, symbol CropTop:UCAM-M8Q
- added U?: LIS3DH, symbol CropTop:LIS3DH
- added U?: Si7006-A20, symbol CropTop:Si7006-A20
- added U?: W25N01GV, symbol CropTop:W25N01GV
Connections:
- net DGND: now also C?.2, C?.2, C?.2, C?.2, C?.2, C?.2, C?.2, C?.2, R?.1, R?.1, R?.1, R?.1, R?.2, R?.2, R?.2, R?.2, U?.10 (GND), U?.10 (RES), U?.11 (GND), U?.12 (GND), U?.12 (GND), U?.13 (GND), U?.14 (GND), U?.15 (GND), U?.18 (GND), U?.19 (GND), U?.2 (GND), U?.21 (GND), U?.22 (GND), U?.27 (GND), U?.31 (GND), U?.4 (GND), U?.4 (GND), U?.5 (GND), U?.5 (GND)
- net DVDD: now also C?.1, C?.1, C?.1, C?.1, C?.1, C?.1, C?.1, C?.1, SW?.2, SW?.2, SW?.2, SW?.2, U?.1 (VCC_IO), U?.1 (Vdd_IO), U?.14 (Vdd), U?.5 (VDD), U?.7 (SA0), U?.8 (CS), U?.8 (VCC), U?.8 (V_BCKP), U?.9 (VCC)
- net GPS_INT: now also U?.7 (EXTINT)
- net MISO_1: now also U?.2 (DO)
- net MOSI_1: now also R?.2
- net NAND_CS: now also U?.1 (~CS)
- net NAND_HOLD: now also U?.7 (~HOLD)
- net NAND_WP: now also U?.3 (~WP)
- net SCLK_1: now also R?.2
- net SCL_1: now also U?.4 (SCL), U?.6 (SCL), U?.6 (SCL)
- net SDA_1: now also U?.1 (SDA), U?.3 (SDA), U?.6 (SDA)
- net at R?.1: now also U?.25 (TXD)
- net at R?.1: now also U?.26 (RXD)
- new net: U?.16 (RF_OUT), U?.17 (RF_IN)
- new net: R?.1, U?.5 (DI)
- new net: R?.1, U?.6 (CLK)
- new net: R?.1, R?.2, SW?.1 (x4)
- new net: D?.1 (K), R?.2 (x4)
- new net BTN_A: R?.1
- new net BTN_B: R?.1
- new net BTN_C: R?.1
- new net BTN_D: R?.1
- new net LED_A: D?.2 (A)
- new net LED_B: D?.2 (A)
- new net LED_C: D?.2 (A)
- new net LED_D: D?.2 (A)
Other:
- note added: "Debugging Buttons and LEDs"
- note removed: "Make less ugly"
- note removed: "Replace\nw/ New"
- moved on the sheet: R?
