File: KiCAD/psu.sch (KiCad schematic (older format))
At the start: 26 parts

Commit message: Decoupling caps & more
Parts:
- removed C? (x2): 4.7uF, symbol Device:C
- removed C?: 10uF, symbol Device:C
- removed C? (x2): 1uF, symbol Device:C
- removed C?: 0.1uF, symbol Device:C
- removed C? (x2): 27pF, symbol Device:C
- added C? (x4): 10uF, symbol Device:C
- added C? (x5): 0.1uF, symbol Device:C
- added C? (x5): 1uF, symbol Device:C
Connections:
- net LCD_LED+ is gone; now on net LCD_ANODE: D?.1 (K)
- net AGND: now also C?.2, C?.2, C?.2, C?.2, C?.2, C?.2, C?.2, C?.2, C?.2, C?.2, C?.2, C?.2, C?.2, C?.2
- net DVDD: now also C?.1, C?.1, C?.1
- net DVDD_UNREG: now also C?.1, C?.1, C?.1, C?.1, C?.1, C?.1
- net LCD_ANODE: now reaches D?.1 (K)
- net LCD_ANODE: now also C?.1, C?.1, C?.1
- net LCD_LED- renamed LCD_CATHODE
- net LCD_CATHODE: now also C?.1, C?.1
Other:
- note added: "25.6"
- note added: "Check\nCurrent\nLimit"
- note added: "Need to do\nanything\nto get 25.6V?"
- note added: "Pick D"
- note removed: "5.5V"
- moved on the sheet: C?, D?, J?, L?, R?, U?

Commit message: Before changing files
Parts:
- removed C?: 10uF, symbol Device:C
- removed C?: 1uF, symbol Device:C
- removed D?: MBR0540, symbol Device:D
- removed D?: 3SMAJ5935B, symbol Device:D_Schottky
- removed L?: 1uH, symbol Device:L
- removed U?: REG71055, symbol croptop_rev1-rescue:REG71055-croptop
- removed U?: TC1014, symbol croptop_rev1-rescue:TC1014-croptop
- removed U?: MIC23050, symbol croptop_rev1-rescue:MIC23050
- removed U?: FAN5333BSX, symbol croptop_rev1-rescue:FAN5333BSX
- added D?: 3SMAJ5935B, symbol Device:D_Zener
- added D?: BAT42W, symbol Device:D_Schottky
- added L?: 1uH, symbol Device:L
- added U?: FAN5333BSX, symbol CropTop:FAN5333BSX
- added U?: MIC23050, symbol CropTop:MIC23050
- added U?: REG71055, symbol CropTop:REG71055
- added U?: TC1014, symbol CropTop:TC1014
Connections:
- net AGND: now also U?.2 (GND), U?.2 (GND), U?.6 (AGND), U?.8 (PGND), U?.~ (GND)
- net AVDD: now also U?.5 (VOUT)
- net BLK_PWM: now also U?.4 (~SHDN)
- net DVDD: now also L?.1, U?.4 (SNS)
- net DVDD_UNREG: now also U?.2 (EN), U?.3 (EN), U?.5 (VIN), U?.5 (VIN), U?.7 (VIN)
- net LCD_ANODE: now also D?.1 (K), D?.1 (K)
- net LCD_CATHODE: now also D?.2 (A), U?.3 (FB)
- net at C?.1, C?.1: now also U?.1 (VIN), U?.1 (VOUT), U?.3 (~SHDN)
- net at C?.1: now also U?.6 (C+)
- net at C?.2: now also U?.4 (C-)
- net at C?.1: now also U?.4 (BP)
- net at C?.1: now also U?.5 (CFF)
- net at L?.1: now also D?.2 (A), U?.1 (SW)
- new net: L?.2, U?.1 (SW)
Other:
- note added: "25.6V"
- note added: "add led"
- note removed: "25.6"
- note removed: "Need to do\nanything\nto get 25.6V?"
- note removed: "Pick D"
- moved on the sheet: C?
