File: KiCAD/croptop_io.sch (KiCad schematic (older format))
At the start: 65 parts, among them J5 Terminal Block, J6 DNP, J7 DNP, U10 AD7799, U11 74HCT125D, U17 DT6250-06MR-13, U18 PUSBM5V5X4, U8 74HCT125D, U9 DRV8872

Commit message: Got to PCB layout
Parts:
- D9: footprint (none) -> Package_TO_SOT_SMD:TO-252-3_TabPin2
- J5: footprint (none) -> TerminalBlock_4Ucon:TerminalBlock_4Ucon_1x15_P3.50mm_Horizontal
- J6, J7: footprint (none) -> Connector_PinHeader_2.54mm:PinHeader_1x04_P2.54mm_Vertical
- U17: footprint (none) -> Package_SO:MSOP-8_3x3mm_P0.65mm
- U18: footprint (none) -> croptop:PUSBM5V5X4
Changed lines of the file:
@@
 F 0 "D9" H 4575 4825 50  0000 C CNN
 F 1 "SBRD10200TR" H 4550 4925 50  0000 C CNN
-F 2 "" H 4600 5050 50  0001 C CNN
+F 2 "Package_TO_SOT_SMD:TO-252-3_TabPin2" H 4600 5050 50  0001 C CNN
 F 3 "~" H 4600 5050 50  0001 C CNN
 	1    4600 5050
@@
 F 0 "J5" V 3025 6600 50  0000 L CNN
 F 1 "Terminal Block" V 3125 6125 50  0000 L CNN
-F 2 "" H 3075 7500 50  0001 C CNN
+F 2 "TerminalBlock_4Ucon:TerminalBlock_4Ucon_1x15_P3.50mm_Horizontal" H 3075 7500 50  0001 C CNN
 F 3 "~" H 3075 7500 50  0001 C CNN
 	1    3075 7500
@@
 F 0 "J6" H 10279 2142 50  0000 L CNN
 F 1 "DNP" H 10279 2051 50  0000 L CNN
-F 2 "" H 10200 2150 50  0001 C CNN
+F 2 "Connector_PinHeader_2.54mm:PinHeader_1x04_P2.54mm_Vertical" H 10200 2150 50  0001 C CNN
 F 3 "~" H 10200 2150 50  0001 C CNN
 	1    10200 2150
@@
 F 0 "J7" H 10279 2592 50  0000 L CNN
 F 1 "DNP" H 10279 2501 50  0000 L CNN
-F 2 "" H 10200 2600 50  0001 C CNN
+F 2 "Connector_PinHeader_2.54mm:PinHeader_1x04_P2.54mm_Vertical" H 10200 2600 50  0001 C CNN
 F 3 "~" H 10200 2600 50  0001 C CNN
 	1    10200 2600
@@
 F 0 "U17" H 8250 3076 50  0000 C CNN
 F 1 "DT6250-06MR-13" H 8250 2985 50  0000 C CNN
-F 2 "" V 8500 2750 50  0001 C CNN
+F 2 "Package_SO:MSOP-8_3x3mm_P0.65mm" V 8500 2750 50  0001 C CNN
 F 3 "" V 8500 2750 50  0001 C CNN
 	1    8250 3300
@@
 F 0 "U18" H 9200 5675 50  0000 C CNN
 F 1 "PUSBM5V5X4" H 9200 5775 50  0000 C CNN
-F 2 "" V 9450 5550 50  0001 C CNN
+F 2 "croptop:PUSBM5V5X4" V 9450 5550 50  0001 C CNN
 F 3 "" V 9450 5550 50  0001 C CNN
 	1    9200 6100

Commit message: Save before netlist read
Parts:
- removed C55: 100uF, Capacitor_SMD:CP_Elec_6.3x7.7, symbol Device:CP1
Changed lines of the file:
@@
 Wire Wire Line
 	3200 5150 3200 5450
-$Comp
-L Device:CP1 C55
-U 1 1 5C2CADB9
-P 4950 1300
-F 0 "C55" H 5065 1346 50  0000 L CNN
-F 1 "100uF" H 5065 1255 50  0000 L CNN
-F 2 "Capacitor_SMD:CP_Elec_6.3x7.7" H 4950 1300 50  0001 C CNN
-F 3 "~" H 4950 1300 50  0001 C CNN
-	1    4950 1300
-	1    0    0    -1
-$EndComp
-Wire Wire Line
-	4950 1450 4950 1500
-Wire Wire Line
-	4950 1100 4950 1150
 Wire Wire Line
 	3100 5050 3500 5050
@@
 Wire Wire Line
 	4250 1100 4600 1100
-Connection ~ 4600 1100
-Wire Wire Line
-	4600 1100 4950 1100
 Connection ~ 9250 1900
 Wire Wire Line
@@
 	1    0    0    -1
 $EndComp
-$Comp
-L CropTop:AGND #PWR0113
-U 1 1 5C4CEC28
-P 4950 1500
-F 0 "#PWR0113" H 4950 1250 50  0001 C CNN
-F 1 "AGND" H 4955 1327 50  0000 C CNN
-F 2 "" H 4950 1500 50  0001 C CNN
-F 3 "" H 4950 1500 50  0001 C CNN
-	1    4950 1500
-	1    0    0    -1
-$EndComp

Commit message: Dec 18th
Parts:
- removed C72: 0.1uF, Capacitor_SMD:C_0402_1005Metric, symbol Device:C
- D9: footprint Package_TO_SOT_SMD:TO-252-3_TabPin2 -> croptop:SizeOfThisLad
Connections:
- net ADC_A1+: now also U17.4 (IO1); no longer U17.6 (IO3)
- net ADC_A1-: now also U17.3 (IO3); no longer U17.5 (IO2)
- net ROT_A1: now also U11.2 (A1); no longer U11.3 (Y1)
- net ROT_A2: now also U11.5 (A2); no longer U11.6 (Y2)
- net at J6.3 (Pin_3), R43.1: now also U17.6 (IO3); no longer U17.4 (IO1)
- net at J6.4 (Pin_4), R46.1: now also U17.5 (IO2); no longer U17.3 (IO3)
- net at C52.1, C61.2, R42.2: now also U10.7 (AIN2(+)); no longer U10.5 (AIN1(+))
- net at C52.2, C60.2, R45.2: now also U10.8 (AIN2(-)); no longer U10.6 (AIN1(-))
- net at C53.1, C59.2, R43.2: now also U10.5 (AIN1(+)); no longer U10.7 (AIN2(+))
- net at C53.2, C58.2, R46.2: now also U10.6 (AIN1(-)); no longer U10.8 (AIN2(-))
- net at R48.1: now also U11.3 (Y1); no longer U11.2 (A1)
- net at R49.1: now also U11.6 (Y2); no longer U11.5 (A2)
Other:
- moved on the sheet: C52, C53, C58, C59, C60, C61, J6, R42, R43, R45, R46
Changed lines of the file:
@@
 F 0 "D9" H 4575 4825 50  0000 C CNN
 F 1 "SBRD10200TR" H 4550 4925 50  0000 C CNN
-F 2 "Package_TO_SOT_SMD:TO-252-3_TabPin2" H 4600 5050 50  0001 C CNN
+F 2 "croptop:SizeOfThisLad" H 4600 5050 50  0001 C CNN
 F 3 "~" H 4600 5050 50  0001 C CNN
 	1    4600 5050
@@
 L Device:R R?
 U 1 1 5C644C28
-P 6700 1900
+P 6700 2200
 AR Path="/5C644C28" Ref="R?"  Part="1"
 AR Path="/669AB112/5C644C28" Ref="R42"  Part="1"
-F 0 "R42" V 6600 1900 50  0000 C CNN
+F 0 "R42" V 6600 2200 50  0000 C CNN
+F 1 "100" V 6700 2200 50  0000 C CNN
+F 2 "Resistor_SMD:R_0402_1005Metric" V 6630 2200 50  0001 C CNN
+F 3 "~" H 6700 2200 50  0001 C CNN
+	1    6700 2200
+	0    1    1    0
+$EndComp
+$Comp
+L Device:R R?
+U 1 1 5C644C2F
+P 7000 2350
+AR Path="/5C644C2F" Ref="R?"  Part="1"
+AR Path="/669AB112/5C644C2F" Ref="R45"  Part="1"
+F 0 "R45" V 6900 2350 50  0000 C CNN
+F 1 "100" V 7000 2350 50  0000 C CNN
+F 2 "Resistor_SMD:R_0402_1005Metric" V 6930 2350 50  0001 C CNN
+F 3 "~" H 7000 2350 50  0001 C CNN
+	1    7000 2350
+	0    1    1    0
+$EndComp
+$Comp
+L Device:R R?
+U 1 1 5C644C36
+P 6700 1900
+AR Path="/5C644C36" Ref="R?"  Part="1"
+AR Path="/669AB112/5C644C36" Ref="R43"  Part="1"
+F 0 "R43" V 6600 1900 50  0000 C CNN
 F 1 "100" V 6700 1900 50  0000 C CNN
 F 2 "Resistor_SMD:R_0402_1005Metric" V 6630 1900 50  0001 C CNN
@@
 $Comp
 L Device:R R?
-U 1 1 5C644C2F
+U 1 1 5C644C3D
 P 7000 2050
-AR Path="/5C644C2F" Ref="R?"  Part="1"
-AR Path="/669AB112/5C644C2F" Ref="R45"  Part="1"
-F 0 "R45" V 6900 2050 50  0000 C CNN
+AR Path="/5C644C3D" Ref="R?"  Part="1"
+AR Path="/669AB112/5C644C3D" Ref="R46"  Part="1"
+F 0 "R46" V 6900 2050 50  0000 C CNN
 F 1 "100" V 7000 2050 50  0000 C CNN
 F 2 "Resistor_SMD:R_0402_1005Metric" V 6930 2050 50  0001 C CNN
 F 3 "~" H 7000 2050 50  0001 C CNN
 	1    7000 2050
-	0    1    1    0
-$EndComp
-$Comp
-L Device:R R?
-U 1 1 5C644C36
-P 6700 2200
-AR Path="/5C644C36" Ref="R?"  Part="1"
-AR Path="/669AB112/5C644C36" Ref="R43"  Part="1"
-F 0 "R43" V 6600 2200 50  0000 C CNN
-F 1 "100" V 6700 2200 50  0000 C CNN
-F 2 "Resistor_SMD:R_0402_1005Metric" V 6630 2200 50  0001 C CNN
-F 3 "~" H 6700 2200 50  0001 C CNN
-	1    6700 2200
-	0    1    1    0
-$EndComp
-$Comp
-L Device:R R?
-U 1 1 5C644C3D
-P 7000 2350
-AR Path="/5C644C3D" Ref="R?"  Part="1"
-AR Path="/669AB112/5C644C3D" Ref="R46"  Part="1"
-F 0 "R46" V 6900 2350 50  0000 C CNN
-F 1 "100" V 7000 2350 50  0000 C CNN
-F 2 "Resistor_SMD:R_0402_1005Metric" V 6930 2350 50  0001 C CNN
-F 3 "~" H 7000 2350 50  0001 C CNN
-	1    7000 2350
 	0    1    1    0
 $EndComp
@@
 	0    1    1    0
 $EndComp
-Text GLabel 10000 1700 2    39   Input ~ 0
-ADC_GND
-Text GLabel 10000 1600 2    39   Input ~ 0
+Text GLabel 10000 2050 2    39   Input ~ 0
 ADC_VDD
-Text GLabel 10000 1800 2    39   Input ~ 0
+Text GLabel 10000 2250 2    39   Input ~ 0
 ADC_A1+
-Text GLabel 10000 1900 2    39   Input ~ 0
+Text GLabel 10000 2350 2    39   Input ~ 0
 ADC_A1-
 Wire Wire Line
@@
 L Device:C C?
 U 1 1 5D3C0A96
-P 5550 2900
+P 6150 2900
 AR Path="/5D3C0A96" Ref="C?"  Part="1"
 AR Path="/669AB112/5D3C0A96" Ref="C58"  Part="1"
-F 0 "C58" H 5500 2800 50  0000 R CNN
+F 0 "C58" H 6100 2800 50  0000 R CNN
+F 1 "0.1uF" H 6100 3000 50  0000 R CNN
+F 2 "Capacitor_SMD:C_0402_1005Metric" H 6188 2750 50  0001 C CNN
+F 3 "~" H 6150 2900 50  0001 C CNN
+	1    6150 2900
+	-1   0    0    1
+$EndComp
+$Comp
+L Device:C C?
+U 1 1 5D3C0A9D
+P 6450 2900
+AR Path="/5D3C0A9D" Ref="C?"  Part="1"
+AR Path="/669AB112/5D3C0A9D" Ref="C59"  Part="1"
+F 0 "C59" H 6400 2800 50  0000 R CNN
+F 1 "0.1uF" H 6400 3000 50  0000 R CNN
+F 2 "Capacitor_SMD:C_0402_1005Metric" H 6488 2750 50  0001 C CNN
+F 3 "~" H 6450 2900 50  0001 C CNN
+	1    6450 2900
+	-1   0    0    1
+$EndComp
+$Comp
+L Device:C C?
+U 1 1 5D3C0AA4
+P 5550 2900
+AR Path="/5D3C0AA4" Ref="C?"  Part="1"
+AR Path="/669AB112/5D3C0AA4" Ref="C60"  Part="1"
+F 0 "C60" H 5500 2800 50  0000 R CNN
 F 1 "0.1uF" H 5500 3000 50  0000 R CNN
 F 2 "Capacitor_SMD:C_0402_1005Metric" H 5588 2750 50  0001 C CNN
@@
 $Comp
 L Device:C C?
-U 1 1 5D3C0A9D
+U 1 1 5D3C0AAB
 P 5850 2900
-AR Path="/5D3C0A9D" Ref="C?"  Part="1"
-AR Path="/669AB112/5D3C0A9D" Ref="C59"  Part="1"
-F 0 "C59" H 5800 2800 50  0000 R CNN
+AR Path="/5D3C0AAB" Ref="C?"  Part="1"
+AR Path="/669AB112/5D3C0AAB" Ref="C61"  Part="1"
+F 0 "C61" H 5800 2800 50  0000 R CNN
 F 1 "0.1uF" H 5800 3000 50  0000 R CNN
 F 2 "Capacitor_SMD:C_0402_1005Metric" H 5888 2750 50  0001 C CNN
 F 3 "~" H 5850 2900 50  0001 C CNN
 	1    5850 2900
-	-1   0    0    1
-$EndComp
-$Comp
-L Device:C C?
-U 1 1 5D3C0AA4
-P 6150 2900
-AR Path="/5D3C0AA4" Ref="C?"  Part="1"
-AR Path="/669AB112/5D3C0AA4" Ref="C60"  Part="1"
-F 0 "C60" H 6100 2800 50  0000 R CNN
-F 1 "0.1uF" H 6100 3000 50  0000 R CNN
-F 2 "Capacitor_SMD:C_0402_1005Metric" H 6188 2750 50  0001 C CNN
-F 3 "~" H 6150 2900 50  0001 C CNN
-	1    6150 2900
-	-1   0    0    1
-$EndComp
-$Comp
-L Device:C C?
-U 1 1 5D3C0AAB
-P 6450 2900
-AR Path="/5D3C0AAB" Ref="C?"  Part="1"
-AR Path="/669AB112/5D3C0AAB" Ref="C61"  Part="1"
-F 0 "C61" H 6400 2800 50  0000 R CNN
-F 1 "0.1uF" H 6400 3000 50  0000 R CNN
-F 2 "Capacitor_SMD:C_0402_1005Metric" H 6488 2750 50  0001 C CNN
-F 3 "~" H 6450 2900 50  0001 C CNN
-	1    6450 2900
 	-1   0    0    1
 $EndComp
@@
 L Device:C_Small C53
 U 1 1 5C8AAC3C
-P 4550 2300
-F 0 "C53" H 4575 2375 50  0000 L CNN
-F 1 "0.1uF" H 4575 2225 50  0000 L CNN
-F 2 "Capacitor_SMD:C_0402_1005Metric" H 4550 2300 50  0001 C CNN
-F 3 "~" H 4550 2300 50  0001 C CNN
-	1    4550 2300
+P 4550 1950
+F 0 "C53" H 4575 2025 50  0000 L CNN
+F 1 "0.1uF" H 4575 1875 50  0000 L CNN
+F 2 "Capacitor_SMD:C_0402_1005Metric" H 4550 1950 50  0001 C CNN
+F 3 "~" H 4550 1950 50  0001 C CNN
+	1    4550 1950
 	1    0    0    -1
 $EndComp
@@
 L Device:C_Small C52
 U 1 1 5C8AA644
-P 4550 1950
-F 0 "C52" H 4575 2025 50  0000 L CNN
-F 1 "0.1uF" H 4575 1875 50  0000 L CNN
-F 2 "Capacitor_SMD:C_0402_1005Metric" H 4550 1950 50  0001 C CNN
-F 3 "~" H 4550 1950 50  0001 C CNN
-	1    4550 1950
+P 4550 2300
+F 0 "C52" H 4575 2375 50  0000 L CNN
+F 1 "0.1uF" H 4575 2225 50  0000 L CNN
+F 2 "Capacitor_SMD:C_0402_1005Metric" H 4550 2300 50  0001 C CNN
+F 3 "~" H 4550 2300 50  0001 C CNN
+	1    4550 2300
 	1    0    0    -1
 $EndComp
@@
 L Connector:Screw_Terminal_01x04 J6
 U 1 1 5BFAFD9F
-P 10200 2150
-F 0 "J6" H 10279 2142 50  0000 L CNN
-F 1 "DNP" H 10279 2051 50  0000 L CNN
-F 2 "Connector_PinHeader_2.54mm:PinHeader_1x04_P2.54mm_Vertical" H 10200 2150 50  0001 C CNN
-F 3 "~" H 10200 2150 50  0001 C CNN
-	1    10200 2150
+P 10200 1700
+F 0 "J6" H 10279 1692 50  0000 L CNN
+F 1 "DNP" H 10279 1601 50  0000 L CNN
+F 2 "Connector_PinHeader_2.54mm:PinHeader_1x04_P2.54mm_Vertical" H 10200 1700 50  0001 C CNN
+F 3 "~" H 10200 1700 50  0001 C CNN
+	1    10200 1700
 	1    0    0    -1
 $EndComp
@@
 F 3 "" H 9000 5200 50  0001 C CNN
 	1    7950 5200
-	1    0    0    -1
+	-1   0    0    -1
 $EndComp
 Text Notes 3400 5750 0    50   ~ 10
@@
 Wire Wire Line
 	7700 3400 7800 3400
-$Comp
-L Device:C C?
-U 1 1 5C8A4043
-P 9450 3350
-AR Path="/5C8A4043" Ref="C?"  Part="1"
-AR Path="/65B709D0/5C8A4043" Ref="C?"  Part="1"
-AR Path="/66A12230/5C8A4043" Ref="C?"  Part="1"
-AR Path="/669AB112/5C8A4043" Ref="C72"  Part="1"
-F 0 "C72" H 9500 3450 50  0000 L CNN
-F 1 "0.1uF" H 9500 3250 50  0000 L CNN
-F 2 "Capacitor_SMD:C_0402_1005Metric" H 9488 3200 50  0001 C CNN
-F 3 "~" H 9450 3350 50  0001 C CNN
-	1    9450 3350
-	1    0    0    -1
-$EndComp
 Wire Notes Line
 	3600 3900 10450 3900
 Wire Wire Line
 	3750 3100 3900 3100
-$Comp
-L CropTop:AGND #PWR0132
-U 1 1 5C9AC406
-P 9450 3550
-F 0 "#PWR0132" H 9450 3300 50  0001 C CNN
-F 1 "AGND" H 9455 3377 50  0000 C CNN
-F 2 "" H 9450 3550 50  0001 C CNN
-F 3 "" H 9450 3550 50  0001 C CNN
-	1    9450 3550
-	1    0    0    -1
-$EndComp
 Wire Wire Line
 	8700 3400 8800 3400
 Wire Wire Line
 	8800 3400 8800 3300
-$Comp
-L CropTop:AVDD #PWR0131
-U 1 1 5C9F3A68
-P 9450 3150
-F 0 "#PWR0131" H 9450 3000 50  0001 C CNN
-F 1 "AVDD" H 9465 3323 50  0000 C CNN
-F 2 "" H 9450 3150 50  0001 C CNN
-F 3 "" H 9450 3150 50  0001 C CNN
-	1    9450 3150
-	1    0    0    -1
-$EndComp
-Wire Wire Line
-	9450 3550 9450 3500
-Wire Wire Line
-	9450 3200 9450 3150
 $Comp
 L CropTop:PUSBM5V5X4 U?
@@
 Wire Wire Line
 	8800 6200 8900 6200
+Text GLabel 10000 2150 2    39   Input ~ 0
+ADC_GND
 $EndSCHEMATC

Commit message: Finished working board
Parts:
- removed C62: 10uF, Capacitor_SMD:C_0805_2012Metric, symbol Device:C
- removed R48, R49: 10, Resistor_SMD:R_0402_1005Metric, symbol Device:R
- removed TP63, TP67, TP69, TP75: TestPoint_Alt, TestPoint:TestPoint_Pad_D2.0mm, symbol Connector:TestPoint_Alt
Connections:
- net DVDD: no longer U18.6 (VCC)
- net DVDD_UNREG: now also U18.6 (VCC)
- net ROT_Y1: now also U11.3 (Y1)
- net ROT_Y2: now also U11.6 (Y2)

Commit message: Changed testpoint size
Parts:
- TP60, TP61, TP62, TP64, TP65, TP66, TP68, TP70, TP71, TP72, TP73, TP74: footprint TestPoint:TestPoint_Pad_D2.0mm -> TestPoint:TestPoint_Pad_1.0x1.0mm
Changed lines of the file:
@@
 F 0 "TP64" V 1150 3280 50  0000 L CNN
 F 1 "TestPoint_Alt" V 1185 3285 50  0001 L CNN
-F 2 "TestPoint:TestPoint_Pad_D2.0mm" H 1350 3100 50  0001 C CNN
+F 2 "TestPoint:TestPoint_Pad_1.0x1.0mm" H 1350 3100 50  0001 C CNN
 F 3 "~" H 1350 3100 50  0001 C CNN
 	1    1150 3100
@@
 F 0 "TP65" V 1150 3430 50  0000 L CNN
 F 1 "TestPoint_Alt" V 1185 3435 50  0001 L CNN
-F 2 "TestPoint:TestPoint_Pad_D2.0mm" H 1350 3250 50  0001 C CNN
+F 2 "TestPoint:TestPoint_Pad_1.0x1.0mm" H 1350 3250 50  0001 C CNN
 F 3 "~" H 1350 3250 50  0001 C CNN
 	1    1150 3250
@@
 F 0 "TP66" V 1150 3580 50  0000 L CNN
 F 1 "TestPoint_Alt" V 1185 3585 50  0001 L CNN
-F 2 "TestPoint:TestPoint_Pad_D2.0mm" H 1350 3400 50  0001 C CNN
+F 2 "TestPoint:TestPoint_Pad_1.0x1.0mm" H 1350 3400 50  0001 C CNN
 F 3 "~" H 1350 3400 50  0001 C CNN
 	1    1150 3400
@@
 F 0 "TP72" V 5950 1530 50  0000 L CNN
 F 1 "TestPoint_Alt" V 5985 1535 50  0001 L CNN
-F 2 "TestPoint:TestPoint_Pad_D2.0mm" H 6150 1350 50  0001 C CNN
+F 2 "TestPoint:TestPoint_Pad_1.0x1.0mm" H 6150 1350 50  0001 C CNN
 F 3 "~" H 6150 1350 50  0001 C CNN
 	1    5950 1350
@@
 F 0 "TP70" V 5950 1230 50  0000 L CNN
 F 1 "TestPoint_Alt" V 5985 1235 50  0001 L CNN
-F 2 "TestPoint:TestPoint_Pad_D2.0mm" H 6150 1050 50  0001 C CNN
+F 2 "TestPoint:TestPoint_Pad_1.0x1.0mm" H 6150 1050 50  0001 C CNN
 F 3 "~" H 6150 1050 50  0001 C CNN
 	1    5950 1050
@@
 F 0 "TP71" V 5950 1380 50  0000 L CNN
 F 1 "TestPoint_Alt" V 5985 1385 50  0001 L CNN
-F 2 "TestPoint:TestPoint_Pad_D2.0mm" H 6150 1200 50  0001 C CNN
+F 2 "TestPoint:TestPoint_Pad_1.0x1.0mm" H 6150 1200 50  0001 C CNN
 F 3 "~" H 6150 1200 50  0001 C CNN
 	1    5950 1200
@@
 F 0 "TP61" V 1200 5580 50  0000 L CNN
 F 1 "TestPoint_Alt" V 1235 5585 50  0001 L CNN
-F 2 "TestPoint:TestPoint_Pad_D2.0mm" H 1400 5400 50  0001 C CNN
+F 2 "TestPoint:TestPoint_Pad_1.0x1.0mm" H 1400 5400 50  0001 C CNN
 F 3 "~" H 1400 5400 50  0001 C CNN
 	1    1200 5400
@@
 F 0 "TP62" V 1200 5730 50  0000 L CNN
 F 1 "TestPoint_Alt" V 1235 5735 50  0001 L CNN
-F 2 "TestPoint:TestPoint_Pad_D2.0mm" H 1400 5550 50  0001 C CNN
+F 2 "TestPoint:TestPoint_Pad_1.0x1.0mm" H 1400 5550 50  0001 C CNN
 F 3 "~" H 1400 5550 50  0001 C CNN
 	1    1200 5550
@@
 F 0 "TP60" V 1200 5430 50  0000 L CNN
 F 1 "TestPoint_Alt" V 1235 5435 50  0001 L CNN
-F 2 "TestPoint:TestPoint_Pad_D2.0mm" H 1400 5250 50  0001 C CNN
+F 2 "TestPoint:TestPoint_Pad_1.0x1.0mm" H 1400 5250 50  0001 C CNN
 F 3 "~" H 1400 5250 50  0001 C CNN
 	1    1200 5250
@@
 F 0 "TP68" V 8100 6630 50  0000 L CNN
 F 1 "TestPoint_Alt" V 8135 6635 50  0001 L CNN
-F 2 "TestPoint:TestPoint_Pad_D2.0mm" H 8300 6450 50  0001 C CNN
+F 2 "TestPoint:TestPoint_Pad_1.0x1.0mm" H 8300 6450 50  0001 C CNN
 F 3 "~" H 8300 6450 50  0001 C CNN
 	1    8100 6450
@@
 F 0 "TP73" V 7250 6480 50  0000 L CNN
 F 1 "TestPoint_Alt" V 7285 6485 50  0001 L CNN
-F 2 "TestPoint:TestPoint_Pad_D2.0mm" H 7450 6300 50  0001 C CNN
+F 2 "TestPoint:TestPoint_Pad_1.0x1.0mm" H 7450 6300 50  0001 C CNN
 F 3 "~" H 7450 6300 50  0001 C CNN
 	1    7250 6300
@@
 F 0 "TP74" V 7250 6630 50  0000 L CNN
 F 1 "TestPoint_Alt" V 7285 6635 50  0001 L CNN
-F 2 "TestPoint:TestPoint_Pad_D2.0mm" H 7450 6450 50  0001 C CNN
+F 2 "TestPoint:TestPoint_Pad_1.0x1.0mm" H 7450 6450 50  0001 C CNN
 F 3 "~" H 7450 6450 50  0001 C CNN
 	1    7250 6450
@@
 	9650 4850 9900 4850
 $Comp
-L CropTop:DVDD_UNREG #PWR?
+L CropTop:DVDD_UNREG #PWR0113
 U 1 1 5C2F763A
 P 9900 4750
-F 0 "#PWR?" H 9900 4600 50  0001 C CNN
+F 0 "#PWR0113" H 9900 4600 50  0001 C CNN
 F 1 "DVDD_UNREG" H 9915 4923 50  0000 C CNN
 F 2 "" H 9900 4750 50  0001 C CNN
@@
 P 2775 6875
 AR Path="/65B709D0/5C399758" Ref="#PWR?"  Part="1"
-AR Path="/669AB112/5C399758" Ref="#PWR?"  Part="1"
-F 0 "#PWR?" H 2775 6725 50  0001 C CNN
+AR Path="/669AB112/5C399758" Ref="#PWR0115"  Part="1"
+F 0 "#PWR0115" H 2775 6725 50  0001 C CNN
 F 1 "DVDD" H 2790 7048 50  0000 C CNN
 F 2 "" H 2775 6875 50  0001 C CNN

Commit message: Complete PCB version 1
Parts:
- TP60, TP61, TP62, TP64, TP65, TP66, TP68, TP70, TP71, TP72, TP73, TP74: footprint TestPoint:TestPoint_Pad_1.0x1.0mm -> croptop:TestPoint
Changed lines of the file:
@@
 F 0 "TP64" V 1150 3280 50  0000 L CNN
 F 1 "TestPoint_Alt" V 1185 3285 50  0001 L CNN
-F 2 "TestPoint:TestPoint_Pad_1.0x1.0mm" H 1350 3100 50  0001 C CNN
+F 2 "croptop:TestPoint" H 1350 3100 50  0001 C CNN
 F 3 "~" H 1350 3100 50  0001 C CNN
 	1    1150 3100
@@
 F 0 "TP65" V 1150 3430 50  0000 L CNN
 F 1 "TestPoint_Alt" V 1185 3435 50  0001 L CNN
-F 2 "TestPoint:TestPoint_Pad_1.0x1.0mm" H 1350 3250 50  0001 C CNN
+F 2 "croptop:TestPoint" H 1350 3250 50  0001 C CNN
 F 3 "~" H 1350 3250 50  0001 C CNN
 	1    1150 3250
@@
 F 0 "TP66" V 1150 3580 50  0000 L CNN
 F 1 "TestPoint_Alt" V 1185 3585 50  0001 L CNN
-F 2 "TestPoint:TestPoint_Pad_1.0x1.0mm" H 1350 3400 50  0001 C CNN
+F 2 "croptop:TestPoint" H 1350 3400 50  0001 C CNN
 F 3 "~" H 1350 3400 50  0001 C CNN
 	1    1150 3400
@@
 F 0 "TP72" V 5950 1530 50  0000 L CNN
 F 1 "TestPoint_Alt" V 5985 1535 50  0001 L CNN
-F 2 "TestPoint:TestPoint_Pad_1.0x1.0mm" H 6150 1350 50  0001 C CNN
+F 2 "croptop:TestPoint" H 6150 1350 50  0001 C CNN
 F 3 "~" H 6150 1350 50  0001 C CNN
 	1    5950 1350
@@
 F 0 "TP70" V 5950 1230 50  0000 L CNN
 F 1 "TestPoint_Alt" V 5985 1235 50  0001 L CNN
-F 2 "TestPoint:TestPoint_Pad_1.0x1.0mm" H 6150 1050 50  0001 C CNN
+F 2 "croptop:TestPoint" H 6150 1050 50  0001 C CNN
 F 3 "~" H 6150 1050 50  0001 C CNN
 	1    5950 1050
@@
 F 0 "TP71" V 5950 1380 50  0000 L CNN
 F 1 "TestPoint_Alt" V 5985 1385 50  0001 L CNN
-F 2 "TestPoint:TestPoint_Pad_1.0x1.0mm" H 6150 1200 50  0001 C CNN
+F 2 "croptop:TestPoint" H 6150 1200 50  0001 C CNN
 F 3 "~" H 6150 1200 50  0001 C CNN
 	1    5950 1200
@@
 F 0 "TP61" V 1200 5580 50  0000 L CNN
 F 1 "TestPoint_Alt" V 1235 5585 50  0001 L CNN
-F 2 "TestPoint:TestPoint_Pad_1.0x1.0mm" H 1400 5400 50  0001 C CNN
+F 2 "croptop:TestPoint" H 1400 5400 50  0001 C CNN
 F 3 "~" H 1400 5400 50  0001 C CNN
 	1    1200 5400
@@
 F 0 "TP62" V 1200 5730 50  0000 L CNN
 F 1 "TestPoint_Alt" V 1235 5735 50  0001 L CNN
-F 2 "TestPoint:TestPoint_Pad_1.0x1.0mm" H 1400 5550 50  0001 C CNN
+F 2 "croptop:TestPoint" H 1400 5550 50  0001 C CNN
 F 3 "~" H 1400 5550 50  0001 C CNN
 	1    1200 5550
@@
 F 0 "TP60" V 1200 5430 50  0000 L CNN
 F 1 "TestPoint_Alt" V 1235 5435 50  0001 L CNN
-F 2 "TestPoint:TestPoint_Pad_1.0x1.0mm" H 1400 5250 50  0001 C CNN
+F 2 "croptop:TestPoint" H 1400 5250 50  0001 C CNN
 F 3 "~" H 1400 5250 50  0001 C CNN
 	1    1200 5250
@@
 F 0 "TP68" V 8100 6630 50  0000 L CNN
 F 1 "TestPoint_Alt" V 8135 6635 50  0001 L CNN
-F 2 "TestPoint:TestPoint_Pad_1.0x1.0mm" H 8300 6450 50  0001 C CNN
+F 2 "croptop:TestPoint" H 8300 6450 50  0001 C CNN
 F 3 "~" H 8300 6450 50  0001 C CNN
 	1    8100 6450
@@
 F 0 "TP73" V 7250 6480 50  0000 L CNN
 F 1 "TestPoint_Alt" V 7285 6485 50  0001 L CNN
-F 2 "TestPoint:TestPoint_Pad_1.0x1.0mm" H 7450 6300 50  0001 C CNN
+F 2 "croptop:TestPoint" H 7450 6300 50  0001 C CNN
 F 3 "~" H 7450 6300 50  0001 C CNN
 	1    7250 6300
@@
 F 0 "TP74" V 7250 6630 50  0000 L CNN
 F 1 "TestPoint_Alt" V 7285 6635 50  0001 L CNN
-F 2 "TestPoint:TestPoint_Pad_1.0x1.0mm" H 7450 6450 50  0001 C CNN
+F 2 "croptop:TestPoint" H 7450 6450 50  0001 C CNN
 F 3 "~" H 7450 6450 50  0001 C CNN
 	1    7250 6450

Commit message: Adding images
Other:
- note added: "Change nets to have directions\nRemove global nets on power\nAdd missing pullups and pulldowns on temp/memory\nSpace out componentts more, use a bigger board\nConsider 0603 resistors/caps\nCheck regulators can carry high current\nMove far end of\nMove micro usb and lcd connector further forward"
- note added: "List of things to do:\nRemove electrolytic input on DC motor driver\nChange AVDD to 5V0_REG, DVDD to 3V3"
Changed lines of the file:
@@
 	1    0    0    -1
 $EndComp
+Text Notes 11200 2750 0    50   ~ 0
+List of things to do:\nRemove electrolytic input on DC motor driver\nChange AVDD to 5V0_REG, DVDD to 3V3
+Text Notes 11200 3400 0    50   ~ 0
+Change nets to have directions\nRemove global nets on power\nAdd missing pullups and pulldowns on temp/memory\nSpace out componentts more, use a bigger board\nConsider 0603 resistors/caps\nCheck regulators can carry high current\nMove far end of\nMove micro usb and lcd connector further forward
 $EndSCHEMATC

Commit message: Getting example files
Parts:
- added TP?: TestPoint_Alt, croptop:TestPoint, symbol Connector:TestPoint_Alt
Connections:
- net MOSI: now also TP?.1
Changed lines of the file:
@@
 Text Notes 11200 3400 0    50   ~ 0
 Change nets to have directions\nRemove global nets on power\nAdd missing pullups and pulldowns on temp/memory\nSpace out componentts more, use a bigger board\nConsider 0603 resistors/caps\nCheck regulators can carry high current\nMove far end of\nMove micro usb and lcd connector further forward
+Text GLabel 1050 3550 0    39   Input ~ 0
+MOSI
+Wire Wire Line
+	1150 3550 1050 3550
+$Comp
+L Connector:TestPoint_Alt TP?
+U 1 1 5C632DBE
+P 1150 3550
+AR Path="/64809F0C/5C632DBE" Ref="TP?"  Part="1"
+AR Path="/669AB112/5C632DBE" Ref="TP?"  Part="1"
+F 0 "TP?" V 1150 3730 50  0000 L CNN
+F 1 "TestPoint_Alt" V 1185 3735 50  0001 L CNN
+F 2 "croptop:TestPoint" H 1350 3550 50  0001 C CNN
+F 3 "~" H 1350 3550 50  0001 C CNN
+	1    1150 3550
+	0    1    1    0
+$EndComp
 $EndSCHEMATC
