File: PCB 2.0/croptop_io.sch (KiCad schematic (older format))
At the start: 57 parts, among them J5 Terminal Block, J6 DNP, J7 DNP, U10 AD7799, U11 74HCT125D, U17 DT6250-06MR-13, U18 PUSBM5V5X4, U8 74HCT125D, U9 DRV8872

Commit message: Fixed it
Parts:
- removed C43: 10uF, Capacitor_SMD:C_0805_2012Metric, symbol Device:C
- removed C44, C63: 0.1uF, Capacitor_SMD:C_0402_1005Metric, symbol Device:C
- removed C50: 100uF, Capacitor_SMD:CP_Elec_6.3x7.7, symbol Device:CP1
- removed D9: SBRD10200TR, croptop:SizeOfThisLad, symbol Device:D
- removed J5: Terminal Block, TerminalBlock_4Ucon:TerminalBlock_4Ucon_1x15_P3.50mm_Horizontal, symbol Connector:Screw_Terminal_01x15
- removed J6, J7: DNP, Connector_PinHeader_2.54mm:PinHeader_1x04_P2.54mm_Vertical, symbol Connector:Screw_Terminal_01x04
- removed R34, R35: 10, Resistor_SMD:R_0402_1005Metric, symbol Device:R
- removed R50, R51: 0, Resistor_SMD:R_0402_1005Metric, symbol Device:R
- removed TP60, TP61, TP62, TP64, TP65, TP66, TP68, TP70, TP71, TP72, TP73, TP74, TP?: TestPoint_Alt, croptop:TestPoint, symbol Connector:TestPoint_Alt
- removed U11, U8: 74HCT125D, Package_SO:SOIC-14_3.9x8.7mm_P1.27mm, symbol CropTop:74LVC125A
- removed U18: PUSBM5V5X4, croptop:PUSBM5V5X4, symbol CropTop:PUSBM5V5X4
- added C? (x2): 0.1uF, Capacitor_SMD:C_0805_2012Metric, symbol Device:C
- added C?: 0.1uF, Capacitor_SMD:C_0402_1005Metric, symbol Device:C
- added C?: 100uF, Capacitor_SMD:CP_Elec_6.3x7.7, symbol Device:CP1
- added D?: D_Schottky, symbol Device:D_Schottky
- added J?: Rotary Encoder Term. Block, symbol Connector:Screw_Terminal_01x08
- added L?: 10uH, Inductor_SMD:L_1210_3225Metric, symbol Device:L
- added Q?: Q_PMOS_DGS, symbol Device:Q_PMOS_DGS
- added R? (x3): 2K, Resistor_SMD:R_0402_1005Metric, symbol Device:R
- added R? (x4): 0, Resistor_SMD:R_0402_1005Metric, symbol Device:R
- added R? (x4): R, symbol Device:R
- added TP? (x24): TestPoint, symbol Connector:TestPoint
- added U?: A5984, symbol CropTop:A5984
- added U?: 74HCT125D, symbol CropTop:74LVC125
- added U?: DT6250-06MR-13, Package_SO:MSOP-8_3x3mm_P0.65mm, symbol CropTop:DT6250-06MR-13
- added U?: PUSBM5V5X4, croptop:PUSBM5V5X4, symbol CropTop:PUSBM5V5X4
- added U?: 74HCT125D, Package_SO:SOIC-14_3.9x8.7mm_P1.27mm, symbol CropTop:74LVC125A
- R?: renamed from R38; value 100 -> 22
- R?: renamed from R39; value 100 -> 22
- R?: renamed from R40; value 100 -> 22
- R?: renamed from R41; value 100 -> 22
- renumbered C49 to C?, C51 to C?, C46 to C?, C45 to C?, C52 to C?, C53 to C?, C54 to C?, C56 to C?, C57 to C?, C58 to C?, C59 to C?, C60 to C?, C61 to C?, C47 to C?, R42 to R?, R45 to R?, R43 to R?, R46 to R?, R44 to R?, R47 to R?, R37 to R?, R36 to R?, U10 to U?, U17 to U?, U9 to U?
Connections:
- net AGND: now also U?.7 (GND)
- net DGND: now also C?.2, C?.2, J?.4 (Pin_4), J?.8 (Pin_8), R?.2, R?.2, R?.2, R?.2, U?.1 (~OE1), U?.10 (~OE3), U?.13 (GND), U?.13 (~OE4), U?.24 (GND), U?.4 (~OE2), U?.7 (GND), U?.7 (GND), U?.7 (GND), U?.8 (ROSC); no longer U?.7 (ISEN)
- net DRV_FLT: now also R?.2
- net DRV_OUT1: now also TP?.1
- net DRV_OUT2: now also TP?.1
- net LIN_IN: now also U?.1 (IO1)
- net ROT_A1: now also U?.2 (A1), U?.3 (IO3)
- net ROT_A2: now also U?.2 (IO2), U?.5 (A2)
- net ROT_VDD: now also R?.1, R?.2
- net ROT_Y1: now also U?.3 (Y1)
- net ROT_Y2: now also U?.6 (Y2)
- net ADI_A1+: now reaches R?.1, U?.6 (IO3)
- net ADI_A1+: now also TP?.1
- net ADI_A1-: now reaches R?.1, U?.5 (IO2)
- net ADI_A1-: now also TP?.1
- net ADI_A3+: now reaches R?.1, U?.2 (IO2)
- net ADI_A3+: now also TP?.1
- net ADI_A3-: now reaches R?.1, U?.1 (IO1)
- net ADI_A3-: now also TP?.1
- net at C?.1, U?.5 (VM): now also C?.1, C?.1, D?.1 (K), Q?.3 (S), TP?.1, U?.16 (VBB1), U?.21 (VBB2)
- net CS_1: now reaches R?.2
- net SCLK_1: now reaches R?.2
- net MOSI_1: now reaches R?.2
- net MISO_1: now reaches R?.2
- net ADC_A1+ renamed ADI_A2+
- net ADI_A2+: now also TP?.1
- net ADC_A1- renamed ADI_A2-
- net ADI_A2-: now also TP?.1
- net ADC_GND renamed ADI_PSW
- net AVDD: no longer names the net of C?.1, C?.1, U?.13 (AVDD), U?.9 (RENIN(+))
- net AVDD: now also L?.2; no longer U?.8 (VCC)
- net DVDD renamed +3V3
- net +3V3: now also C?.1, R?.1, R?.1, R?.1, R?.1, R?.1, TP?.1, U?.12 (REF), U?.14 (VCC), U?.14 (VCC)
- new net: C?.1, U?.1 (CP1)
- new net: R?.1, U?.17 (SENSE1)
- new net: C?.2, U?.2 (CP2)
- new net: R?.1, U?.20 (SENSE2)
- new net: C?.2, TP?.1, U?.3 (VCP)
- new net: R?.1, U?.7 (ISEN)
- new net: J?.7 (Pin_7), U?.11 (Y4)
- new net: J?.2 (Pin_2), U?.3 (Y1)
- new net: J?.3 (Pin_3), U?.6 (Y2)
- new net: J?.6 (Pin_6), U?.8 (Y3)
- new net: J?.1 (Pin_1), J?.5 (Pin_5), R?.1, R?.2
- new net: D?.2 (A), Q?.2 (G), R?.1
- new net +5V: R?.2, R?.2, U?.6 (VCC)
- new net +5V_REG: L?.1, U?.8 (VCC)
- new net AUX_BATTERY: Q?.1 (D)
- new net INPUT_CAP_1: U?.2 (A1)
- new net INPUT_CAP_2: U?.5 (A2)
- new net INPUT_CAP_3: U?.9 (A3)
- new net INPUT_CAP_4: U?.12 (A4)
- new net STEP_DIR: TP?.1, U?.14 (DIR)
- new net STEP_FAULT: R?.2, TP?.1, U?.4 (nFAULT)
- new net STEP_MS1: TP?.1, U?.5 (MS1)
- new net STEP_MS2: TP?.1, U?.6 (MS2)
- new net STEP_MS3: TP?.1, U?.10 (MS3)
- new net STEP_OUT1A: TP?.1, U?.18 (OUT1A)
- new net STEP_OUT1B: TP?.1, U?.15 (OUT1B)
- new net STEP_OUT2A: TP?.1, U?.19 (OUT2A)
- new net STEP_OUT2B: TP?.1, U?.22 (OUT2B)
- new net STEP_STEP: TP?.1, U?.11 (STEP)
- new net ~STEP_ENABLE: TP?.1, U?.23 (~ENABLE)
- new net ~STEP_RESET: TP?.1, U?.7 (~RESET)
- new net ~STEP_SLEEP: R?.2, TP?.1, U?.9 (~SLEEP)
- no-connect marks 6 -> 10
Other:
- note added: "Check pinout of PMOS"
- note added: "DC Motor & Stepper Motor Drivers"
- note added: "I think I can\njust tie this\nto 3v3?"
- note added: "Rotary Encoder Interface"
- note removed: "12V"
- note removed: "3V3"
- note removed: "50V"
- note removed: "5V"
- note removed: "A"
- note removed: "A1+"
- note removed: "A1-"
- note removed: "B"
- note removed: "BAT"
- note removed: "GND"
- note removed: "IN"
- note removed: "Linear Actuator Interface w/ DC Motor Driver"
- note removed: "Load Cell"
- note removed: "Motor"
- note removed: "O1"
- note removed: "O2\n"
- note removed: "POT"
- note removed: "Peripheral Terminal Block"
- note removed: "Rot Encoder"
- moved on the sheet: C?, R?, U?
