File: PCB 2.0/croptop_lcd.sch (KiCad schematic (older format))
At the start: 79 parts, among them J4 4-1734839-0, U6 FT812Q, Y2 12MHz

Commit message: Fixed it
Parts:
- removed R10, R11, R12, R13, R14, R15, R16, R17, R18, R19, R20, R21, R22, R23, R29, R30, R31, R32, R33, R5, R6, R7, R73, R74, R75, R76, R77, R8, R9: 22, Resistor_SMD:R_0402_1005Metric, symbol Device:R_Small
- removed TP10, TP11, TP12, TP13, TP14, TP15, TP16, TP17, TP18, TP19, TP20, TP21, TP22, TP23, TP24, TP25, TP26, TP27, TP28, TP29, TP30, TP31, TP32, TP33, TP34, TP35, TP36, TP37, TP38, TP39, TP40, TP41, TP42, TP43, TP44, TP45, TP46, TP8, TP9: TestPoint_Alt, croptop:TestPoint, symbol Connector:TestPoint_Alt
- added R?: 4.7k, symbol Device:R
- added R? (x29): 22, symbol Device:R
- added TP? (x33): TestPoint, symbol Connector:TestPoint
- renumbered C37 to C?, C39 to C?, C40 to C?, C38 to C?, C34 to C?, C35 to C?, C36 to C?, C33 to C?, J4 to J?, U6 to U?, Y2 to Y?
Connections:
- net LCD_INT: now also R?.2
- net at J?.10 (R5): now also R?.1
- net at J?.11 (R6): now also R?.1
- net at J?.12 (R7): now also R?.1
- net at J?.13 (G0): now also R?.1
- net at J?.14 (G1): now also R?.1
- net at J?.15 (G2): now also R?.1
- net at J?.16 (G3): now also R?.1
- net at J?.17 (G4): now also R?.1
- net at J?.18 (G5): now also R?.1
- net at J?.19 (G6): now also R?.1
- net at J?.20 (G7): now also R?.1
- net at J?.21 (B0): now also R?.1
- net at J?.22 (B1): now also R?.1, TP?.1
- net at J?.23 (B2): now also R?.1, TP?.1
- net at J?.24 (B3): now also R?.1, TP?.1
- net at J?.25 (B4): now also R?.1, TP?.1
- net at J?.26 (B5): now also R?.1, TP?.1
- net at J?.27 (B6): now also R?.1, TP?.1
- net at J?.28 (B7): now also R?.1, TP?.1
- net at J?.30 (CLK): now also R?.1, TP?.1
- net at J?.31 (DISP): now also R?.1, TP?.1
- net at J?.32 (HSYNC): now also R?.1, TP?.1
- net at J?.33 (VSYNC): now also R?.1, TP?.1
- net at J?.34 (DE): now also R?.1, TP?.1
- net at J?.5 (R0): now also R?.1
- net at J?.6 (R1): now also R?.1
- net at J?.7 (R2): now also R?.1
- net at J?.8 (R3): now also R?.1
- net at J?.9 (R4): now also R?.1
- net DVDD renamed +3V3
- net +3V3: now also R?.1
- net LCD_ANODE renamed LCD_A
- net LCD_B0: no longer names the net of U?.41 (B0)
- net LCD_B0: now also R?.2, TP?.1
- net LCD_B1: no longer names the net of U?.40 (B1)
- net LCD_B1: now also R?.2
- net LCD_B2: no longer names the net of U?.39 (B2)
- net LCD_B2: now also R?.2
- net LCD_B3: no longer names the net of U?.38 (B3)
- net LCD_B3: now also R?.2
- net LCD_B4: no longer names the net of U?.37 (B4)
- net LCD_B4: now also R?.2
- net LCD_B5: no longer names the net of U?.36 (B5)
- net LCD_B5: now also R?.2
- net LCD_B6: no longer names the net of U?.35 (B6)
- net LCD_B6: now also R?.2
- net LCD_B7: no longer names the net of U?.34 (B7)
- net LCD_B7: now also R?.2
- net LCD_CATHODE renamed LCD_K
- net LCD_DEN: no longer names the net of U?.29 (DE)
- net LCD_DEN: now also R?.2
- net LCD_DISP: no longer names the net of U?.32 (DISP)
- net LCD_DISP: now also R?.2
- net LCD_G0: no longer names the net of U?.50 (G0)
- net LCD_G0: now also R?.2, TP?.1
- net LCD_G1: no longer names the net of U?.49 (G1)
- net LCD_G1: now also R?.2, TP?.1
- net LCD_G2: no longer names the net of U?.48 (G2)
- net LCD_G2: now also R?.2, TP?.1
- net LCD_G3: no longer names the net of U?.47 (G3)
- net LCD_G3: now also R?.2, TP?.1
- net LCD_G4: no longer names the net of U?.46 (G4)
- net LCD_G4: now also R?.2, TP?.1
- net LCD_G5: no longer names the net of U?.45 (G5)
- net LCD_G5: now also R?.2, TP?.1
- net LCD_G6: no longer names the net of U?.44 (G6)
- net LCD_G6: now also R?.2, TP?.1
- net LCD_G7: no longer names the net of U?.43 (G7)
- net LCD_G7: now also R?.2, TP?.1
- net LCD_HSYNC: no longer names the net of U?.31 (HSYNC)
- net LCD_HSYNC: now also R?.2
- net LCD_R0: no longer names the net of U?.2 (R0)
- net LCD_R0: now also R?.2, TP?.1
- net LCD_R1: no longer names the net of U?.1 (R1)
- net LCD_R1: now also R?.2, TP?.1
- net LCD_R2: no longer names the net of U?.56 (R2)
- net LCD_R2: now also R?.2, TP?.1
- net LCD_R3: no longer names the net of U?.55 (R3)
- net LCD_R3: now also R?.2, TP?.1
- net LCD_R4: no longer names the net of U?.54 (R4)
- net LCD_R4: now also R?.2, TP?.1
- net LCD_R5: no longer names the net of U?.53 (R5)
- net LCD_R5: now also R?.2, TP?.1
- net LCD_R6: no longer names the net of U?.52 (R6)
- net LCD_R6: now also R?.2, TP?.1
- net LCD_R7: no longer names the net of U?.51 (R7)
- net LCD_R7: now also R?.2, TP?.1
- net LCD_SHIFT: no longer names the net of U?.33 (PCLK)
- net LCD_SHIFT: now also R?.2
- net LCD_VSYNC: no longer names the net of U?.30 (VSYNC)
- net LCD_VSYNC: now also R?.2
- net SCLK2: no longer names the net of U?.5 (SCK)
- net SDIO2: no longer names the net of U?.6 (MISO/IO1)
- net SDO2: no longer names the net of U?.7 (MOSI/IO0)
- net SS2: no longer names the net of U?.8 (CS_N)
- net TCH_DOWN: no longer names the net of J?.38 (YD), U?.26 (Y-)
- net TCH_DOWN: now also TP?.1
- net TCH_LEFT: no longer names the net of J?.39 (XL), U?.25 (X-)
- net TCH_LEFT: now also TP?.1
- net TCH_RIGHT: no longer names the net of J?.37 (XR), U?.23 (X+)
- net TCH_RIGHT: now also TP?.1
- net TCH_UP: no longer names the net of J?.40 (YU), U?.24 (Y+)
- net TCH_UP: now also TP?.1
Other:
- moved on the sheet: C?, J?, U?, Y?
