File: PCB 2.0/croptop_mcu.sch (KiCad schematic (older format))
At the start: 32 parts, among them J1 PICKit Header, J2 USB_A, U1 PIC32MX795F512L, U16 PUSBM5V5X4, Y1 CXO

Commit message: Fixed it
Parts:
- removed C17: 10uF, Capacitor_SMD:C_0805_2012Metric, symbol Device:C
- removed J1: PICKit Header, Connector_PinHeader_2.54mm:PinHeader_1x06_P2.54mm_Vertical, symbol Connector:Conn_01x06_Male
- removed J2: USB_A, croptop:USB_A_Assmann_Horizontal, symbol Connector:USB_A
- removed U16: PUSBM5V5X4, croptop:PUSBM5V5X4, symbol CropTop:PUSBM5V5X4
- added C? (x2): 10uF, Capacitor_SMD:C_0805_2012Metric, symbol Device:C
- added C? (x2): 26pF, Capacitor_SMD:C_0402_1005Metric, symbol Device:C
- added C?: 0.1uF, Capacitor_SMD:C_0402_1005Metric, symbol Device:C
- added C?: 10uF, symbol Device:C
- added J?: 5V USB, croptop:USB_Micro-B_Molex_47346-0001, symbol Connector:USB_B_Micro
- added J? (x2): USB_A, croptop:USB_A_Assmann_Horizontal, symbol Connector:USB_A
- added J?: PICKit3 Header, symbol Connector_Generic:Conn_01x06
- added L?: 10uH, symbol Device:L
- added U? (x2): PIC32MX795F512L-80I_PT_0, digikey-footprints:TQFP-100_12x12mm, symbol CropTop:PIC32MX795F512L-80I_PT_0
- added U? (x2): PUSBM5V5X4, croptop:PUSBM5V5X4, symbol CropTop:PUSBM5V5X4
- added Y?: CXO, croptop:ABLS_OX, symbol Device:Crystal
- renumbered C3 to C?, C13 to C?, C12 to C?, C11 to C?, C10 to C?, C9 to C?, C8 to C?, C7 to C?, C5 to C?, C2 to C?, C4 to C?, C6 to C?, C1 to C?, FID1 to FID?, FID2 to FID?, H1 to H?, H3 to H?, H2 to H?, H4 to H?, L1 to L?, R70 to R?, R25 to R?, R24 to R?, R1 to R?, R27 to R?, R26 to R?, U1 to U?, Y1 to Y?
Connections:
- net DVDD_UNREG is gone; now on net +3V3: U?.54 (VBUS)
- net DGND: now also C?.1, C?.2, C?.2, C?.2, C?.2, C?.2, J?.3 (Pin_3), J?.4 (GND), J?.4 (GND), J?.5 (GND), J?.5 (Shield), J?.5 (Shield), J?.6 (Shield), U?.15 (VSS), U?.31 (AVSS), U?.36 (VSS), U?.45 (VSS), U?.65 (VSS), U?.7 (GND), U?.7 (GND), U?.75 (VSS)
- net PKT_MCLR: now also J?.1 (Pin_1)
- net PKT_PGEC: now also J?.5 (Pin_5)
- net PKT_PGED: now also J?.4 (Pin_4)
- net USB_D+: now also J?.3 (D+), J?.3 (D+), U?.1 (IO1), U?.1 (IO1)
- net USB_D-: now also J?.2 (D-), J?.2 (D-), U?.2 (IO2), U?.2 (IO2)
- net DVDD renamed +3V3
- net +3V3: now also C?.1, J?.2 (Pin_2), L?.1, U?.16 (VDD), U?.2 (VDD), U?.37 (VDD), U?.46 (VDD), U?.54 (VBUS), U?.55 (VUSB3V3), U?.62 (VDD), U?.86 (VDD)
- new net: C?.1, U?.63 (OSC1), Y?.1
- new net: C?.1, U?.64 (OSC2), Y?.2
- new net: L?.2, U?.30 (AVDD)
- new net: C?.2, U?.85 (VCAP/VDDCORE)
- new net +5V: C?.1, C?.1, J?.1 (VBUS), J?.1 (VBUS), U?.6 (VCC), U?.6 (VCC)
- no-connect marks 53 -> 61
Other:
- note added: "Address = 0101100b"
- note added: "Peripheral USB Ports"
- note removed: "Peripheral USB Port"
- moved on the sheet: C?, FID?, H?, L?, R?, U?, Y?
