File: PCB 2.0/croptop_onboard.sch (KiCad schematic (older format))
At the start: 34 parts, among them SW1 BTNA, SW2 BTNA, U12 Si7006-A20, U13 UCAM-M8Q, U14 W25N01GV, U15 LIS3DH

Commit message: Fixed it
Parts:
- removed SW2: BTNA, Button_Switch_SMD:SW_SPST_PTS645, symbol CropTop:SW_Push
- removed TP100, TP91, TP92, TP99: TestPoint_Alt, croptop:TestPoint, symbol Connector:TestPoint_Alt
- added D?: LED, LED_SMD:LED_0805_2012Metric, symbol Device:LED
- added R? (x2): 10k, Resistor_SMD:R_0402_1005Metric, symbol Device:R
- added R?: 60, Resistor_SMD:R_0402_1005Metric, symbol Device:R
- added SW? (x2): BTN, Button_Switch_SMD:SW_SPST_PTS645, symbol CropTop:SW_Push
- D?: renamed from D24; value LED2 -> LED
- D?: renamed from D25; value LED1 -> LED
- SW?: renamed from SW1; value BTNA -> BTN
- renumbered C68 to C?, C71 to C?, C65 to C?, C69 to C?, R55 to R?, R54 to R?, R62 to R?, R63 to R?, R57 to R?, R56 to R?, R67 to R?, R66 to R?, R52 to R?, R53 to R?, TP82 to TP?, TP83 to TP?, TP89 to TP?, TP90 to TP?, TP88 to TP?, TP78 to TP?, TP85 to TP?, TP86 to TP?, U13 to U?, U15 to U?, U12 to U?, U14 to U?
Connections:
- net DGND: now also R?.1, R?.2
- net at R?.1, R?.2: now also SW?.1
- net BTN_A renamed BTN_1
- net BTN_B renamed BTN_2
- net DVDD renamed +3V3
- net +3V3: now also SW?.2, SW?.2
- net LED_A renamed LED_2
- net LED_B renamed LED_3
- new net: R?.1, R?.2, SW?.1
- new net: D?.1 (K), R?.2
- new net BTN_3: R?.1
- new net LED_1: D?.2 (A)
Other:
- moved on the sheet: D?, R?, SW?
