File: pcb2/croptop_conn.sch (KiCad schematic (older format))
At the start: 3 parts

Commit message: Schematic near completion
Parts:
- removed C?: 10uF, Capacitor_SMD:C_0805_2012Metric, symbol Device:C
- removed J?: ADI Terminal, symbol Connector:Screw_Terminal_01x12
- removed J?: Terminal Block, TerminalBlock_4Ucon:TerminalBlock_4Ucon_1x15_P3.50mm_Horizontal, symbol Connector:Screw_Terminal_01x15
Connections:
- net labels removed: +3V3, +5V_REG, ADC_A1+, ADC_A1-, ADC_GND, ADC_VDD, ADI_A1+, ADI_A1-, ADI_A2+, ADI_A2-, ADI_A3+, ADI_A3-, ADI_PSW, AGND, AUX_BATTERY, DRV_BAT, DRV_GND, DRV_OUT1, DRV_OUT2, LIN_GND, LIN_IN, ROT_A1, ROT_A2, ROT_GND, ROT_VDD
- wire segments 20 -> 0
Other:
- note removed: "12V"
- note removed: "3V3"
- note removed: "5V"
- note removed: "A"
- note removed: "A1+"
- note removed: "A1-"
- note removed: "B"
- note removed: "BAT"
- note removed: "GND"
- note removed: "IN"
- note removed: "Load Cell"
- note removed: "Motor"
- note removed: "O1"
- note removed: "O2\n"
- note removed: "POT"
- note removed: "Rot Encoder"
