File: pcb2/croptop_io.sch (KiCad schematic (older format))
At the start: 159 parts, among them J10 39357-0004, J11 39357-0015, J12 39357-0008, J8 39357-0004, J9 39357-0004, Q3 FDMA530PZ, U21 AP22802AW5, U22 74HCT125D, U23 AP22802AW5, U24 AD7799, U25 TPD4E1U06, U26 AP22802AW5, U27 TPD4E1U06, U28 TPD4E1U06, U29 TPD4E1U06, U30 DRV8872, U31 DRV8825, U32 AP22802AW5

Commit message: Final Schematic
Connections:
- net ADI_5V_FLG renamed ADI_5V_FAULT
- net ENCODE_PWR_FLG renamed ENCODE_PWR_FAULT
- net POTEN_PWR_FLG renamed POTEN_PWR_FAULT
- net SONIC_PWR_FLG renamed SONIC_PWR_FAULT
Other:
- moved on the sheet: R91, R92
Changed lines of the file:
@@
 Wire Wire Line
 	3150 3350 3150 3400
-Text GLabel 10150 2400 2    39   Input ~ 0
+Text GLabel 10150 2400 2    33   Input ~ 0
 ADI_A1-
-Text GLabel 10150 2250 2    39   Input ~ 0
+Text GLabel 10150 2250 2    33   Input ~ 0
 ADI_A1+
-Text GLabel 3300 3400 2    39   Input ~ 0
+Text GLabel 3300 3400 2    33   Input ~ 0
 ADI_PSW
 Wire Wire Line
@@
 	8800 2850 9450 2850
 Connection ~ 8900 2700
-Text GLabel 10150 2700 2    39   Input ~ 0
+Text GLabel 10150 2700 2    33   Input ~ 0
 ADI_A2-
-Text GLabel 10150 2550 2    39   Input ~ 0
+Text GLabel 10150 2550 2    33   Input ~ 0
 ADI_A2+
-Text GLabel 10150 3000 2    39   Input ~ 0
+Text GLabel 10150 3000 2    33   Input ~ 0
 ADI_A3-
-Text GLabel 10150 2850 2    39   Input ~ 0
+Text GLabel 10150 2850 2    33   Input ~ 0
 ADI_A3+
 $Comp
@@
 L power:+3V3 #PWR?
 U 1 1 5C762ECA
-P 8900 8200
+P 9000 8200
 AR Path="/64807BBC/5C762ECA" Ref="#PWR?"  Part="1"
 AR Path="/669AB112/5C762ECA" Ref="#PWR0172"  Part="1"
 AR Path="/5EC973C3/5C762ECA" Ref="#PWR?"  Part="1"
-F 0 "#PWR0172" H 8900 8050 50  0001 C CNN
-F 1 "+3V3" H 8915 8373 50  0000 C CNN
-F 2 "" H 8900 8200 50  0001 C CNN
-F 3 "" H 8900 8200 50  0001 C CNN
-	1    8900 8200
+F 0 "#PWR0172" H 9000 8050 50  0001 C CNN
+F 1 "+3V3" H 9015 8373 50  0000 C CNN
+F 2 "" H 9000 8200 50  0001 C CNN
+F 3 "" H 9000 8200 50  0001 C CNN
+	1    9000 8200
 	1    0    0    -1
 $EndComp
 Wire Wire Line
-	8900 8200 8900 8250
+	9000 8200 9000 8250
 $Comp
 L Device:C C?
@@
 	0    -1   -1   0
 $EndComp
-Text GLabel 8450 8800 0    39   Output ~ 0
+Text GLabel 8550 8750 0    33   Output ~ 0
 ~STEP_HOME
 Wire Wire Line
@@
 L power:+3V3 #PWR?
 U 1 1 5C9E2DB0
-P 8550 8200
+P 8650 8200
 AR Path="/64807BBC/5C9E2DB0" Ref="#PWR?"  Part="1"
 AR Path="/669AB112/5C9E2DB0" Ref="#PWR0170"  Part="1"
 AR Path="/5EC973C3/5C9E2DB0" Ref="#PWR?"  Part="1"
-F 0 "#PWR0170" H 8550 8050 50  0001 C CNN
-F 1 "+3V3" H 8565 8373 50  0000 C CNN
-F 2 "" H 8550 8200 50  0001 C CNN
-F 3 "" H 8550 8200 50  0001 C CNN
-	1    8550 8200
+F 0 "#PWR0170" H 8650 8050 50  0001 C CNN
+F 1 "+3V3" H 8665 8373 50  0000 C CNN
+F 2 "" H 8650 8200 50  0001 C CNN
+F 3 "" H 8650 8200 50  0001 C CNN
+	1    8650 8200
 	1    0    0    -1
 $EndComp
 Wire Wire Line
-	8550 8200 8550 8250
+	8650 8200 8650 8250
 $Comp
 L Connector:TestPoint TP103
@@
 	11150 8950 11200 8950
 Wire Wire Line
-	8900 8550 8900 8650
+	9000 8550 9000 8650
 Wire Wire Line
 	12350 6350 12600 6350
@@
 Wire Wire Line
 	2250 8350 2250 8250
-Text GLabel 1000 9200 0    39   Output ~ 0
+Text GLabel 1000 9200 0    33   Output ~ 0
 ROTARY_1A
 $Comp
@@
 Wire Wire Line
 	2450 9850 2450 9950
-Text GLabel 1000 9300 0    39   Output ~ 0
+Text GLabel 1000 9300 0    33   Output ~ 0
 ROTARY_1B
 $Comp
@@
 $EndComp
 Wire Wire Line
-	8550 8550 8550 8800
+	8650 8550 8650 8750
 $Comp
 L Device:R R?
@@
 L Device:R R?
 U 1 1 5DB66B95
-P 8550 8400
+P 8650 8400
 AR Path="/64809F0C/5DB66B95" Ref="R?"  Part="1"
 AR Path="/66A12230/5DB66B95" Ref="R?"  Part="1"
 AR Path="/669AB112/5DB66B95" Ref="R91"  Part="1"
-F 0 "R91" H 8620 8446 50  0000 L CNN
-F 1 "10k" H 8620 8355 50  0000 L CNN
-F 2 "Resistor_SMD:R_0402_1005Metric" V 8480 8400 50  0001 C CNN
-F 3 "" H 8550 8400 50  0001 C CNN
-	1    8550 8400
+F 0 "R91" H 8720 8446 50  0000 L CNN
+F 1 "10k" H 8720 8355 50  0000 L CNN
+F 2 "Resistor_SMD:R_0402_1005Metric" V 8580 8400 50  0001 C CNN
+F 3 "" H 8650 8400 50  0001 C CNN
+	1    8650 8400
 	1    0    0    -1
 $EndComp
@@
 L Device:R R?
 U 1 1 5DB66C61
-P 8900 8400
+P 9000 8400
 AR Path="/64809F0C/5DB66C61" Ref="R?"  Part="1"
 AR Path="/66A12230/5DB66C61" Ref="R?"  Part="1"
 AR Path="/669AB112/5DB66C61" Ref="R92"  Part="1"
-F 0 "R92" H 8970 8446 50  0000 L CNN
-F 1 "10k" H 8970 8355 50  0000 L CNN
-F 2 "Resistor_SMD:R_0402_1005Metric" V 8830 8400 50  0001 C CNN
-F 3 "" H 8900 8400 50  0001 C CNN
-	1    8900 8400
+F 0 "R92" H 9070 8446 50  0000 L CNN
+F 1 "10k" H 9070 8355 50  0000 L CNN
+F 2 "Resistor_SMD:R_0402_1005Metric" V 8930 8400 50  0001 C CNN
+F 3 "" H 9000 8400 50  0001 C CNN
+	1    9000 8400
 	1    0    0    -1
 $EndComp
@@
 Wire Wire Line
 	2000 1050 2100 1050
-Text GLabel 1450 2450 0    39   Input ~ 0
+Text GLabel 1450 2450 0    33   Input ~ 0
 ADI_MOSI
-Text GLabel 1450 2150 0    39   Input ~ 0
+Text GLabel 1450 2150 0    33   Input ~ 0
 ADI_SCLK
-Text GLabel 1450 2750 0    39   Output ~ 0
+Text GLabel 1450 2750 0    33   Output ~ 0
 ADI_MISO
-Text GLabel 1450 3050 0    39   Input ~ 0
+Text GLabel 1450 3050 0    33   Input ~ 0
 ~ADI_CS
-Text GLabel 14950 2300 0    39   Output ~ 0
+Text GLabel 14950 2300 0    33   Output ~ 0
 ADI_A1-
-Text GLabel 14950 2200 0    39   Output ~ 0
+Text GLabel 14950 2200 0    33   Output ~ 0
 ADI_A1+
-Text GLabel 14950 2800 0    39   Output ~ 0
+Text GLabel 14950 2800 0    33   Output ~ 0
 ADI_A2-
-Text GLabel 14950 2700 0    39   Output ~ 0
+Text GLabel 14950 2700 0    33   Output ~ 0
 ADI_A2+
-Text GLabel 14950 3300 0    39   Output ~ 0
+Text GLabel 14950 3300 0    33   Output ~ 0
 ADI_A3-
-Text GLabel 14950 3200 0    39   Output ~ 0
+Text GLabel 14950 3200 0    33   Output ~ 0
 ADI_A3+
 $Comp
@@
 	1    0    0    -1
 $EndComp
-Text GLabel 9550 4950 0    39   Input ~ 0
+Text GLabel 9550 4950 0    33   Input ~ 0
 DC_PWM_1
-Text GLabel 9700 6100 0    39   Output ~ 0
+Text GLabel 9700 6100 0    33   Output ~ 0
 ~DC_FAULT
-Text GLabel 9550 5250 0    39   Input ~ 0
+Text GLabel 9550 5250 0    33   Input ~ 0
 DC_PWM_2
 $Comp
@@
 Wire Wire Line
 	11100 1400 11100 1500
-Text GLabel 11000 1900 0    39   Output ~ 0
-ADI_5V_FLG
+Text GLabel 11000 1900 0    33   Output ~ 0
+ADI_5V_FAULT
 Wire Wire Line
 	10950 2000 10950 2150
@@
 Wire Wire Line
 	13650 2450 13650 2600
-Text GLabel 5050 5050 0    39   Output ~ 0
+Text GLabel 5050 5050 0    33   Output ~ 0
 POTEN_1
-Text GLabel 5050 5400 0    39   Output ~ 0
+Text GLabel 5050 5400 0    33   Output ~ 0
 POTEN_2
 $Comp
@@
 Wire Wire Line
 	3750 8050 3750 8150
-Text GLabel 3650 8550 0    39   Output ~ 0
-ENCODE_PWR_FLG
+Text GLabel 3650 8550 0    33   Output ~ 0
+ENCODE_PWR_FAULT
 Wire Wire Line
 	3650 8650 3650 8800
@@
 Wire Wire Line
 	1600 4200 1600 4300
-Text GLabel 1500 4700 0    39   Output ~ 0
-POTEN_PWR_FLG
+Text GLabel 1500 4700 0    33   Output ~ 0
+POTEN_PWR_FAULT
 Wire Wire Line
 	1500 4800 1500 4950
@@
 F 1 "DRV8825" H 11400 8700 50  0000 C CNN
 F 2 "" H 11150 8550 50  0001 C CNN
-F 3 "" H 11150 8550 50  0001 C CNN
+F 3 "http://www.ti.com/lit/ds/symlink/drv8825.pdf" H 11150 8550 50  0001 C CNN
 	1    11150 8050
 	1    0    0    -1
 $EndComp
-Text GLabel 9600 7950 0    39   Input ~ 0
+Text GLabel 9600 7950 0    33   Input ~ 0
 STEP_MODE2
-Text GLabel 9600 7850 0    39   Input ~ 0
+Text GLabel 9600 7850 0    33   Input ~ 0
 STEP_MODE1
-Text GLabel 9600 7750 0    39   Input ~ 0
+Text GLabel 9600 7750 0    33   Input ~ 0
 STEP_MODE0
-Text GLabel 9600 7650 0    39   Input ~ 0
+Text GLabel 9600 7650 0    33   Input ~ 0
 STEP_STEP
-Text GLabel 9600 7550 0    39   Input ~ 0
+Text GLabel 9600 7550 0    33   Input ~ 0
 ~STEP_ENBL
-Text GLabel 9600 8150 0    39   Input ~ 0
+Text GLabel 9600 8150 0    33   Input ~ 0
 STEP_DECAY
-Text GLabel 8450 8650 0    39   Output ~ 0
+Text GLabel 8550 8650 0    33   Output ~ 0
 ~STEP_FAULT
-Text GLabel 9600 8300 0    39   Input ~ 0
+Text GLabel 9600 8350 0    33   Input ~ 0
 ~STEP_SLEEP
-Text GLabel 9600 8500 0    39   Input ~ 0
+Text GLabel 9600 8450 0    33   Input ~ 0
 ~STEP_RESET
-Text GLabel 9600 8050 0    39   Input ~ 0
+Text GLabel 9600 8050 0    33   Input ~ 0
 STEP_DIR
 $Comp
@@
 $EndComp
 Wire Wire Line
-	9600 8500 9800 8500
-Wire Wire Line
-	9800 8500 9800 8450
-Wire Wire Line
 	10200 8650 10200 8550
 Wire Wire Line
 	10200 8550 10600 8550
 Wire Wire Line
-	10400 8800 10400 8650
+	10400 8750 10400 8650
 Wire Wire Line
 	10400 8650 10600 8650
@@
 	9900 8450 9900 9050
 Wire Wire Line
-	9500 9050 9500 8800
+	9500 9050 9500 8750
 Wire Wire Line
 	5050 5400 5200 5400
@@
 Wire Wire Line
 	3050 9650 3400 9650
-Text GLabel 5750 6900 0    39   Output ~ 0
+Text GLabel 5750 6900 0    33   Output ~ 0
 SONIC_TRIG
-Text GLabel 5750 7250 0    39   Output ~ 0
+Text GLabel 5750 7250 0    33   Output ~ 0
 SONIC_ECHO
 $Comp
@@
 Wire Wire Line
 	2200 6050 2200 6150
-Text GLabel 2100 6550 0    39   Output ~ 0
-SONIC_PWR_FLG
+Text GLabel 2100 6550 0    33   Output ~ 0
+SONIC_PWR_FAULT
 Wire Wire Line
 	2100 6650 2100 6800
@@
 Wire Wire Line
 	9900 8450 10600 8450
+Connection ~ 9500 8750
 Wire Wire Line
-	9800 8450 9900 8450
-Connection ~ 9500 8800
-Wire Wire Line
-	9500 8800 10400 8800
-Wire Wire Line
-	9800 8350 9800 8300
-Wire Wire Line
-	9800 8300 9600 8300
-Wire Wire Line
-	9800 8350 10100 8350
+	9500 8750 10400 8750
 Connection ~ 10100 8350
 Wire Wire Line
@@
 Wire Wire Line
 	9700 8650 10200 8650
-Connection ~ 8550 8800
 Wire Wire Line
-	8550 8800 9500 8800
-Connection ~ 8900 8650
+	9600 8450 9900 8450
+Wire Wire Line
+	9600 8350 10100 8350
+Connection ~ 8650 8750
+Wire Wire Line
+	8650 8750 9500 8750
+Connection ~ 9000 8650
 Wire Wire Line
-	8900 8650 9700 8650
+	9000 8650 9700 8650
 Wire Wire Line
-	8450 8800 8550 8800
+	8550 8750 8650 8750
 Wire Wire Line
-	8450 8650 8900 8650
+	8550 8650 9000 8650
 $EndSCHEMATC

Commit message: Schematic Done
Parts:
- removed J11: 39357-0015, symbol Connector:Screw_Terminal_01x15
- removed J12: 39357-0008, symbol Connector:Screw_Terminal_01x08
- added J11, J12, J13, J14, J7: 1702474, symbol Connector:Screw_Terminal_01x04
- C45, C46, C51, C52, C56, C58, C66, C74: value 10uF -> 10u
- C47: renamed from C48; value 10uF -> 10u
- C48: renamed from C47; value 10uF -> 10u
- C49, C50, C53, C54, C55, C57, C59, C63, C64, C65, C67, C68, C69, C70, C71, C73, C75: value 0.1uF -> 0.1u
- C60: renamed from C62; value 0.1uF -> 0.1u
- C61: renamed from C60; value 10uF -> 10u
- C62: renamed from C61; value 10uF -> 10u
- C72: value 100uF -> 100u
- J10, J8, J9: value 39357-0004 -> 1702474
- U19: renamed from U22; value 74HCT125D -> 74HCT125D653
- U22: renamed from U25; value TPD4E1U06 -> TPD4E1U06DBV
- U24: renamed from U27; value TPD4E1U06 -> TPD4E1U06DBV
- U25: renamed from U28; value TPD4E1U06 -> TPD4E1U06DBV
- U26: renamed from U29; value TPD4E1U06 -> TPD4E1U06DBV
- renumbered L6 to L4, R103 to R100, R104 to R101, R105 to R102, R63 to R60, R64 to R61, R65 to R62, R66 to R63, R67 to R64, R68 to R65, R69 to R66, R70 to R67, R71 to R68, R72 to R69, R73 to R70, R74 to R71, R75 to R72, R76 to R73, R77 to R74, R78 to R75, R79 to R76, R80 to R77, R81 to R78, R82 to R79, R83 to R80, R84 to R81, R85 to R82, R86 to R83, R87 to R84, R88 to R85, R89 to R86, R90 to R87, R91 to R88, R92 to R89, R93 to R90, R94 to R91, R95 to R92, R96 to R93, R97 to R94, R98 to R95, R99 to R96, R100 to R97, R101 to R98, R102 to R99, TP107 to TP100, TP108 to TP101, TP109 to TP102, TP110 to TP103, TP111 to TP104, TP60 to TP53, TP61 to TP54, TP62 to TP55, TP63 to TP56, TP64 to TP57, TP65 to TP58, TP66 to TP59, TP67 to TP60, TP68 to TP61, TP69 to TP62, TP70 to TP63, TP71 to TP64, TP72 to TP65, TP73 to TP66, TP74 to TP67, TP75 to TP68, TP76 to TP69, TP77 to TP70, TP78 to TP71, TP79 to TP72, TP80 to TP73, TP81 to TP74, TP83 to TP75, TP84 to TP76, TP82 to TP77, TP87 to TP78, TP88 to TP79, TP85 to TP80, TP86 to TP81, TP89 to TP82, TP92 to TP83, TP93 to TP84, TP94 to TP85, TP90 to TP86, TP91 to TP87, TP97 to TP88, TP95 to TP89, TP96 to TP90, TP98 to TP91, TP99 to TP92, TP100 to TP93, TP101 to TP94, TP102 to TP95, TP103 to TP96, TP104 to TP97, TP105 to TP98, TP106 to TP99, U21 to U18, U23 to U20, U24 to U21, U26 to U23, U30 to U27, U31 to U28, U32 to U29
Connections:
- net AGND is gone; now on net DGND: C50.2, C57.1, C59.1, C60.1, C63.1, C64.1, C65.1, C66.2, C74.2, C75.1, R97.2, R99.2, U21.10 (RENIN(-)), U25.2 (GND), U26.2 (GND), U29.2 (GND)
- net ADI_A1+: now also J10.2 (Pin_2)
- net ADI_A1-: now also J10.3 (Pin_3)
- net ADI_A2+: now also J11.2 (Pin_2)
- net ADI_A2-: now also J11.3 (Pin_3)
- net ADI_A3+: now also J12.2 (Pin_2)
- net ADI_A3-: now also J12.3 (Pin_3)
- net ADI_PSW: now also J10.4 (Pin_4), J11.4 (Pin_4), J12.4 (Pin_4)
- net DGND: now also J13.4 (Pin_4), J7.4 (Pin_4); no longer J10.4 (Pin_4)
- net SONIC_ECHO: now also U24.1 (D1+)
- net SONIC_TRIG: now also U24.6 (D1-)
- net at D22.2 (A2), TP98.1, U27.6 (OUT1): now also J13.1 (Pin_1)
- net at D22.1 (A1), TP97.1, U27.8 (OUT2): now also J13.2 (Pin_2)
- net at D25.2 (A2), TP104.1, U28.10 (BOUT1): now also J14.3 (Pin_3)
- net at D24.2 (A2), TP102.1, U28.5 (AOUT1): now also J14.1 (Pin_1)
- net at D24.1 (A1), TP100.1, U28.7 (AOUT2): now also J14.2 (Pin_2)
- net at D25.1 (A1), TP103.1, U28.8 (BOUT2): now also J14.4 (Pin_4)
- net at D23.1 (A1), D23.2 (A2), Q3.1 (D): now also J13.3 (Pin_3)
- net at C74.1, C75.2, D19.2 (A)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: now also J10.1 (Pin_1), J11.1 (Pin_1), J12.1 (Pin_1)
- net at C62.1, D17.2 (A), D18.2 (A2)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: now also J7.1 (Pin_1); no longer J8.1 (Pin_1)
- net at C52.1, D13.2 (A), D15.2 (A2)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: now also J8.1 (Pin_1); no longer J9.1 (Pin_1)
- net at J8.2 (Pin_2): now also R78.1; no longer R76.1
- net at J8.3 (Pin_3): now also R79.1; no longer R77.1
- net at C56.1, D14.2 (A), D16.2 (A2)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: now also J9.1 (Pin_1); no longer J10.1 (Pin_1)
- net ADI_5V_FAULT renamed ~ADI_PWR_FAULT
- net ENCODE_PWR_FAULT renamed ~ENCDR_PWR_FAULT
- net POTEN_1 renamed POTEN_ADC_1
- net POTEN_ADC_1: now also U24.4 (D2-)
- net POTEN_2 renamed POTEN_ADC_2
- net POTEN_ADC_2: now also U24.3 (D2+)
- net POTEN_PWR_FAULT renamed ~POTEN_PWR_FAULT
- net ROTARY_1A renamed ENCDR_A
- net ROTARY_1B renamed ENCDR_B
- net SONIC_PWR_FAULT renamed ~SONIC_PWR_FAULT
- new net: J9.2 (Pin_2), R80.1
- new net: J9.3 (Pin_3), R81.1
- new net: J7.2 (Pin_2), R76.1
- new net: J7.3 (Pin_3), R77.1
Other:
- note added: "Both DC and Stepper\nMotor are powered\nfrom External Battery"
- note added: "Low-noise analog section of digital ground plane\nUse strong routing discipline, paying attention\nto the return current of all device\n"
- note added: "Remove resistor \nif using jumper"
- note removed: "Low Noise 5V Plane"
- moved on the sheet: C71, R77, R78, R79, R80, R81, U24
