File: pcb2/croptop_lcd.sch (KiCad schematic (older format))
At the start: 74 parts

Commit message: Added USB port control
Parts:
- removed C?: 0.1uF, Capacitor_SMD:C_0402_1005Metric, symbol Device:C
- added C?: 0.1uF, Capacitor_SMD:C_0402_1005Metric, symbol Device:C
Connections:
- wire segments 329 -> 330
Other:
- moved on the sheet: C?
Changed lines of the file:
@@
 Comment4 ""
 $EndDescr
-Wire Wire Line
-	3050 5350 3400 5350
 $Comp
 L CropTop:DGND #PWR?
@@
 	3400 4450 3500 4450
 Wire Wire Line
-	3400 5750 3400 5800
-Wire Wire Line
-	3050 5750 3050 5800
-Wire Wire Line
-	2700 5750 2700 5800
-Wire Wire Line
-	2350 5750 2350 5800
+	3350 5700 3350 5800
+Wire Wire Line
+	2900 5700 2900 5800
+Wire Wire Line
+	2450 5700 2450 5800
+Wire Wire Line
+	2000 5700 2000 5800
 $Comp
 L CropTop:DGND #PWR?
 U 1 1 5D9BF7E3
-P 3400 5800
-F 0 "#PWR?" H 3400 5550 50  0001 C CNN
-F 1 "DGND" H 3404 5645 50  0000 C CNN
-F 2 "" H 3400 5800 50  0001 C CNN
-F 3 "" H 3400 5800 50  0001 C CNN
-	1    3400 5800
+P 3350 5800
+F 0 "#PWR?" H 3350 5550 50  0001 C CNN
+F 1 "DGND" H 3354 5645 50  0000 C CNN
+F 2 "" H 3350 5800 50  0001 C CNN
+F 3 "" H 3350 5800 50  0001 C CNN
+	1    3350 5800
 	1    0    0    -1
 $EndComp
@@
 L CropTop:DGND #PWR?
 U 1 1 5D9BF6F8
-P 3050 5800
-F 0 "#PWR?" H 3050 5550 50  0001 C CNN
-F 1 "DGND" H 3054 5645 50  0000 C CNN
-F 2 "" H 3050 5800 50  0001 C CNN
-F 3 "" H 3050 5800 50  0001 C CNN
-	1    3050 5800
+P 2900 5800
+F 0 "#PWR?" H 2900 5550 50  0001 C CNN
+F 1 "DGND" H 2904 5645 50  0000 C CNN
+F 2 "" H 2900 5800 50  0001 C CNN
+F 3 "" H 2900 5800 50  0001 C CNN
+	1    2900 5800
 	1    0    0    -1
 $EndComp
@@
 L CropTop:DGND #PWR?
 U 1 1 5D9BF60D
-P 2700 5800
-F 0 "#PWR?" H 2700 5550 50  0001 C CNN
-F 1 "DGND" H 2704 5645 50  0000 C CNN
-F 2 "" H 2700 5800 50  0001 C CNN
-F 3 "" H 2700 5800 50  0001 C CNN
-	1    2700 5800
+P 2450 5800
+F 0 "#PWR?" H 2450 5550 50  0001 C CNN
+F 1 "DGND" H 2454 5645 50  0000 C CNN
+F 2 "" H 2450 5800 50  0001 C CNN
+F 3 "" H 2450 5800 50  0001 C CNN
+	1    2450 5800
 	1    0    0    -1
 $EndComp
@@
 L CropTop:DGND #PWR?
 U 1 1 5D9BF522
-P 2350 5800
-F 0 "#PWR?" H 2350 5550 50  0001 C CNN
-F 1 "DGND" H 2354 5645 50  0000 C CNN
-F 2 "" H 2350 5800 50  0001 C CNN
-F 3 "" H 2350 5800 50  0001 C CNN
-	1    2350 5800
-	1    0    0    -1
-$EndComp
-Wire Wire Line
-	3050 5450 3050 5350
-Connection ~ 3050 5350
-Wire Wire Line
-	2700 5350 3050 5350
-Wire Wire Line
-	2700 5450 2700 5350
-Wire Wire Line
-	3400 5350 3400 5450
-Wire Wire Line
-	2350 5450 2350 5350
-Wire Wire Line
-	2350 5250 2350 5350
-Connection ~ 2350 5350
-Wire Wire Line
-	2350 5350 2700 5350
-$Comp
-L Device:C C?
-U 1 1 5D8DF21F
-P 2350 5600
-AR Path="/5D8DF21F" Ref="C?"  Part="1"
-AR Path="/65B709D0/5D8DF21F" Ref="C?"  Part="1"
-AR Path="/66A12230/5D8DF21F" Ref="C?"  Part="1"
-AR Path="/669AB112/5D8DF21F" Ref="C?"  Part="1"
-F 0 "C?" H 2400 5700 50  0000 L CNN
-F 1 "0.1uF" H 2400 5500 50  0000 L CNN
-F 2 "Capacitor_SMD:C_0402_1005Metric" H 2388 5450 50  0001 C CNN
-F 3 "~" H 2350 5600 50  0001 C CNN
-	1    2350 5600
-	1    0    0    -1
-$EndComp
+P 2000 5800
+F 0 "#PWR?" H 2000 5550 50  0001 C CNN
+F 1 "DGND" H 2004 5645 50  0000 C CNN
+F 2 "" H 2000 5800 50  0001 C CNN
+F 3 "" H 2000 5800 50  0001 C CNN
+	1    2000 5800
+	1    0    0    -1
+$EndComp
+Wire Wire Line
+	2900 5400 2900 5300
+Wire Wire Line
+	2450 5400 2450 5300
+Wire Wire Line
+	3350 5300 3350 5400
+Wire Wire Line
+	2000 5400 2000 5300
+Wire Wire Line
+	1900 5200 1900 5300
 $Comp
 L Device:C C?
 U 1 1 5D8B2D88
-P 3400 5600
+P 3350 5550
 AR Path="/5D8B2D88" Ref="C?"  Part="1"
 AR Path="/65B709D0/5D8B2D88" Ref="C?"  Part="1"
 AR Path="/66A12230/5D8B2D88" Ref="C?"  Part="1"
 AR Path="/669AB112/5D8B2D88" Ref="C?"  Part="1"
-F 0 "C?" H 3450 5700 50  0000 L CNN
-F 1 "0.1uF" H 3450 5500 50  0000 L CNN
-F 2 "Capacitor_SMD:C_0402_1005Metric" H 3438 5450 50  0001 C CNN
-F 3 "~" H 3400 5600 50  0001 C CNN
-	1    3400 5600
+F 0 "C?" H 3465 5596 50  0000 L CNN
+F 1 "0.1uF" H 3465 5505 50  0000 L CNN
+F 2 "Capacitor_SMD:C_0402_1005Metric" H 3388 5400 50  0001 C CNN
+F 3 "~" H 3350 5550 50  0001 C CNN
+	1    3350 5550
 	1    0    0    -1
 $EndComp
@@
 L Device:C C?
 U 1 1 5D8B2C8E
-P 3050 5600
+P 2900 5550
 AR Path="/5D8B2C8E" Ref="C?"  Part="1"
 AR Path="/65B709D0/5D8B2C8E" Ref="C?"  Part="1"
 AR Path="/66A12230/5D8B2C8E" Ref="C?"  Part="1"
 AR Path="/669AB112/5D8B2C8E" Ref="C?"  Part="1"
-F 0 "C?" H 3100 5700 50  0000 L CNN
-F 1 "0.1uF" H 3100 5500 50  0000 L CNN
-F 2 "Capacitor_SMD:C_0402_1005Metric" H 3088 5450 50  0001 C CNN
-F 3 "~" H 3050 5600 50  0001 C CNN
-	1    3050 5600
+F 0 "C?" H 3015 5596 50  0000 L CNN
+F 1 "0.1uF" H 3015 5505 50  0000 L CNN
+F 2 "Capacitor_SMD:C_0402_1005Metric" H 2938 5400 50  0001 C CNN
+F 3 "~" H 2900 5550 50  0001 C CNN
+	1    2900 5550
 	1    0    0    -1
 $EndComp
@@
 L Device:C C?
 U 1 1 5D8B2B8A
-P 2700 5600
+P 2450 5550
 AR Path="/5D8B2B8A" Ref="C?"  Part="1"
 AR Path="/65B709D0/5D8B2B8A" Ref="C?"  Part="1"
 AR Path="/66A12230/5D8B2B8A" Ref="C?"  Part="1"
 AR Path="/669AB112/5D8B2B8A" Ref="C?"  Part="1"
-F 0 "C?" H 2750 5700 50  0000 L CNN
-F 1 "0.1uF" H 2750 5500 50  0000 L CNN
-F 2 "Capacitor_SMD:C_0402_1005Metric" H 2738 5450 50  0001 C CNN
-F 3 "~" H 2700 5600 50  0001 C CNN
-	1    2700 5600
+F 0 "C?" H 2565 5596 50  0000 L CNN
+F 1 "0.1uF" H 2565 5505 50  0000 L CNN
+F 2 "Capacitor_SMD:C_0402_1005Metric" H 2488 5400 50  0001 C CNN
+F 3 "~" H 2450 5550 50  0001 C CNN
+	1    2450 5550
 	1    0    0    -1
 $EndComp
@@
 L CropTop:DGND #PWR?
 U 1 1 5D62F7FF
-P 3150 6500
-F 0 "#PWR?" H 3150 6250 50  0001 C CNN
-F 1 "DGND" H 3154 6345 50  0000 C CNN
-F 2 "" H 3150 6500 50  0001 C CNN
-F 3 "" H 3150 6500 50  0001 C CNN
-	1    3150 6500
+P 3000 6600
+F 0 "#PWR?" H 3000 6350 50  0001 C CNN
+F 1 "DGND" H 3004 6445 50  0000 C CNN
+F 2 "" H 3000 6600 50  0001 C CNN
+F 3 "" H 3000 6600 50  0001 C CNN
+	1    3000 6600
 	1    0    0    -1
 $EndComp
@@
 L CropTop:DGND #PWR?
 U 1 1 5D62F7F2
-P 3500 6500
-F 0 "#PWR?" H 3500 6250 50  0001 C CNN
-F 1 "DGND" H 3504 6345 50  0000 C CNN
-F 2 "" H 3500 6500 50  0001 C CNN
-F 3 "" H 3500 6500 50  0001 C CNN
-	1    3500 6500
-	1    0    0    -1
-$EndComp
-Wire Wire Line
-	3150 6150 3150 6100
-Wire Wire Line
-	3500 6500 3500 6450
-Wire Wire Line
-	3150 6500 3150 6450
-Wire Wire Line
-	3150 6100 3500 6100
-Wire Wire Line
-	3500 6100 3950 6100
-Connection ~ 3500 6100
-Wire Wire Line
-	3500 6150 3500 6100
+P 3450 6600
+F 0 "#PWR?" H 3450 6350 50  0001 C CNN
+F 1 "DGND" H 3454 6445 50  0000 C CNN
+F 2 "" H 3450 6600 50  0001 C CNN
+F 3 "" H 3450 6600 50  0001 C CNN
+	1    3450 6600
+	1    0    0    -1
+$EndComp
+Wire Wire Line
+	3450 6600 3450 6500
+Wire Wire Line
+	3000 6600 3000 6500
 $Comp
 L Device:C C?
 U 1 1 5D62F7E5
-P 3150 6300
+P 3000 6350
 AR Path="/5D62F7E5" Ref="C?"  Part="1"
 AR Path="/65B709D0/5D62F7E5" Ref="C?"  Part="1"
 AR Path="/66A12230/5D62F7E5" Ref="C?"  Part="1"
 AR Path="/669AB112/5D62F7E5" Ref="C?"  Part="1"
-F 0 "C?" H 3200 6400 50  0000 L CNN
-F 1 "10uF" H 3200 6200 50  0000 L CNN
-F 2 "Capacitor_SMD:C_0805_2012Metric" H 3188 6150 50  0001 C CNN
-F 3 "~" H 3150 6300 50  0001 C CNN
-	1    3150 6300
+F 0 "C?" H 3114 6396 50  0000 L CNN
+F 1 "10uF" H 3114 6305 50  0000 L CNN
+F 2 "Capacitor_SMD:C_0805_2012Metric" H 3038 6200 50  0001 C CNN
+F 3 "~" H 3000 6350 50  0001 C CNN
+	1    3000 6350
 	1    0    0    -1
 $EndComp
@@
 L Device:C C?
 U 1 1 5D62F7DE
-P 3500 6300
+P 3450 6350
 AR Path="/5D62F7DE" Ref="C?"  Part="1"
 AR Path="/65B709D0/5D62F7DE" Ref="C?"  Part="1"
 AR Path="/66A12230/5D62F7DE" Ref="C?"  Part="1"
 AR Path="/669AB112/5D62F7DE" Ref="C?"  Part="1"
-F 0 "C?" H 3550 6400 50  0000 L CNN
-F 1 "0.1uF" H 3550 6200 50  0000 L CNN
-F 2 "Capacitor_SMD:C_0402_1005Metric" H 3538 6150 50  0001 C CNN
-F 3 "~" H 3500 6300 50  0001 C CNN
-	1    3500 6300
+F 0 "C?" H 3565 6396 50  0000 L CNN
+F 1 "0.1uF" H 3565 6305 50  0000 L CNN
+F 2 "Capacitor_SMD:C_0402_1005Metric" H 3488 6200 50  0001 C CNN
+F 3 "~" H 3450 6350 50  0001 C CNN
+	1    3450 6350
 	1    0    0    -1
 $EndComp
@@
 L power:+3V3 #PWR?
 U 1 1 5C758084
-P 2350 5250
+P 1900 5200
 AR Path="/64807BBC/5C758084" Ref="#PWR?"  Part="1"
 AR Path="/65B709D0/5C758084" Ref="#PWR?"  Part="1"
-F 0 "#PWR?" H 2350 5100 50  0001 C CNN
-F 1 "+3V3" H 2365 5423 50  0000 C CNN
-F 2 "" H 2350 5250 50  0001 C CNN
-F 3 "" H 2350 5250 50  0001 C CNN
-	1    2350 5250
+F 0 "#PWR?" H 1900 5050 50  0001 C CNN
+F 1 "+3V3" H 1915 5373 50  0000 C CNN
+F 2 "" H 1900 5200 50  0001 C CNN
+F 3 "" H 1900 5200 50  0001 C CNN
+	1    1900 5200
 	1    0    0    -1
 $EndComp
@@
 	0    1    1    0
 $EndComp
-Connection ~ 2700 5350
 Wire Wire Line
 	6250 2900 6350 2900
@@
 Wire Wire Line
 	9200 5300 8550 5300
-Wire Wire Line
-	3400 5350 3750 5350
-Wire Wire Line
-	3750 5350 3750 5600
-Connection ~ 3400 5350
 Connection ~ 3750 5600
 $Comp
@@
 Wire Wire Line
 	3350 3500 3350 3600
+$Comp
+L Device:C C?
+U 1 1 5D6336C5
+P 2000 5550
+AR Path="/5D6336C5" Ref="C?"  Part="1"
+AR Path="/65B709D0/5D6336C5" Ref="C?"  Part="1"
+AR Path="/66A12230/5D6336C5" Ref="C?"  Part="1"
+AR Path="/669AB112/5D6336C5" Ref="C?"  Part="1"
+F 0 "C?" H 2115 5596 50  0000 L CNN
+F 1 "0.1uF" H 2115 5505 50  0000 L CNN
+F 2 "Capacitor_SMD:C_0402_1005Metric" H 2038 5400 50  0001 C CNN
+F 3 "~" H 2000 5550 50  0001 C CNN
+	1    2000 5550
+	1    0    0    -1
+$EndComp
+Wire Wire Line
+	1900 5300 2000 5300
+Wire Wire Line
+	3750 5300 3750 5600
+Connection ~ 2000 5300
+Connection ~ 2450 5300
+Connection ~ 2900 5300
+Connection ~ 3350 5300
+Wire Wire Line
+	3350 5300 3750 5300
+Wire Wire Line
+	2900 5300 3350 5300
+Wire Wire Line
+	2450 5300 2900 5300
+Wire Wire Line
+	2000 5300 2450 5300
+Wire Wire Line
+	3450 6100 3450 6200
+Wire Wire Line
+	3000 6100 3000 6200
+Connection ~ 3450 6100
+Wire Wire Line
+	3450 6100 3950 6100
+Wire Wire Line
+	3000 6100 3450 6100
 $EndSCHEMATC

Commit message: Schematic near completion
Parts:
- C?: footprint Capacitor_SMD:C_0805_2012Metric -> Capacitor_SMD:C_0402_1005Metric
- J?: Note (none) -> LCD
- R? (x30): footprint (none) -> Resistor_SMD:R_0402_1005Metric
- Y?: value 12MHz -> ABLS-12.000MHZ-B2-T

Commit message: Added pmod
Parts:
- removed J?: 4-1734839-0, croptop:4-1734839-0, symbol CropTop:54104-4031
- removed Y?: ABLS-12.000MHZ-B2-T, croptop:ABLS_OX, symbol Device:Crystal_Small
- added C?: 0.1uF, Capacitor_SMD:C_0402_1005Metric, symbol Device:C
- added D? (x2): LTSTC171GKT, LED_SMD:LED_0805_2012Metric, symbol Device:LED
- added J?: 0541044031, symbol CropTop:0541044031
- added J?: 0522070433, symbol CropTop:0522070433
- added J?: D.N.P., symbol Connector_Generic:Conn_01x02
- added Q? (x2): BSS138, symbol Device:Q_NMOS_GSD
- added R? (x3): 10k, Resistor_SMD:R_0402_1005Metric, symbol Device:R
- added R? (x4): 22, Resistor_SMD:R_0402_1005Metric, symbol Device:R
- added R? (x4): 100, Resistor_SMD:R_0402_1005Metric, symbol Device:R
- added TP? (x12): TestPoint, symbol Connector:TestPoint
- added Y?: ABLS-12.000MHZ-B2-T, symbol Device:Crystal
- R?: value 4.7k -> 10k
Connections:
- net labels added: GPU_LED_1, GPU_LED_2, GPU_MISO, GPU_MOSI, GPU_PWM, GPU_SCLK, ~GPU_CS, ~GPU_INT, ~GPU_PD
- net labels removed: LCD_INT, LCD_PD, LCD_PWM
- wire segments 330 -> 392
- no-connect marks 6 -> 7
Other:
- note added: "Connects to 7" 800x480 TFT LCD\nNHD-7.0-800480EF-ASXN#-T\n"
- note added: "D.N.P."
- note added: "Resistive Touch\nPanel Interface"
- moved on the sheet: C?, R?, TP?, U?

Commit message: pwm
Parts:
- R23, R26, R28, R30: renamed from R?; value 100 -> 100Ω
- R24, R25, R27, R29: renamed from R?; value 10k -> 10kΩ
- R31, R32, R33, R34, R35, R36, R37, R38, R39, R40, R41, R42, R43, R44, R45, R46, R47, R48, R49, R50, R51, R52, R53, R54, R55, R56, R57, R58, R59, R60, R61, R62, R63: renamed from R?; value 22 -> 22Ω
- gave numbers to parts that had none: 63

Commit message: Added TVS diodes
Parts:
- removed C36: 0.1uF, Capacitor_SMD:C_0402_1005Metric, symbol Device:C
- removed C40: 26pF, Capacitor_SMD:C_0402_1005Metric, symbol Device:C
- removed R63: 22Ω, Resistor_SMD:R_0402_1005Metric, symbol Device:R
- removed TP60, TP61, TP62, TP63: TestPoint, symbol Connector:TestPoint
- added C41: 26pF, Capacitor_SMD:C_0402_1005Metric, symbol Device:C
- added D11: TPD2E007, symbol Device:D_TVS_x2_AAC
- added D12: TPD1E6B06, symbol Device:D_TVS
- added R34: 22Ω, Resistor_SMD:R_0402_1005Metric, symbol Device:R
- added U11, U13, U14, U15, U16, U17, U18, U19, U20: TPD4E1U06, symbol CropTop:TPD4E1U06
- J6: renamed from J7; value 0522070433 -> 686104183422
- J7: renamed from J6; value 0541044031 -> 62684-402100ALF
- renumbered C39 to C38, C38 to C39, C41 to C40, R25 to R22, R27 to R23, R23 to R24, R24 to R25, R31 to R27, R32 to R28, R33 to R29, R34 to R30, R28 to R31, R29 to R32, R30 to R33, TP21 to TP19, TP19 to TP21, TP27 to TP24, TP28 to TP27, TP29 to TP28, TP30 to TP29, TP24 to TP30, U11 to U12
Connections:
- net +3V3: now also D12.2 (A2)
- net DGND: now also C41.2, D11.3 (common), D12.1 (A1), U11.2 (GND), U13.2 (GND), U14.2 (GND), U15.2 (GND), U16.2 (GND), U17.2 (GND), U18.2 (GND), U19.2 (GND), U20.2 (GND)
- net LCD_A: now also D11.2 (A2)
- net LCD_K: now also D11.1 (A1)
- net ~GPU_INT: now also TP20.1; no longer TP19.1
- net ~GPU_PD: now also TP19.1; no longer TP20.1
- net at TP28.1, U12.17 (X2), Y2.2: now also C41.1
- net at TP31.1, U12.2 (R0): now also R34.2; no longer R35.2
- net GPU_X+: now reaches J6.1 (XR), U12.23 (X+)
- net GPU_X+: now also U11.1 (D1+)
- net GPU_Y+: now reaches J6.4 (YU), U12.24 (Y+)
- net GPU_Y+: now also U11.4 (D2-)
- net GPU_X-: now reaches J6.3 (XL), U12.25 (X-)
- net GPU_X-: now also U11.3 (D2+)
- net GPU_Y-: now reaches J6.2 (YD), U12.26 (Y-)
- net GPU_Y-: now also U11.6 (D1-)
- net at R49.2: now also TP33.1, U12.1 (R1); no longer U12.29 (DE)
- net at U12.30 (VSYNC): now also R62.2, TP34.1
- net at R48.2: now also TP32.1, U12.29 (DE); no longer U12.31 (HSYNC)
- net at U12.32 (DISP): now also R61.2, TP38.1; no longer R62.2
- net at R47.2: now also TP36.1, U12.31 (HSYNC); no longer U12.33 (PCLK)
- net at U12.34 (B7): now also R60.2, TP42.1; no longer R61.2
- net at R46.2: now also TP40.1, U12.33 (PCLK); no longer U12.35 (B6)
- net at U12.36 (B5): now also R59.2, TP46.1; no longer R60.2
- net at R45.2: now also TP44.1, U12.35 (B6); no longer U12.37 (B4)
- net at U12.38 (B3): now also R58.2, TP50.1; no longer R59.2
- net at R44.2: now also TP48.1, U12.37 (B4); no longer U12.39 (B2)
- net at U12.40 (B1): now also R57.2, TP54.1; no longer R58.2
- net at J7.10 (R5): now also R51.1, U14.3 (D2+); no longer R52.1
- net at J7.11 (R6): now also R37.1, U14.6 (D1-); no longer R38.1
- net at J7.12 (R7): now also R52.1, U14.1 (D1+); no longer R53.1
- net at J7.13 (G0): now also R38.1, U15.4 (D2-); no longer R39.1
- net at J7.14 (G1): now also R53.1, U15.3 (D2+); no longer R54.1
- net at J7.15 (G2): now also R39.1, U15.6 (D1-); no longer R40.1
- net at J7.16 (G3): now also R54.1, U15.1 (D1+); no longer R55.1
- net at J7.17 (G4): now also R40.1, U16.4 (D2-); no longer R41.1
- net at J7.18 (G5): now also R55.1, U16.3 (D2+); no longer R56.1
- net at J7.19 (G6): now also R41.1, U16.6 (D1-); no longer R42.1
- net at J7.20 (G7): now also R56.1, U16.1 (D1+); no longer R57.1
- net at J7.21 (B0): now also R42.1, U17.4 (D2-); no longer R43.1
- net at TP58.1: now also R56.2, U12.43 (G7); no longer J7.33 (VSYNC)
- net at J7.5 (R0): now also R34.1, U13.4 (D2-); no longer R35.1
- net at J7.6 (R1): now also R49.1, U13.3 (D2+); no longer R50.1
- net at J7.7 (R2): now also R35.1, U13.6 (D1-); no longer R36.1
- net at J7.8 (R3): now also R50.1, U13.1 (D1+); no longer R51.1
- net at J7.9 (R4): now also R36.1, U14.4 (D2-); no longer R37.1
- new net: R43.2, TP52.1, U12.39 (B2)
- new net: R42.2, TP56.1, U12.41 (B0)
- new net: R41.2, TP59.1, U12.44 (G6)
- new net: R55.2, TP57.1, U12.45 (G5)
- new net: R40.2, TP55.1, U12.46 (G4)
- new net: R54.2, TP53.1, U12.47 (G3)
- new net: R39.2, TP51.1, U12.48 (G2)
- new net: R53.2, TP49.1, U12.49 (G1)
- new net: R38.2, TP47.1, U12.50 (G0)
- new net: R52.2, TP45.1, U12.51 (R7)
- new net: R37.2, TP43.1, U12.52 (R6)
- new net: R51.2, TP41.1, U12.53 (R5)
- new net: R36.2, TP39.1, U12.54 (R4)
- new net: R50.2, TP37.1, U12.55 (R3)
- new net: R35.2, TP35.1, U12.56 (R2)
- new net: J7.22 (B1), R57.1, U17.3 (D2+)
- new net: J7.23 (B2), R43.1, U17.6 (D1-)
- new net: J7.24 (B3), R58.1, U17.1 (D1+)
- new net: J7.25 (B4), R44.1, U18.4 (D2-)
- new net: J7.26 (B5), R59.1, U18.3 (D2+)
- new net: J7.27 (B6), R45.1, U18.6 (D1-)
- new net: J7.28 (B7), R60.1, U18.1 (D1+)
- new net: J7.30 (CLK), R46.1, U19.4 (D2-)
- new net: J7.31 (DISP), R61.1, U19.3 (D2+)
- new net: J7.32 (HSYNC), R47.1, U19.6 (D1-)
- new net: J7.33 (VSYNC), R62.1, U19.1 (D1+)
- new net: J7.34 (DE), R48.1, U20.4 (D2-)
- no-connect marks 7 -> 19
Other:
- note added: "Graphics Processing Unit"
- note added: "Resittive Touch Panel FPC Connector"
- note added: "TFT LCD Display FPC Connector"
- note removed: "FCP Connector for TFT LCD"
- note removed: "Graphics Controller"
- note removed: "Resistive Touch\nPanel Interface"
- moved on the sheet: C37, C38, C39, C40, C42, C43, C44, D10, D9, J5, J6, J7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
