File: pcb2/croptop_lcd.sch (KiCad schematic (older format))
At the start: 110 parts, among them J5 D.N.P., J6 686104183422, J7 62684-402100ALF, Q1 BSS138, Q2 BSS138, U11 TPD4E1U06, U12 FT812Q, U13 TPD4E1U06, U14 TPD4E1U06, U15 TPD4E1U06, U16 TPD4E1U06, U17 TPD4E1U06, U18 TPD4E1U06, U19 TPD4E1U06, U20 TPD4E1U06, Y2 ABLS-12.000MHZ-B2-T

Commit message: Final Schematic
Parts:
- added C?: 0.1uF, Capacitor_SMD:C_0402_1005Metric, symbol Device:C
Connections:
- net DGND: now also C?.2
- net ~GPU_INT: now also U12.13 (INT_N); no longer U12.14 (PD_N)
- net ~GPU_PD: now also U12.14 (PD_N), C?.1; no longer U12.13 (INT_N)
Other:
- note added: "TFT GPU Display FPC Connector"
- note removed: "TFT LCD Display FPC Connector"
- moved on the sheet: TP19, TP20
Changed lines of the file:
@@
 Wire Wire Line
 	3550 6100 3750 6100
-Text GLabel 950  4050 0    39   Input ~ 0
+Text GLabel 900  4200 0    33   Input ~ 0
 ~GPU_PD
-Text GLabel 950  4250 0    39   Output ~ 0
+Text GLabel 900  4100 0    33   Output ~ 0
 ~GPU_INT
 Wire Wire Line
@@
 Wire Wire Line
 	3750 5400 3650 5400
-Text GLabel 3650 5400 0    39   Output ~ 0
+Text GLabel 3650 5400 0    33   Output ~ 0
 GPU_PWM
 $Comp
@@
 F 1 "FT812Q" H 4600 7176 50  0000 C CNN
 F 2 "Package_DFN_QFN:QFN-56-1EP_8x8mm_P0.5mm_EP4.5x5.2mm" H 4625 5175 50  0001 C CNN
-F 3 "" H 4625 5175 50  0001 C CNN
+F 3 "https://brtchip.com/wp-content/uploads/Support/Documentation/Datasheets/ICs/EVE/DS_FT81x.pdf" H 4625 5175 50  0001 C CNN
 	1    4550 5300
 	1    0    0    -1
@@
 Graphics Processing Unit
 Text Notes 13900 1300 0    98   ~ 20
-TFT LCD Display FPC Connector
+TFT GPU Display FPC Connector
 $Comp
 L power:+3V3 #PWR?
@@
 Wire Wire Line
 	1800 4400 1800 5000
-Text GLabel 2100 3400 0    39   Input ~ 0
+Text GLabel 2100 3400 0    33   Input ~ 0
 GPU_MOSI
-Text GLabel 2100 4000 0    39   Input ~ 0
+Text GLabel 2100 4000 0    33   Input ~ 0
 GPU_SCLK
-Text GLabel 2100 3700 0    39   Output ~ 0
+Text GLabel 2100 3700 0    33   Output ~ 0
 GPU_MISO
-Text GLabel 2100 3100 0    39   Input ~ 0
+Text GLabel 2100 3100 0    33   Input ~ 0
 ~GPU_CS
 Wire Wire Line
@@
 Wire Wire Line
 	1500 3650 1500 3700
-Wire Wire Line
-	1150 4000 1150 4100
-Wire Wire Line
-	1500 4000 1500 4200
 Wire Wire Line
 	2100 4000 2200 4000
@@
 Wire Wire Line
 	2200 4000 3050 4000
-Wire Wire Line
-	1500 4200 1600 4200
 $Comp
 L Device:Q_NMOS_GSD Q?
@@
 Wire Wire Line
 	2500 7900 2500 8000
-Text GLabel 1600 9000 0    39   Input ~ 0
+Text GLabel 1600 9000 0    33   Input ~ 0
 GPU_LED_1
 $Comp
@@
 Wire Wire Line
 	4450 7900 4450 8000
-Text GLabel 3550 9000 0    39   Input ~ 0
+Text GLabel 3550 9000 0    33   Input ~ 0
 GPU_LED_2
 $Comp
@@
 Wire Wire Line
 	4050 8900 4050 9000
-Text GLabel 3650 5200 0    39   Output ~ 0
+Text GLabel 3650 5200 0    33   Output ~ 0
 GPU_LED_2
 NoConn ~ 3750 4800
 NoConn ~ 3750 4900
-Text GLabel 3650 5100 0    39   Output ~ 0
+Text GLabel 3650 5100 0    33   Output ~ 0
 GPU_LED_1
 Wire Wire Line
@@
 L Connector:TestPoint TP?
 U 1 1 5FB7E1C8
-P 1250 4300
+P 1400 4400
 AR Path="/64809F0C/5FB7E1C8" Ref="TP?"  Part="1"
 AR Path="/65B709D0/5FB7E1C8" Ref="TP19"  Part="1"
-F 0 "TP19" H 1160 4500 50  0000 L CNN
-F 1 "TestPoint" H 1308 4329 50  0001 L CNN
-F 2 "" H 1450 4300 50  0001 C CNN
-F 3 "" H 1450 4300 50  0001 C CNN
-	1    1250 4300
+F 0 "TP19" H 1310 4600 50  0000 L CNN
+F 1 "TestPoint" H 1458 4429 50  0001 L CNN
+F 2 "" H 1600 4400 50  0001 C CNN
+F 3 "" H 1600 4400 50  0001 C CNN
+	1    1400 4400
 	-1   0    0    1
 $EndComp
@@
 Wire Wire Line
 	3500 2050 3500 2200
-Text GLabel 2850 1300 0    39   Output ~ 0
+Text GLabel 2850 1300 0    33   Output ~ 0
 GPU_X+
-Text GLabel 2850 1400 0    39   Output ~ 0
+Text GLabel 2850 1400 0    33   Output ~ 0
 GPU_Y-
-Text GLabel 2850 1600 0    39   Output ~ 0
+Text GLabel 2850 1600 0    33   Output ~ 0
 GPU_Y+
-Text GLabel 2850 1500 0    39   Output ~ 0
+Text GLabel 2850 1500 0    33   Output ~ 0
 GPU_X-
-Text GLabel 5550 6700 2    39   Input ~ 0
+Text GLabel 5550 6700 2    33   Input ~ 0
 GPU_X+
-Text GLabel 5550 6800 2    39   Input ~ 0
+Text GLabel 5550 6800 2    33   Input ~ 0
 GPU_Y-
-Text GLabel 5550 7000 2    39   Input ~ 0
+Text GLabel 5550 7000 2    33   Input ~ 0
 GPU_Y+
-Text GLabel 5550 6900 2    39   Input ~ 0
+Text GLabel 5550 6900 2    33   Input ~ 0
 GPU_X-
 Wire Wire Line
@@
 	2200 4900 3250 4900
 Connection ~ 2200 4900
-Wire Wire Line
-	1150 4100 1050 4100
-Wire Wire Line
-	1050 4100 1050 4050
-Wire Wire Line
-	1050 4050 950  4050
-Connection ~ 1150 4100
-Wire Wire Line
-	950  4250 1050 4250
-Wire Wire Line
-	1050 4250 1050 4200
-Connection ~ 1500 4200
 $Comp
 L Connector:TestPoint TP?
 U 1 1 60F30E3B
-P 1600 4400
+P 1650 4400
 AR Path="/64809F0C/60F30E3B" Ref="TP?"  Part="1"
 AR Path="/65B709D0/60F30E3B" Ref="TP20"  Part="1"
-F 0 "TP20" H 1510 4600 50  0000 L CNN
-F 1 "TestPoint" H 1658 4429 50  0001 L CNN
-F 2 "" H 1800 4400 50  0001 C CNN
-F 3 "" H 1800 4400 50  0001 C CNN
-	1    1600 4400
+F 0 "TP20" H 1560 4600 50  0000 L CNN
+F 1 "TestPoint" H 1708 4429 50  0001 L CNN
+F 2 "" H 1850 4400 50  0001 C CNN
+F 3 "" H 1850 4400 50  0001 C CNN
+	1    1650 4400
 	-1   0    0    1
 $EndComp
-Wire Wire Line
-	1600 4400 1600 4200
-Connection ~ 1600 4200
-Wire Wire Line
-	1600 4200 3750 4200
-Wire Wire Line
-	1150 4100 1250 4100
-Wire Wire Line
-	1050 4200 1500 4200
-Wire Wire Line
-	1250 4300 1250 4100
 Wire Wire Line
 	8500 2000 9150 2000
@@
 Wire Wire Line
 	3100 5600 3750 5600
-Connection ~ 1250 4100
-Wire Wire Line
-	1250 4100 3750 4100
 Text Notes 2100 1150 0    98   ~ 20
 Resittive Touch Panel FPC Connector
@@
 Wire Wire Line
 	14600 6500 14600 8400
+Wire Wire Line
+	1000 4600 1000 4700
+$Comp
+L CropTop:DGND #PWR?
+U 1 1 5D6170F4
+P 1000 4700
+F 0 "#PWR?" H 1000 4450 50  0001 C CNN
+F 1 "DGND" H 1004 4545 50  0000 C CNN
+F 2 "" H 1000 4700 50  0001 C CNN
+F 3 "" H 1000 4700 50  0001 C CNN
+	1    1000 4700
+	1    0    0    -1
+$EndComp
+$Comp
+L Device:C C?
+U 1 1 5D6170FB
+P 1000 4450
+AR Path="/5D6170FB" Ref="C?"  Part="1"
+AR Path="/65B709D0/5D6170FB" Ref="C?"  Part="1"
+AR Path="/66A12230/5D6170FB" Ref="C?"  Part="1"
+AR Path="/669AB112/5D6170FB" Ref="C?"  Part="1"
+F 0 "C?" H 1115 4496 50  0000 L CNN
+F 1 "0.1uF" H 1115 4405 50  0000 L CNN
+F 2 "Capacitor_SMD:C_0402_1005Metric" H 1038 4300 50  0001 C CNN
+F 3 "" H 1000 4450 50  0001 C CNN
+	1    1000 4450
+	1    0    0    -1
+$EndComp
+Wire Wire Line
+	1650 4400 1650 4100
+Connection ~ 1650 4100
+Wire Wire Line
+	1650 4100 3750 4100
+Wire Wire Line
+	900  4200 1000 4200
+Wire Wire Line
+	1500 4000 1500 4100
+Connection ~ 1500 4100
+Wire Wire Line
+	1500 4100 1650 4100
+Wire Wire Line
+	1400 4400 1400 4200
+Connection ~ 1400 4200
+Wire Wire Line
+	1400 4200 3750 4200
+Wire Wire Line
+	1000 4300 1000 4200
+Connection ~ 1000 4200
+Wire Wire Line
+	1000 4200 1150 4200
+Wire Wire Line
+	900  4100 1150 4100
+Wire Wire Line
+	1150 4100 1500 4100
+Connection ~ 1150 4200
+Wire Wire Line
+	1150 4200 1400 4200
+Wire Wire Line
+	1150 4000 1150 4200
 $EndSCHEMATC

Commit message: Schematic Done
Parts:
- removed J5: D.N.P., symbol Connector_Generic:Conn_01x02
- removed TP25, TP26: TestPoint, symbol Connector:TestPoint
- added J4: TSM-102-01-T-DV, symbol Connector_Generic:Conn_02x02_Odd_Even
- C36: renamed from C?; value 0.1uF -> 0.1u
- C37, C42, C44: value 0.1uF -> 0.1u
- C38: renamed from C39; value 26pF -> 26p
- C39: renamed from C38; value 0.1uF -> 0.1u
- C40: renamed from C41; value 26pF -> 26p
- C41: renamed from C40; value 0.1uF -> 0.1u
- C43: value 10uF -> 10u
- U10: renamed from U13; value TPD4E1U06 -> TPD4E1U06DBV
- U11: renamed from U14; value TPD4E1U06 -> TPD4E1U06DBV
- U12: renamed from U15; value TPD4E1U06 -> TPD4E1U06DBV
- U13: renamed from U16; value TPD4E1U06 -> TPD4E1U06DBV
- U14: renamed from U17; value TPD4E1U06 -> TPD4E1U06DBV
- U15: renamed from U18; value TPD4E1U06 -> TPD4E1U06DBV
- U16: renamed from U19; value TPD4E1U06 -> TPD4E1U06DBV
- U17: renamed from U20; value TPD4E1U06 -> TPD4E1U06DBV
- U8: renamed from U11; value TPD4E1U06 -> TPD4E1U06DBV
- renumbered J6 to J5, J7 to J6, R22 to R19, R23 to R20, R24 to R21, R25 to R22, R26 to R23, R27 to R24, R28 to R25, R29 to R26, R30 to R27, R31 to R28, R32 to R29, R33 to R30, R34 to R31, R35 to R32, R36 to R33, R37 to R34, R38 to R35, R39 to R36, R40 to R37, R41 to R38, R42 to R39, R43 to R40, R44 to R41, R45 to R42, R46 to R43, R47 to R44, R48 to R45, R49 to R46, R50 to R47, R51 to R48, R52 to R49, R53 to R50, R54 to R51, R55 to R52, R56 to R53, R57 to R54, R58 to R55, R59 to R56, R60 to R57, R61 to R58, R62 to R59, TP19 to TP14, TP20 to TP15, TP21 to TP16, TP22 to TP17, TP23 to TP18, TP24 to TP19, TP27 to TP20, TP28 to TP21, TP29 to TP22, TP30 to TP23, TP31 to TP24, TP32 to TP25, TP33 to TP26, TP34 to TP27, TP35 to TP28, TP36 to TP29, TP37 to TP30, TP38 to TP31, TP39 to TP32, TP40 to TP33, TP41 to TP34, TP42 to TP35, TP43 to TP36, TP44 to TP37, TP45 to TP38, TP46 to TP39, TP47 to TP40, TP48 to TP41, TP49 to TP42, TP50 to TP43, TP51 to TP44, TP52 to TP45, TP53 to TP46, TP54 to TP47, TP55 to TP48, TP56 to TP49, TP57 to TP50, TP58 to TP51, TP59 to TP52, U12 to U9
Connections:
- net DGND: now also J4.1 (Pin_1), J4.3 (Pin_3), J4.4 (Pin_4)
- net at U9.3 (AUDIO_L): now also J4.2 (Pin_2)
- net ~GPU_PD renamed ~GPU_PWR_DWN
Other:
- note added: "Audio Header"
- note added: "Resistive Touch Panel FPC Connector"
- note removed: "D.N.P."
- note removed: "Resittive Touch Panel FPC Connector"
- moved on the sheet: C36, C37, C38, C39, C40, C41, C42, C43, C44, D10, D11, D12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
