File: pcb2/croptop_lcd.sch (KiCad schematic (older format))
At the start: 109 parts, among them J4 TSM-102-01-T-DV, J5 686104183422, J6 62684-402100ALF, Q1 BSS138, Q2 BSS138, U10 TPD4E1U06DBV, U11 TPD4E1U06DBV, U12 TPD4E1U06DBV, U13 TPD4E1U06DBV, U14 TPD4E1U06DBV, U15 TPD4E1U06DBV, U16 TPD4E1U06DBV, U17 TPD4E1U06DBV, U8 TPD4E1U06DBV, U9 FT812Q, Y2 ABLS-12.000MHZ-B2-T

Commit message: Footprints done, board started
Parts:
- removed D10, D9: LTSTC171GKT, LED_SMD:LED_0805_2012Metric, symbol Device:LED
- removed Q1, Q2: BSS138, symbol Device:Q_NMOS_GSD
- removed R21, R23, R28, R30: 100, Resistor_SMD:R_0402_1005Metric, symbol Device:R
- removed R22, R29: 10k, Resistor_SMD:R_0402_1005Metric, symbol Device:R
- removed TP16, TP23: TestPoint, symbol Connector:TestPoint
- C38, C40: value 26p -> 27p
- C43: footprint Capacitor_SMD:C_0402_1005Metric -> Capacitor_SMD:C_1206_3216Metric
- D10: renamed from D11; footprint (none) -> Package_TO_SOT_SMD:SOT-323_SC-70
- D11: renamed from D12; footprint (none) -> Diode_SMD:D_0201_0603Metric
- J4: value TSM-102-01-T-DV -> TSM-102-01-L-DV; footprint (none) -> Connector_PinHeader_2.54mm:PinHeader_2x02_P2.54mm_Vertical_SMD
- J5: footprint (none) -> Connector_FFC-FPC:TE_84952-4_1x04-1MP_P1.0mm_Horizontal
- J6: footprint (none) -> Connector_FFC-FPC:Hirose_FH12-40S-0.5SH_1x40-1MP_P0.50mm_Horizontal
- TP13: renamed from TP14; footprint (none) -> croptop:TestPoint
- TP14: renamed from TP15; footprint (none) -> croptop:TestPoint
- TP15: renamed from TP17; footprint (none) -> croptop:TestPoint
- TP16: renamed from TP18; footprint (none) -> croptop:TestPoint
- TP17: renamed from TP19; footprint (none) -> croptop:TestPoint
- TP18: renamed from TP20; footprint (none) -> croptop:TestPoint
- TP19: renamed from TP21; footprint (none) -> croptop:TestPoint
- TP20: renamed from TP22; footprint (none) -> croptop:TestPoint
- TP21: renamed from TP24; footprint (none) -> croptop:TestPoint
- TP22: renamed from TP25; footprint (none) -> croptop:TestPoint
- TP23: renamed from TP26; footprint (none) -> croptop:TestPoint
- TP24: renamed from TP27; footprint (none) -> croptop:TestPoint
- TP25: renamed from TP28; footprint (none) -> croptop:TestPoint
- TP26: renamed from TP29; footprint (none) -> croptop:TestPoint
- TP27: renamed from TP30; footprint (none) -> croptop:TestPoint
- TP28: renamed from TP31; footprint (none) -> croptop:TestPoint
- TP29: renamed from TP32; footprint (none) -> croptop:TestPoint
- TP30: renamed from TP33; footprint (none) -> croptop:TestPoint
- TP31: renamed from TP34; footprint (none) -> croptop:TestPoint
- TP32: renamed from TP35; footprint (none) -> croptop:TestPoint
- TP33: renamed from TP36; footprint (none) -> croptop:TestPoint
- TP34: renamed from TP37; footprint (none) -> croptop:TestPoint
- TP35: renamed from TP38; footprint (none) -> croptop:TestPoint
- TP36: renamed from TP39; footprint (none) -> croptop:TestPoint
- TP37: renamed from TP40; footprint (none) -> croptop:TestPoint
- TP38: renamed from TP41; footprint (none) -> croptop:TestPoint
- TP39: renamed from TP42; footprint (none) -> croptop:TestPoint
- TP40: renamed from TP43; footprint (none) -> croptop:TestPoint
- TP41: renamed from TP44; footprint (none) -> croptop:TestPoint
- TP42: renamed from TP45; footprint (none) -> croptop:TestPoint
- TP43: renamed from TP46; footprint (none) -> croptop:TestPoint
- TP44: renamed from TP47; footprint (none) -> croptop:TestPoint
- TP45: renamed from TP48; footprint (none) -> croptop:TestPoint
- TP46: renamed from TP49; footprint (none) -> croptop:TestPoint
- TP47: renamed from TP50; footprint (none) -> croptop:TestPoint
- TP48: renamed from TP51; footprint (none) -> croptop:TestPoint
- TP49: renamed from TP52; footprint (none) -> croptop:TestPoint
- Y2: footprint (none) -> croptop:ABLS_OX
- renumbered R19 to R20, R20 to R21, R24 to R22, R25 to R23, R26 to R24, R27 to R25, R31 to R26, R32 to R27, R33 to R28, R34 to R29, R35 to R30, R36 to R31, R37 to R32, R38 to R33, R39 to R34, R40 to R35, R41 to R36, R42 to R37, R43 to R38, R44 to R39, R45 to R40, R46 to R41, R47 to R42, R48 to R43, R49 to R44, R50 to R45, R51 to R46, R52 to R47, R53 to R48, R54 to R49, R55 to R50, R56 to R51, R57 to R52, R58 to R53, R59 to R54
Connections:
- net +3V3: now also J4.1 (Pin_1)
- net DGND: no longer J4.1 (Pin_1)
- net GPU_LED_1: no longer names the net of U9.12 (GPIO2)
- net GPU_LED_2: no longer names the net of U9.15 (GPIO3)
- no-connect marks 19 -> 21
Other:
- moved on the sheet: J4, J5, U8

Commit message: Updated prez
Parts:
- U10, U11, U12, U13, U14, U15, U16, U17, U8: footprint (none) -> Package_TO_SOT_SMD:SOT-23-6
Changed lines of the file:
@@
 F 0 "U10" H 9200 8626 50  0000 C CNN
 F 1 "TPD4E1U06DBV" H 9200 8535 50  0000 C CNN
-F 2 "" V 9450 8300 50  0001 C CNN
+F 2 "Package_TO_SOT_SMD:SOT-23-6" V 9450 8300 50  0001 C CNN
 F 3 "http://www.ti.com/lit/ds/symlink/tpd4e1u06.pdf" V 9450 8300 50  0001 C CNN
 	1    9200 8850
@@
 F 0 "U11" H 10050 8626 50  0000 C CNN
 F 1 "TPD4E1U06DBV" H 10050 8535 50  0000 C CNN
-F 2 "" V 10300 8300 50  0001 C CNN
+F 2 "Package_TO_SOT_SMD:SOT-23-6" V 10300 8300 50  0001 C CNN
 F 3 "http://www.ti.com/lit/ds/symlink/tpd4e1u06.pdf" V 10300 8300 50  0001 C CNN
 	1    10050 8850
@@
 F 0 "U12" H 10900 8626 50  0000 C CNN
 F 1 "TPD4E1U06DBV" H 10900 8535 50  0000 C CNN
-F 2 "" V 11150 8300 50  0001 C CNN
+F 2 "Package_TO_SOT_SMD:SOT-23-6" V 11150 8300 50  0001 C CNN
 F 3 "http://www.ti.com/lit/ds/symlink/tpd4e1u06.pdf" V 11150 8300 50  0001 C CNN
 	1    10900 8850
@@
 F 0 "U13" H 11750 8626 50  0000 C CNN
 F 1 "TPD4E1U06DBV" H 11750 8535 50  0000 C CNN
-F 2 "" V 12000 8300 50  0001 C CNN
+F 2 "Package_TO_SOT_SMD:SOT-23-6" V 12000 8300 50  0001 C CNN
 F 3 "http://www.ti.com/lit/ds/symlink/tpd4e1u06.pdf" V 12000 8300 50  0001 C CNN
 	1    11750 8850
@@
 F 0 "U14" H 12600 8626 50  0000 C CNN
 F 1 "TPD4E1U06DBV" H 12600 8535 50  0000 C CNN
-F 2 "" V 12850 8300 50  0001 C CNN
+F 2 "Package_TO_SOT_SMD:SOT-23-6" V 12850 8300 50  0001 C CNN
 F 3 "http://www.ti.com/lit/ds/symlink/tpd4e1u06.pdf" V 12850 8300 50  0001 C CNN
 	1    12600 8850
@@
 F 0 "U15" H 13450 8626 50  0000 C CNN
 F 1 "TPD4E1U06DBV" H 13450 8535 50  0000 C CNN
-F 2 "" V 13700 8300 50  0001 C CNN
+F 2 "Package_TO_SOT_SMD:SOT-23-6" V 13700 8300 50  0001 C CNN
 F 3 "http://www.ti.com/lit/ds/symlink/tpd4e1u06.pdf" V 13700 8300 50  0001 C CNN
 	1    13450 8850
@@
 F 0 "U16" H 14300 8626 50  0000 C CNN
 F 1 "TPD4E1U06DBV" H 14300 8535 50  0000 C CNN
-F 2 "" V 14550 8300 50  0001 C CNN
+F 2 "Package_TO_SOT_SMD:SOT-23-6" V 14550 8300 50  0001 C CNN
 F 3 "http://www.ti.com/lit/ds/symlink/tpd4e1u06.pdf" V 14550 8300 50  0001 C CNN
 	1    14300 8850
@@
 F 0 "U8" H 3600 8526 50  0000 C CNN
 F 1 "TPD4E1U06DBV" H 3600 8435 50  0000 C CNN
-F 2 "" V 3850 8200 50  0001 C CNN
+F 2 "Package_TO_SOT_SMD:SOT-23-6" V 3850 8200 50  0001 C CNN
 F 3 "http://www.ti.com/lit/ds/symlink/tpd4e1u06.pdf" V 3850 8200 50  0001 C CNN
 	1    3600 8750
@@
 F 0 "U17" H 15150 8526 50  0000 C CNN
 F 1 "TPD4E1U06DBV" H 15150 8435 50  0000 C CNN
-F 2 "" V 15400 8200 50  0001 C CNN
+F 2 "Package_TO_SOT_SMD:SOT-23-6" V 15400 8200 50  0001 C CNN
 F 3 "http://www.ti.com/lit/ds/symlink/tpd4e1u06.pdf" V 15400 8200 50  0001 C CNN
 	1    15150 8750

Commit message: Board almost done
Parts:
- removed TP19, TP20, TP21, TP22, TP23, TP24, TP25, TP26, TP27, TP28, TP29, TP30, TP31, TP32, TP33, TP34, TP35, TP36, TP37, TP38, TP39, TP40, TP41, TP42, TP43, TP44, TP45, TP46, TP47, TP48, TP49: TestPoint, croptop:TestPoint, symbol Connector:TestPoint
- J5: footprint Connector_FFC-FPC:TE_84952-4_1x04-1MP_P1.0mm_Horizontal -> croptop:TE_84952-4_1x04-1MP_P1.0mm_Horizontal
- renumbered TP13 to TP10, TP14 to TP11, TP15 to TP12, TP16 to TP13, TP17 to TP14, TP18 to TP15
