File: pcb2/croptop_onboard.sch (KiCad schematic (older format))
At the start: 35 parts

Commit message: Added USB port control
Parts:
- removed C?: 0.1uF, Capacitor_SMD:C_0402_1005Metric, symbol Device:C
- removed R? (x2): 10, Resistor_SMD:R_0402_1005Metric, symbol Device:R
- removed R? (x4): 10k, Resistor_SMD:R_0402_1005Metric, symbol Device:R
- removed SW? (x3): BTN, Button_Switch_SMD:SW_SPST_PTS645, symbol CropTop:SW_Push
- removed TP? (x3): TestPoint_Alt, croptop:TestPoint, symbol Connector:TestPoint_Alt
- removed U?: W25N01GV, croptop:W25N01GV, symbol CropTop:W25N01GV
- added C?: 0.1uF, Capacitor_SMD:C_0402_1005Metric, symbol Device:C
- added C?: 10uF, Capacitor_SMD:C_0402_1005Metric, symbol Device:C
- added C?: 1uF, Capacitor_SMD:C_0402_1005Metric, symbol Device:C
- added D? (x2): LED, LED_SMD:LED_0805_2012Metric, symbol Device:LED
- added J?: MicroSD Card Slot, symbol CropTop:Micro_SD_Card_Det_0
- added R? (x2): 60Ω, symbol Device:R
- added R? (x2): 10kΩ, symbol Device:R
- added R? (x3): 10k, symbol Device:R
- added R?: 10k, Resistor_SMD:R_0402_1005Metric, symbol Device:R
- added R? (x8): 220Ω, symbol Device:R
- added SW? (x3): SW_Push, symbol Switch:SW_Push
- added TP? (x6): TestPoint, symbol Connector:TestPoint
- added U?: TPS22915, symbol CropTop:TPS22915
- added U? (x2): TPD4E1U06, symbol CropTop:TPD4E1U06
Connections:
- net labels added: PMOD_ADC_1, PMOD_ADC_2, PMOD_ADC_3, PMOD_ADC_4, PMOD_CN_1, PMOD_CN_2, PMOD_GPIO_1, PMOD_GPIO_2, PMOD_GPIO_3, PMOD_GPIO_4, PMOD_GPIO_5, PMOD_GPIO_6, PMOD_GPIO_7, PMOD_GPIO_8, PMOD_PWM_1, PMOD_PWM_2, PMOD_RX, PMOD_SCL, PMOD_SDA, PMOD_TX, SDC_CS, SDC_DET, SDC_MISO, SDC_MOSI, SDC_PWR, SDC_SCLK
- net labels removed: MISO, MOSI, NAND_CS, NAND_HOLD, NAND_WP, SCLK
- wire segments 164 -> 206
- no-connect marks 16 -> 20
Other:
- note added: "GNSS Reciever Module"
- note added: "MicroSD Card Interface\n"
- note added: "User Push Buttons and LEDs"
- note removed: "Debugging Buttons and LEDs"
- note removed: "GPS Antenna and Reciever"
- note removed: "NAND Flash Memory\n"
- moved on the sheet: C?, D?, R?, U?

Commit message: Schematic near completion
Parts:
- removed C? (x2): 0.1uF, Capacitor_SMD:C_0402_1005Metric, symbol Device:C
- removed C?: 10uF, Capacitor_SMD:C_0402_1005Metric, symbol Device:C
- removed C?: 1uF, Capacitor_SMD:C_0402_1005Metric, symbol Device:C
- removed D? (x4): LED, LED_SMD:LED_0805_2012Metric, symbol Device:LED
- removed R? (x3): 60, Resistor_SMD:R_0402_1005Metric, symbol Device:R
- removed R?: 60Ω, symbol Device:R
- removed R? (x4): 220Ω, symbol Device:R
- removed R? (x2): 220, Resistor_SMD:R_0402_1005Metric, symbol Device:R
- removed TP? (x5): TestPoint_Alt, croptop:TestPoint, symbol Connector:TestPoint_Alt
- removed TP?: TestPoint, symbol Connector:TestPoint
- removed U?: LIS3DH, Package_LGA:LGA-16_3x3mm_P0.5mm_LayoutBorder3x5y, symbol CropTop:LIS3DH
- removed U?: TPS22915, symbol CropTop:TPS22915
- removed U?: TPD4E1U06, symbol CropTop:TPD4E1U06
- added C? (x8): 10uF, Capacitor_SMD:C_0402_1005Metric, symbol Device:C
- added C? (x4): 0.1uF, Capacitor_SMD:C_0402_1005Metric, symbol Device:C
- added C?: NFM18PC225B1A3D, symbol Device:C_Feedthrough
- added D? (x6): LED, LED_SMD:LED_0805_2012Metric, symbol Device:LED
- added J?: 67997-224HLF, Connector_PinHeader_2.54mm:PinHeader_2x12_P2.54mm_Vertical, symbol Connector_Generic:Conn_02x12_Odd_Even
- added L? (x7): BLM15HD102SN1D, symbol Device:L_Core_Ferrite
- added Q? (x3): BSS138, symbol Device:Q_NMOS_GSD
- added R? (x6): 100, Resistor_SMD:R_0402_1005Metric, symbol Device:R
- added R? (x9): 10k, Resistor_SMD:R_0402_1005Metric, symbol Device:R
- added R? (x16): 220, Resistor_SMD:R_0402_1005Metric, symbol Device:R
- added R? (x3): 60, Resistor_SMD:R_0402_1005Metric, symbol Device:R
- added TP? (x38): TestPoint, symbol Connector:TestPoint
- added U?: ICM-20602, symbol CropTop:ICM-20602
- added U? (x3): AP22802AW5, symbol CropTop:AP22802AW5
- added U?: LIS3DHTR, symbol CropTop:LIS3DHTR
- added U? (x4): TPD4E1U06, symbol CropTop:TPD4E1U06
- J?: value MicroSD Card Slot -> 114-00841-68; Note (none) -> MicroSD
- R?: value 60Ω -> 100; footprint (none) -> Resistor_SMD:R_0402_1005Metric
- R?: value 10kΩ -> 10k; footprint (none) -> Resistor_SMD:R_0402_1005Metric
- R?: value 10kΩ -> 220; footprint (none) -> Resistor_SMD:R_0402_1005Metric
- R? (x3): footprint (none) -> Resistor_SMD:R_0402_1005Metric
- R? (x4): value 220Ω -> 220; footprint (none) -> Resistor_SMD:R_0402_1005Metric
Connections:
- net labels added: +5V, ACCEL_INT1, ACCEL_INT2, GPS_EXTINT, GPS_PPS, GPS_RST, GPS_RX, GPS_TX, IMU_INT, ONBRD_SCL, ONBRD_SDA, PMOD_3V3_FLG, PMOD_5V0_FLG, SDC_PWR_FLG
- net labels removed: GPS_INT, RX, SCL, SDA, SDC_PWR, TX
- wire segments 206 -> 532
- no-connect marks 20 -> 18
Other:
- note added: "I2C ADDRESS: 0011001"
- note added: "I2C ADDRESS: 1000000"
- note added: "I2C ADDRESS: 1000010"
- note added: "I2C ADDRESS: 1101001"
- note added: "Inertial Measurement Unit"
- note added: "Onboard I2C Bus"
- note added: "Peripheral Module Header"
- note added: "Should these rails be software\nor hardware controlled?"
- note removed: "Internal\nADCs"
- note removed: "Interrupts"
- note removed: "Unused\nPins"
- moved on the sheet: C?, D?, J?, R?, SW?, TP?, U?

Commit message: Added pmod
Parts:
- removed R?: 10k, Resistor_SMD:R_0402_1005Metric, symbol Device:R
- added C?: 10uF, Capacitor_SMD:C_0402_1005Metric, symbol Device:C
- added TP? (x3): TestPoint, symbol Connector:TestPoint
- D? (x7): value LED -> LTSTC171GKT
- R? (x3): value 60 -> 100
Connections:
- net labels added: SD_MISO, SD_MOSI, SD_PWR_FLG, SD_SCLK, ~SD_CS
- net labels removed: SDC_CS, SDC_DET, SDC_MISO, SDC_MOSI, SDC_PWR_FLG, SDC_SCLK
- wire segments 532 -> 536
Other:
- note added: "(LEDs are green)"
- note added: "Place on PCB cutout island"
- note added: "User LEDs"
- note added: "User Push Buttons"
- note removed: "Should these rails be software\nor hardware controlled?"
- note removed: "User Push Buttons and LEDs"
- moved on the sheet: C?, D?, J?, R?, TP?, U?

Commit message: pwm
Parts:
- R100, R101, R102, R116, R129, R130, R132, R135, R138, R140, R141, R142, R143, R144, R145: renamed from R?; value 10k -> 10kΩ
- R103, R104, R105, R106, R108, R109, R110, R111, R113, R114, R115, R117, R119, R121, R122, R123, R124, R125, R126, R127, R128: renamed from R?; value 220 -> 220Ω
- R107, R112, R118, R120, R131, R133, R134, R136, R137, R139: renamed from R?; value 100 -> 100Ω
- gave numbers to parts that had none: 96
Other:
- moved on the sheet: R144, R145, SW2, SW3, SW4

Commit message: Added TVS diodes
Parts:
- removed C84: 10uF, Capacitor_SMD:C_0402_1005Metric, symbol Device:C
- removed C85, C86: 0.1uF, Capacitor_SMD:C_0402_1005Metric, symbol Device:C
- removed TP157: TestPoint, symbol Connector:TestPoint
- removed U30: LIS3DHTR, symbol CropTop:LIS3DHTR
- removed U33: ICM-20602, symbol CropTop:ICM-20602
- added U41: LIS3DSHTR, symbol CropTop:LIS3DSHTR
- renumbered C73 to C76, C74 to C77, C75 to C78, C76 to C79, C77 to C80, C78 to C81, C79 to C82, C80 to C83, C81 to C84, C82 to C85, C83 to C86, D15 to D26, D16 to D27, D17 to D28, D18 to D29, D19 to D30, D20 to D31, D21 to D32, J11 to J13, J12 to J14, R100 to R106, R101 to R107, R102 to R108, R103 to R109, R104 to R110, R105 to R111, R106 to R112, R107 to R113, R108 to R114, R109 to R115, R110 to R116, R111 to R117, R112 to R118, R113 to R119, R114 to R120, R115 to R121, R116 to R122, R117 to R123, R118 to R124, R119 to R125, R120 to R126, R121 to R127, R122 to R128, R123 to R129, R124 to R130, R125 to R131, R126 to R132, R127 to R133, R128 to R134, R129 to R135, R130 to R136, R131 to R137, R132 to R138, R133 to R139, R134 to R140, R135 to R141, R136 to R142, R137 to R143, R138 to R144, R139 to R145, R140 to R146, R141 to R147, R142 to R148, R143 to R149, R144 to R150, R145 to R151, TP147 to TP144, TP150 to TP145, TP153 to TP146, TP154 to TP147, TP155 to TP148, TP144 to TP149, TP145 to TP150, TP146 to TP151, TP148 to TP152, TP149 to TP153, TP151 to TP154, TP152 to TP155, U22 to U33, U23 to U34, U24 to U35, U25 to U36, U26 to U37, U27 to U38, U28 to U39, U29 to U40, U31 to U42, U32 to U43
Connections:
- net labels removed: IMU_INT
- wire segments 536 -> 506
- no-connect marks 18 -> 13
Other:
- note removed: "I2C ADDRESS: 1101001"
- note removed: "Inertial Measurement Unit"
- moved on the sheet: C83, C84, C85, C86, C87, C88, L10, L11, L12, L13, L7, L8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

Commit message: Updated pin out
Parts:
- added D33: TPD1E6B06, symbol Device:D_TVS
- added JP? (x2): N.0., symbol Jumper:SolderJumper_2_Open
- R106, R107, R108, R122, R135, R136, R138, R141, R144, R146, R147, R148, R149, R150, R151: value 10kΩ -> 10k
- R109, R110, R111, R112, R114, R115, R116, R117, R119, R120, R121, R123, R125, R127, R128, R129, R130, R131, R132, R133, R134: value 220Ω -> 220
- R113, R118, R124, R126, R137, R139, R140, R142, R143, R145: value 100Ω -> 100
Connections:
- net DGND: now also D33.1 (A1)
- net PMOD_RX: now also JP?.1 (A)
- net PMOD_TX: now also JP?.1 (A)
- net at C80.1, D27.2 (A), J14.4 (VDD)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: now also D33.2 (A2)
- net GPS_RX: no longer names the net of L7.1, TP154.1
- net GPS_RX: now also JP?.2 (B)
- net GPS_TX: no longer names the net of L8.1, TP152.1
- net GPS_TX: now also JP?.2 (B)
Other:
- moved on the sheet: C80, TP127, TP128, TP131, TP133, TP150, TP153, TP154

Commit message: Final Schematic
Parts:
- removed JP? (x2): N.0., symbol Jumper:SolderJumper_2_Open
- removed TP154: TestPoint, symbol Connector:TestPoint
- added JP? (x2): N.0., symbol Jumper:SolderJumper_2_Open
- added R? (x4): 22, Resistor_SMD:R_0402_1005Metric, symbol Device:R
- added TP? (x3): TestPoint, symbol Connector:TestPoint
- U42: value UCAM-M8Q -> CAM-M8C-0
Connections:
- net +3V3: no longer C77.1, U36.3 (FLG)
- net GPS_EXTINT: now also TP153.1; no longer TP151.1
- net GPS_PPS: now also TP?.1; no longer TP155.1
- net ONBRD_SCL: now also TP151.1, TP?.1; no longer TP149.1
- net ONBRD_SDA: now also TP149.1, TP?.1; no longer TP150.1
- net PMOD_RX: now also L7.1, TP152.1
- net PMOD_TX: now also L8.1, TP150.1
- net SD_MISO: now also R?.2; no longer J14.7 (DO/DAT0), TP127.1
- net SD_MOSI: now also R?.2; no longer J14.3 (DI/CMD), TP131.1
- net SD_SCLK: now also R?.2; no longer J14.5 (SCLK), TP128.1
- net ~SD_CS: now also R?.2; no longer J14.2 (CS/DAT3), TP133.1
- net at U42.25 (TXD): now also JP?.2 (B); no longer L7.2
- net at U42.26 (RXD): now also JP?.2 (B); no longer L8.2
- net GPS_RST renamed ~GPS_RST
- net ~GPS_RST: now also TP155.1; no longer TP153.1
- net PMOD_3V3_FLG renamed PMOD_3V3_FAULT
- net PMOD_5V0_FLG renamed PMOD_5V0_FAULT
- net SD_PWR_FLG renamed SD_PWR_FAULT
- new net: J14.5 (SCLK), R?.1, TP128.1
- new net: J14.3 (DI/CMD), R?.1, TP131.1
- new net: J14.2 (CS/DAT3), R?.1, TP133.1
- new net: J14.7 (DO/DAT0), R?.1, TP127.1
- new net: JP?.1 (A), L8.2
- new net: JP?.1 (A), L7.2
- new net: C77.1, U36.3 (FLG)
Other:
- note added: "Onboard I2C Device Bus"
- note added: "Place GPS over uninterrupted ground \nplane and not under screen"
- note added: "Place solder \njumpers as\nclose as \npossible\nto GPS"
- note removed: "Onboard I2C Bus"
- moved on the sheet: C77, C78, C80, C83, C84, C85, C86, C87, C88, D27, D28, D33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

Commit message: Schematic Done
Parts:
- removed TP144, TP145: TestPoint, symbol Connector:TestPoint
- added U35: TPD4E1U06DBV, symbol CropTop:TPD4E1U06
- C76: renamed from C77; value 10uF -> 10u
- C77: renamed from C76; value 10uF -> 10u
- C78, C81, C82, C83, C88: value 10uF -> 10u
- C79: renamed from C80; value 0.1uF -> 0.1u
- C80: renamed from C79; value 10uF -> 10u
- C84, C86, C87: value 0.1uF -> 0.1u
- J15: renamed from J13; value 67997-224HLF -> 0015912240; footprint Connector_PinHeader_2.54mm:PinHeader_2x12_P2.54mm_Vertical -> (none)
- U32: renamed from U34; value TPD4E1U06 -> TPD4E1U06DBV
- U33: renamed from U35; value TPD4E1U06 -> TPD4E1U06DBV
- U34: renamed from U37; value TPD4E1U06 -> TPD4E1U06DBV
- U36: renamed from U38; value TPD4E1U06 -> TPD4E1U06DBV
- U37: renamed from U39; value TPD4E1U06 -> TPD4E1U06DBV
- gave numbers to parts that had none: 9
- renumbered D27 to D26, D26 to D27, D33 to D28, D28 to D29, D29 to D30, D30 to D31, D31 to D32, D32 to D33, J14 to J16, L12 to L10, L13 to L11, L7 to L5, L8 to L6, L9 to L7, L10 to L8, L11 to L9, R108 to R103, R106 to R104, R107 to R105, R118 to R106, R109 to R107, R110 to R108, R111 to R109, R112 to R110, R113 to R111, R114 to R112, R115 to R113, R116 to R114, R117 to R115, R120 to R116, R119 to R117, R122 to R118, R121 to R119, R124 to R120, R123 to R121, R125 to R124, R126 to R127, R127 to R128, R128 to R129, R129 to R130, R130 to R131, R131 to R132, R132 to R133, R133 to R134, R134 to R135, R135 to R136, R136 to R137, R137 to R138, R138 to R139, R139 to R140, R140 to R141, R141 to R142, R142 to R143, R143 to R144, R144 to R145, R145 to R146, R146 to R147, R147 to R148, R148 to R149, R149 to R150, R150 to R151, R151 to R152, TP112 to TP105, TP113 to TP106, TP121 to TP107, TP114 to TP108, TP115 to TP109, TP116 to TP110, TP122 to TP111, TP117 to TP112, TP118 to TP113, TP119 to TP114, TP120 to TP115, TP124 to TP116, TP126 to TP117, TP123 to TP118, TP125 to TP119, TP130 to TP120, TP127 to TP121, TP132 to TP122, TP128 to TP123, TP131 to TP124, TP133 to TP125, TP129 to TP126, TP134 to TP127, TP135 to TP128, TP136 to TP129, TP137 to TP130, TP138 to TP131, TP139 to TP132, TP140 to TP133, TP141 to TP134, TP142 to TP135, TP143 to TP136, TP146 to TP137, TP147 to TP138, TP148 to TP139, TP149 to TP140, TP151 to TP141, TP150 to TP142, TP153 to TP143, TP152 to TP144, TP155 to TP145, TP156 to TP147, U36 to U30, U33 to U31, U40 to U38, U41 to U39, U42 to U40, U43 to U41
Connections:
- net +3V3: now also C76.1, U30.5 (IN)
- net DGND: now also U35.2 (GND)
- net at J16.5 (SCLK), R123.1, TP123.1: now also U35.6 (D1-)
- net at J16.3 (DI/CMD), R125.1, TP124.1: now also U35.3 (D2+)
- net at J16.2 (CS/DAT3), R122.1, TP125.1: now also U35.4 (D2-)
- net at J16.7 (DO/DAT0), R126.1, TP121.1: now also U35.1 (D1+)
- net ~SD_PWR_FAULT: now reaches U30.3 (FLG)
- net ~SD_PWR_FAULT: now also R103.2, TP107.1; no longer C76.1
- net ACCEL_INT1: no longer names the net of U39.11 (INT1)
- net ACCEL_INT2: no longer names the net of U39.9 (INT2)
- net BTN_1 renamed DEBUG_BTN_1
- net BTN_2 renamed DEBUG_BTN_2
- net BTN_3 renamed DEBUG_BTN_3
- net LED_1 renamed DEBUG_LED_1
- net LED_2 renamed DEBUG_LED_2
- net LED_3 renamed DEBUG_LED_3
- net PMOD_3V3_FAULT renamed ~PMOD_3V3_PWR_FAULT
- net PMOD_5V0_FAULT renamed ~PMOD_5V0_PWR_FAULT
- removed net SD_PWR_FAULT: R103.2, TP107.1, U30.5 (IN)
- net ~GPS_RST renamed ~GPS_RESET
- no-connect marks 13 -> 16
Other:
- moved on the sheet: C76, C77, C78, C79, C80, C81, C82, D26, D27, D28, D29, D30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
