File: pcb2/croptop_onboard.sch (KiCad schematic (older format))
At the start: 145 parts, among them J15 0015912240, J16 114-00841-68, Q4 BSS138, Q5 BSS138, Q6 BSS138, SW2 SW_Push, SW3 SW_Push, SW4 SW_Push, U30 AP22802AW5, U31 AP22802AW5, U32 TPD4E1U06DBV, U33 TPD4E1U06DBV, U34 TPD4E1U06DBV, U35 TPD4E1U06DBV, U36 TPD4E1U06DBV, U37 TPD4E1U06DBV, U38 AP22802AW5, U39 LIS3DSHTR, U40 CAM-M8C-0, U41 Si7006-A20

Commit message: Footprints done, board started
Parts:
- removed C85: NFM18PC225B1A3D, symbol Device:C_Feedthrough
- removed D26, D27, D29, D30: LTSTC171GKT, LED_SMD:LED_0805_2012Metric, symbol Device:LED
- removed JP2, JP3: N.0., symbol Jumper:SolderJumper_2_Open
- removed L6: BLM15HD102SN1D, symbol Device:L_Core_Ferrite
- removed R103, R104, R137: 10k, Resistor_SMD:R_0402_1005Metric, symbol Device:R
- removed R106, R111, R120, R127: 100, Resistor_SMD:R_0402_1005Metric, symbol Device:R
- removed TP107, TP108, TP131, TP142, TP144: TestPoint, symbol Connector:TestPoint
- C78: renamed from C76; footprint Capacitor_SMD:C_0402_1005Metric -> Capacitor_SMD:C_1206_3216Metric
- C79: renamed from C77; footprint Capacitor_SMD:C_0402_1005Metric -> Capacitor_SMD:C_1206_3216Metric
- C80: renamed from C78; footprint Capacitor_SMD:C_0402_1005Metric -> Capacitor_SMD:C_1206_3216Metric
- C82: renamed from C80; footprint Capacitor_SMD:C_0402_1005Metric -> Capacitor_SMD:C_1206_3216Metric
- C83: renamed from C81; footprint Capacitor_SMD:C_0402_1005Metric -> Capacitor_SMD:C_1206_3216Metric
- C84: renamed from C82; footprint Capacitor_SMD:C_0402_1005Metric -> Capacitor_SMD:C_1206_3216Metric
- C85: renamed from C83; footprint Capacitor_SMD:C_0402_1005Metric -> Capacitor_SMD:C_1206_3216Metric
- C90: renamed from C88; footprint Capacitor_SMD:C_0402_1005Metric -> Capacitor_SMD:C_1206_3216Metric
- D21: renamed from D28; footprint (none) -> Diode_SMD:D_0201_0603Metric
- D22: renamed from D31; value LTSTC171GKT -> LTSTC190KGKT; footprint LED_SMD:LED_0805_2012Metric -> LED_SMD:LED_0603_1608Metric
- D23: renamed from D32; value LTSTC171GKT -> LTSTC190KGKT; footprint LED_SMD:LED_0805_2012Metric -> LED_SMD:LED_0603_1608Metric
- D24: renamed from D33; value LTSTC171GKT -> LTSTC190KGKT; footprint LED_SMD:LED_0805_2012Metric -> LED_SMD:LED_0603_1608Metric
- J15: value 0015912240 -> TSM-112-01-L-DV; footprint (none) -> Connector_PinHeader_2.54mm:PinHeader_2x12_P2.54mm_Vertical_SMD
- J16: value 114-00841-68 -> DM3D-SF; footprint (none) -> Connector_Card:microSD_HC_Hirose_DM3D-SF
- L10, L11, L7, L8, L9: footprint (none) -> Inductor_SMD:L_0402_1005Metric
- L5: value BLM15HD102SN1D -> BKP1005HS121; footprint (none) -> Inductor_SMD:L_0402_1005Metric
- Q4, Q5, Q6: footprint (none) -> Package_TO_SOT_SMD:SOT-23
- SW2, SW3, SW4: footprint (none) -> Button_Switch_SMD:SW_SPST_PTS645
- TP100: renamed from TP106; footprint (none) -> croptop:TestPoint
- TP101: renamed from TP109; footprint (none) -> croptop:TestPoint
- TP102: renamed from TP110; footprint (none) -> croptop:TestPoint
- TP103: renamed from TP112; footprint (none) -> croptop:TestPoint
- TP104: renamed from TP113; footprint (none) -> croptop:TestPoint
- TP105: renamed from TP114; footprint (none) -> croptop:TestPoint
- TP106: renamed from TP115; footprint (none) -> croptop:TestPoint
- TP107: renamed from TP111; footprint (none) -> croptop:TestPoint
- TP108: renamed from TP117; footprint (none) -> croptop:TestPoint
- TP109: renamed from TP116; footprint (none) -> croptop:TestPoint
- TP110: renamed from TP118; footprint (none) -> croptop:TestPoint
- TP111: renamed from TP119; footprint (none) -> croptop:TestPoint
- TP112: renamed from TP120; footprint (none) -> croptop:TestPoint
- TP113: renamed from TP121; footprint (none) -> croptop:TestPoint
- TP114: renamed from TP122; footprint (none) -> croptop:TestPoint
- TP115: renamed from TP123; footprint (none) -> croptop:TestPoint
- TP116: renamed from TP126; footprint (none) -> croptop:TestPoint
- TP117: renamed from TP124; footprint (none) -> croptop:TestPoint
- TP118: renamed from TP125; footprint (none) -> croptop:TestPoint
- TP119: renamed from TP127; footprint (none) -> croptop:TestPoint
- TP120: renamed from TP128; footprint (none) -> croptop:TestPoint
- TP121: renamed from TP129; footprint (none) -> croptop:TestPoint
- TP122: renamed from TP130; footprint (none) -> croptop:TestPoint
- TP123: renamed from TP132; footprint (none) -> croptop:TestPoint
- TP124: renamed from TP133; footprint (none) -> croptop:TestPoint
- TP125: renamed from TP134; footprint (none) -> croptop:TestPoint
- TP126: renamed from TP135; footprint (none) -> croptop:TestPoint
- TP127: renamed from TP136; footprint (none) -> croptop:TestPoint
- TP128: renamed from TP137; footprint (none) -> croptop:TestPoint
- TP129: renamed from TP138; footprint (none) -> croptop:TestPoint
- TP130: renamed from TP139; footprint (none) -> croptop:TestPoint
- TP131: renamed from TP140; footprint (none) -> croptop:TestPoint
- TP132: renamed from TP141; footprint (none) -> croptop:TestPoint
- TP134: renamed from TP143; footprint (none) -> croptop:TestPoint
- TP136: renamed from TP145; footprint (none) -> croptop:TestPoint
- TP137: renamed from TP146; footprint (none) -> croptop:TestPoint
- TP138: renamed from TP147; footprint (none) -> croptop:TestPoint
- TP139: renamed from TP148; footprint (none) -> croptop:TestPoint
- TP140: renamed from TP149; footprint (none) -> croptop:TestPoint
- TP99: renamed from TP105; footprint (none) -> croptop:TestPoint
- U32: renamed from U30; footprint (none) -> Package_TO_SOT_SMD:SOT-23-5
- U33: renamed from U31; footprint (none) -> Package_TO_SOT_SMD:SOT-23-5
- U36: renamed from U38; footprint (none) -> Package_TO_SOT_SMD:SOT-23-5
- renumbered C79 to C81, C84 to C86, C86 to C88, C87 to C89, R117 to R100, R118 to R101, R119 to R102, R121 to R103, R122 to R104, R123 to R105, R124 to R106, R125 to R107, R126 to R108, R128 to R109, R129 to R110, R130 to R111, R131 to R112, R132 to R113, R133 to R114, R134 to R115, R135 to R116, R136 to R117, R138 to R118, R139 to R119, R140 to R120, R141 to R121, R142 to R122, R143 to R123, R144 to R124, R145 to R125, R146 to R126, R147 to R127, R148 to R128, R149 to R129, R150 to R130, R151 to R131, R152 to R132, R105 to R90, R107 to R91, R108 to R92, R109 to R93, R110 to R94, R112 to R95, R113 to R96, R114 to R97, R115 to R98, R116 to R99, U32 to U30, U33 to U31, U36 to U37, U37 to U38
Connections:
- net ~PMOD_5V0_PWR_FAULT is gone; now on net ~PWR_FAULT: U36.3 (FLG)
- net ~SD_PWR_FAULT is gone; now on net ~PWR_FAULT: U32.3 (FLG)
- net +3V3: now also L5.1
- net ONBRD_SCL: now also TP131.1; no longer TP132.1
- net ONBRD_SDA: now also TP132.1; no longer TP131.1
- net PMOD_RX: no longer L5.1
- net at C88.1, U40.1 (VCC_IO), U40.8 (V_BCKP)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: now also L5.2
- net ~PMOD_3V3_PWR_FAULT renamed ~PWR_FAULT
- no-connect marks 16 -> 18
Other:
- note removed: "Place solder \njumpers as\nclose as \npossible\nto GPS"
- moved on the sheet: C78, C79, C84, C88, L10, L11, L7, L8, L9, R117, R90, TP107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

Commit message: Updated prez
Parts:
- U30, U31, U34, U35, U37, U38: footprint (none) -> Package_TO_SOT_SMD:SOT-23-6
- U39: footprint (none) -> croptop:LISDR
Changed lines of the file:
@@
 F 0 "U30" H 2550 6476 50  0000 C CNN
 F 1 "TPD4E1U06DBV" H 2550 6385 50  0000 C CNN
-F 2 "" V 2800 6150 50  0001 C CNN
+F 2 "Package_TO_SOT_SMD:SOT-23-6" V 2800 6150 50  0001 C CNN
 F 3 "http://www.ti.com/lit/ds/symlink/tpd4e1u06.pdf" V 2800 6150 50  0001 C CNN
 	1    2550 6700
@@
 F 0 "U31" H 2550 8526 50  0000 C CNN
 F 1 "TPD4E1U06DBV" H 2550 8435 50  0000 C CNN
-F 2 "" V 2800 8200 50  0001 C CNN
+F 2 "Package_TO_SOT_SMD:SOT-23-6" V 2800 8200 50  0001 C CNN
 F 3 "http://www.ti.com/lit/ds/symlink/tpd4e1u06.pdf" V 2800 8200 50  0001 C CNN
 	1    2550 8750
@@
 F 0 "U38" H 6550 8526 50  0000 C CNN
 F 1 "TPD4E1U06DBV" H 6550 8435 50  0000 C CNN
-F 2 "" V 6800 8200 50  0001 C CNN
+F 2 "Package_TO_SOT_SMD:SOT-23-6" V 6800 8200 50  0001 C CNN
 F 3 "http://www.ti.com/lit/ds/symlink/tpd4e1u06.pdf" V 6800 8200 50  0001 C CNN
 	1    6550 8750
@@
 F 0 "U34" H 4550 9626 50  0000 C CNN
 F 1 "TPD4E1U06DBV" H 4550 9535 50  0000 C CNN
-F 2 "" V 4800 9300 50  0001 C CNN
+F 2 "Package_TO_SOT_SMD:SOT-23-6" V 4800 9300 50  0001 C CNN
 F 3 "http://www.ti.com/lit/ds/symlink/tpd4e1u06.pdf" V 4800 9300 50  0001 C CNN
 	1    4550 9850
@@
 F 0 "U37" H 6550 6476 50  0000 C CNN
 F 1 "TPD4E1U06DBV" H 6550 6385 50  0000 C CNN
-F 2 "" V 6800 6150 50  0001 C CNN
+F 2 "Package_TO_SOT_SMD:SOT-23-6" V 6800 6150 50  0001 C CNN
 F 3 "http://www.ti.com/lit/ds/symlink/tpd4e1u06.pdf" V 6800 6150 50  0001 C CNN
 	1    6550 6700
@@
 F 0 "U39" H 10950 2917 50  0000 C CNN
 F 1 "LIS3DSHTR" H 10950 2826 50  0000 C CNN
-F 2 "" H 10850 1900 50  0001 C CNN
+F 2 "croptop:LISDR" H 10850 1900 50  0001 C CNN
 F 3 "https://www.st.com/content/ccc/resource/technical/document/datasheet/23/c3/ea/bf/8f/d9/41/df/DM00040962.pdf/files/DM00040962.pdf/jcr:content/translations/en.DM00040962.pdf" H 10850 1900 50  0001 C CNN
 	1    10950 2300
@@
 F 0 "U35" H 5800 2576 50  0000 C CNN
 F 1 "TPD4E1U06DBV" H 5800 2485 50  0000 C CNN
-F 2 "" V 6050 2250 50  0001 C CNN
+F 2 "Package_TO_SOT_SMD:SOT-23-6" V 6050 2250 50  0001 C CNN
 F 3 "http://www.ti.com/lit/ds/symlink/tpd4e1u06.pdf" V 6050 2250 50  0001 C CNN
 	1    5800 2800

Commit message: Board almost done
Parts:
- removed TP100, TP101, TP102, TP103, TP104, TP105, TP106, TP109, TP110, TP111, TP112, TP114, TP116, TP119, TP120, TP121, TP122, TP123, TP124, TP125, TP126, TP127, TP130, TP138, TP99: TestPoint, croptop:TestPoint, symbol Connector:TestPoint
- renumbered C88 to C87, C89 to C88, C90 to C89, L5 to L10, L7 to L5, L8 to L6, L9 to L7, L10 to L8, L11 to L9, R102 to R100, R103 to R101, R104 to R102, R105 to R103, R106 to R104, R107 to R105, R108 to R106, R109 to R107, R110 to R108, R111 to R109, R112 to R110, R113 to R111, R114 to R112, R115 to R113, R116 to R114, R117 to R115, R118 to R116, R119 to R117, R120 to R118, R121 to R119, R122 to R120, R123 to R121, R124 to R122, R125 to R123, R126 to R124, R127 to R125, R128 to R126, R129 to R127, R130 to R128, R131 to R129, R132 to R130, R90 to R88, R91 to R89, R92 to R90, R93 to R91, R94 to R92, R95 to R93, R96 to R94, R97 to R95, R98 to R96, R99 to R97, R100 to R98, R101 to R99, TP107 to TP58, TP108 to TP59, TP113 to TP60, TP115 to TP61, TP117 to TP62, TP118 to TP63, TP128 to TP64, TP129 to TP65, TP131 to TP66, TP134 to TP67, TP132 to TP68, TP136 to TP69, TP137 to TP70, TP139 to TP71, TP140 to TP72
