File: pcb2/croptop_mcu.sch (KiCad schematic (older format))
At the start: 91 parts

Commit message: Schematic Done
Parts:
- added C14, C35: 0.1u, Capacitor_SMD:C_0402_1005Metric, symbol Device:C
- added D5: TPD1E6B06, symbol Device:D_TVS
- added TP1, TP2: TestPoint, symbol Connector:TestPoint
- C1, C11, C13, C18, C19, C20, C21, C24, C25, C26, C28, C30, C31, C32: renamed from C?; value 10uF -> 10u
- C10, C15, C2, C22, C23, C27, C29, C3, C33, C4, C5, C6, C7, C8: renamed from C?; value 0.1uF -> 0.1u
- C12, C9: renamed from C?; value 26pF -> 26p
- C16, C17, C34: renamed from C?; value 100uF -> 100u
- D4: renamed from D?; footprint croptop:D_SOD-123 -> (none)
- J1: renamed from J?; value 68000-206HLF -> TSM-106-01-T-SV
- J2: renamed from J?; value 10118193-0001LF -> 10118194-0001LF; Note (none) -> microUSB B
- J3: renamed from J?; value USB-A1HSW6 -> 87583-3010RPALF
- L2: renamed from L?; value 4.7uH -> 4.7u; footprint Inductor_SMD:L_1210_3225Metric -> (none)
- L3: renamed from L?; value 2.2uH -> 2.2u
- U3: renamed from U?; value REG71055 -> REG71055DDC
- U4: renamed from U?; value TPS61169 -> TPS61169DCK
- U5: renamed from U?; value TPS62131 -> TPS62131RGT
- U6: renamed from U?; value TPS70950 -> TPS70950DBV
- U7: renamed from U?; value TPD4E1U06 -> TPD4E1U06DBV
- gave numbers to parts that had none: 46
Connections:
- net PKT_MCLR is gone; now on net PICKIT_MCLR: C15.1, J1.1 (Pin_1), R5.2, SW1.1, TP3.1
- net PKT_PGEC is gone; now on net PICKIT_PGEC: J1.5 (Pin_5)
- net PKT_PGED is gone; now on net PICKIT_PGED: J1.4 (Pin_4)
- net +3V3: now also U1.55 (VUSB3V3)
- net ADI_MISO: now also U1.9 (SDI1)
- net ADI_MOSI: now also U1.72 (SDO1)
- net ADI_SCLK: now also U1.70 (SCK1)
- net CONFIG_ADC: now also U1.32 (AN8)
- net DC_PWM_1: now also U1.76 (OC2)
- net DC_PWM_2: now also U1.77 (OC3)
- net DGND: now also C14.2, C35.1, D5.2 (A2); no longer J2.6 (Shield), J3.5 (Shield)
- net ENCDR_A: now also U1.68 (IC1)
- net ENCDR_B: now also U1.69 (IC2)
- net GPS_EXTINT: now also U1.7 (RC2)
- net GPS_PPS: now also U1.79 (IC5)
- net GPU_MISO: now also U1.11 (SDI2)
- net GPU_MOSI: now also U1.12 (SDO2)
- net GPU_SCLK: now also U1.10 (SCK2)
- net ONBRD_SCL: now also R3.2, U1.66 (SCL1)
- net ONBRD_SDA: now also R4.2, U1.67 (SDA1)
- net PICKIT_MCLR: now also U1.13 (~MCLR)
- net PICKIT_PGEC: now also U1.26 (PGEC2)
- net PICKIT_PGED: now also U1.27 (PGED2)
- net PMOD_ADC_1: now also U1.35 (AN11)
- net PMOD_ADC_2: now also U1.41 (AN12)
- net PMOD_ADC_3: now also U1.42 (AN13)
- net PMOD_ADC_4: now also U1.43 (AN14)
- net PMOD_CN_1: now also U1.84 (CN16)
- net PMOD_CN_2: now also U1.80 (CN19)
- net PMOD_GPIO_1: now also U1.93 (RE0)
- net PMOD_GPIO_2: now also U1.94 (RE1)
- net PMOD_GPIO_3: now also U1.95 (RG14)
- net PMOD_GPIO_4: now also U1.96 (RG12)
- net PMOD_GPIO_5: now also U1.97 (RG13)
- net PMOD_GPIO_6: now also U1.98 (RE2)
- net PMOD_GPIO_7: now also U1.99 (RE3)
- net PMOD_GPIO_8: now also U1.100 (RE4)
- net PMOD_PWM_1: now also U1.78 (OC4)
- net PMOD_PWM_2: now also U1.81 (OC5)
- net PMOD_RX: now also U1.49 (U2RX)
- net PMOD_SCL: now also R1.2, U1.58 (SCL2)
- net PMOD_SDA: now also R2.2, U1.59 (SDA2)
- net PMOD_TX: now also U1.50 (U2TX)
- net SD_MISO: now also U1.52 (SDI3)
- net SD_MOSI: now also U1.53 (SDO3)
- net SD_SCLK: now also U1.48 (SCK3)
- net SONIC_ECHO: now also U1.71 (IC4)
- net SONIC_TRIG: now also U1.6 (RC1)
- net STEP_DECAY: now also U1.40 (RF12)
- net STEP_DIR: now also U1.39 (RF13)
- net STEP_MODE0: now also U1.28 (RA9)
- net STEP_MODE1: now also U1.29 (RA10)
- net STEP_MODE2: now also U1.38 (RA1)
- net STEP_STEP: now also U1.17 (RA0)
- net USB_D+: now also U1.57 (D+)
- net USB_D-: now also U1.56 (D-)
- net USB_PWR_EN: now also R10.1, U1.20 (VBUSON), U2.4 (EN)
- net ~ADI_PWR_FAULT: now also U1.74 (SOSCO)
- net ~DC_FAULT: now also U1.18 (INT1)
- net ~ENCDR_PWR_FAULT: now also U1.23 (CN4)
- net ~GPS_RESET: now also U1.8 (RC3)
- net ~GPU_INT: now also U1.82 (CN14)
- net ~GPU_PWR_DWN: now also U1.5 (RE7)
- net ~PMOD_3V3_PWR_FAULT: now also U1.21 (CN6)
- net ~PMOD_5V0_PWR_FAULT: now also U1.44 (CN12)
- net ~POTEN_PWR_FAULT: now also U1.24 (CN3)
- net ~SD_PWR_FAULT: now also U1.25 (CN2)
- net ~SONIC_PWR_FAULT: now also U1.22 (CN5)
- net ~STEP_ENBL: now also U1.14 (RG9)
- net ~STEP_FAULT: now also U1.19 (INT2)
- net ~STEP_HOME: now also U1.83 (CN15)
- net ~STEP_RESET: now also U1.60 (RA4)
- net ~STEP_SLEEP: now also U1.47 (RD14)
- net ~USB_PWR_FAULT: now also R9.2, TP6.1, U1.73 (SOSCI), U2.3 (FLG)
- net USB_PWR_SENSE: now reaches C26.1, C27.1, D3.2 (A), J3.1 (VBUS), TP8.1, U2.1 (OUT)
- net USB_PWR_SENSE: now also U1.54 (VBUS), D5.1 (A1)
- net ~ADI_CS: now reaches U1.1 (RG15)
- net ~SD_CS: now reaches U1.3 (RE5)
- net POTEN_ADC_1: now reaches U1.33 (AN9)
- net POTEN_ADC_2: now reaches U1.34 (AN10)
- net ~GPU_CS: now reaches U1.4 (RE6)
- net at C12.1, U1.63 (OSC1), Y1.1: now also TP2.1
- net at C9.1, U1.64 (OSC2), Y1.2: now also TP1.1
- net DEBUG_LED_3: now reaches U1.87 (RF0)
- net DEBUG_LED_2: now reaches U1.88 (RF1)
- net DEBUG_LED_1: now reaches U1.89 (RG1)
- net DEBUG_BTN_3: now reaches U1.90 (RG0)
- net DEBUG_BTN_2: now reaches U1.91 (RA6)
- net DEBUG_BTN_1: now reaches U1.92 (RA7)
- new net: C14.1, J2.6 (Shield)
- new net: C35.2, J3.5 (Shield)
Other:
- note added: "Analog Plane; see ADI ADC note"
- note added: "Cart: 10K\nPusher: 10K\nStabber: DNP"
- note added: "Cart: DNP\nPusher: 10K\nStabber: 10K"
- note added: "Dimming control;\nWill put driver into\nsleep mode if low \nfor >2.5ms"
- note added: "PIC32 Microcontroller Power Pins"
- note removed: "Cart: 10K\nPusher: 10K\nStabber: 2K"
- note removed: "Cart: 2K\nPusher: 10K\nStabber: 10K"
- note removed: "Ensure return currents are local"
- moved on the sheet: C1, C10, C11, C12, C13, C15, C16, C17, C18, C19, C2, C20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

Commit message: Footprints done, board started
Parts:
- removed D3: LTSTC171GKT, LED_SMD:LED_0805_2012Metric, symbol Device:LED
- removed R12: 100, Resistor_SMD:R_0402_1005Metric, symbol Device:R
- removed R9: 10k, Resistor_SMD:R_0402_1005Metric, symbol Device:R
- removed TP6: TestPoint, symbol Connector:TestPoint
- added D1: LTSTC190KGKT, LED_SMD:LED_0603_1608Metric, symbol Device:LED
- added D2: LTSTC190KRKT, LED_SMD:LED_0603_1608Metric, symbol Device:LED
- added F1: MF-NSMF110, croptop:Bourns_Fuse, symbol Device:Polyfuse
- added Q1: BSS138, Package_TO_SOT_SMD:SOT-23, symbol Device:Q_NMOS_GSD
- added Q2: BSS84, Package_TO_SOT_SMD:SOT-23, symbol Device:Q_PMOS_GSD
- added R1: 10k, Resistor_SMD:R_0402_1005Metric, symbol Device:R
- added R2, R3: 100, Resistor_SMD:R_0402_1005Metric, symbol Device:R
- C1, C20, C21, C24, C25, C26, C28, C31, C32: footprint Capacitor_SMD:C_0402_1005Metric -> Capacitor_SMD:C_1206_3216Metric
- C10: renamed from C11; footprint Capacitor_SMD:C_0402_1005Metric -> Capacitor_SMD:C_1206_3216Metric
- C11: renamed from C9; value 26p -> 27p
- C12: renamed from C13; footprint Capacitor_SMD:C_0402_1005Metric -> Capacitor_SMD:C_1206_3216Metric
- C13: renamed from C12; value 26p -> 27p
- C18: renamed from C19; footprint Capacitor_SMD:C_0402_1005Metric -> Capacitor_SMD:C_1206_3216Metric
- C19: renamed from C18; footprint Capacitor_SMD:C_0402_1005Metric -> Capacitor_SMD:C_1206_3216Metric
- C29: Rating (none) -> 16V
- C30: footprint Capacitor_SMD:C_0402_1005Metric -> Capacitor_SMD:C_1206_3216Metric; Rating (none) -> 16V
- D3: renamed from D1; footprint (none) -> Diode_SMD:D_0201_0603Metric
- D4: renamed from D2; value LTSTC171GKT -> LTSTC190KGKT; footprint LED_SMD:LED_0805_2012Metric -> LED_SMD:LED_0603_1608Metric
- D5: renamed from D4; footprint (none) -> Diode_SMD:D_SMA
- D6: renamed from D5; footprint (none) -> Diode_SMD:D_0201_0603Metric
- D7: renamed from D6; value LTSTC171GKT -> LTSTC190KGKT; footprint LED_SMD:LED_0805_2012Metric -> LED_SMD:LED_0603_1608Metric
- D8: renamed from D7; value LTSTC171GKT -> LTSTC190KGKT; footprint LED_SMD:LED_0805_2012Metric -> LED_SMD:LED_0603_1608Metric
- D9: renamed from D8; value LTSTC171GKT -> LTSTC190KGKT; footprint LED_SMD:LED_0805_2012Metric -> LED_SMD:LED_0603_1608Metric
- J1: value TSM-106-01-T-SV -> TSM-106-01-L-SV; footprint (none) -> Connector_PinHeader_2.54mm:PinHeader_1x06_P2.54mm_Vertical_SMD_Pin1Right
- L1: footprint (none) -> Inductor_SMD:L_0402_1005Metric
- L2, L3: footprint (none) -> Inductor_SMD:L_Bourns_SRN6045TA
- SW1: footprint (none) -> Button_Switch_SMD:SW_SPST_PTS645
- TP1, TP2, TP3, TP4, TP5: footprint (none) -> croptop:TestPoint
- TP10: renamed from TP11; footprint (none) -> croptop:TestPoint
- TP11: renamed from TP12; footprint (none) -> croptop:TestPoint
- TP12: renamed from TP13; footprint (none) -> croptop:TestPoint
- TP6: renamed from TP7; footprint (none) -> croptop:TestPoint
- TP7: renamed from TP9; footprint (none) -> croptop:TestPoint
- TP8: renamed from TP10; footprint (none) -> croptop:TestPoint
- TP9: renamed from TP8; footprint (none) -> croptop:TestPoint
- U3: renamed from U2; footprint (none) -> Package_TO_SOT_SMD:SOT-23-5
- renumbered C10 to C9, R7 to R10, R8 to R11, R11 to R12, R10 to R13, R13 to R14, R14 to R15, R15 to R16, R16 to R17, R17 to R18, R18 to R19, R1 to R4, R2 to R5, R3 to R6, R4 to R7, R5 to R8, R6 to R9, U3 to U2
Connections:
- net +3V3: now also Q2.2 (S), R1.1, R2.2
- net +5V: now also F1.1; no longer D3.1 (A1), J2.1 (VBUS)
- net DGND: now also Q1.2 (S), R3.2
- net ~ADI_PWR_FAULT: no longer names the net of U1.74 (SOSCO)
- net ~ENCDR_PWR_FAULT: no longer names the net of U1.23 (CN4)
- net ~PMOD_3V3_PWR_FAULT: no longer names the net of U1.21 (CN6)
- net ~PMOD_5V0_PWR_FAULT: no longer names the net of U1.44 (CN12)
- net ~POTEN_PWR_FAULT: no longer names the net of U1.24 (CN3)
- net ~SD_PWR_FAULT: no longer names the net of U1.25 (CN2)
- net ~SONIC_PWR_FAULT: no longer names the net of U1.22 (CN5)
- net ~USB_PWR_FAULT renamed ~PWR_FAULT
- net ~PWR_FAULT: now also Q1.1 (G), Q2.1 (G), R1.2
- new net: D3.1 (A1), F1.2, J2.1 (VBUS)
- new net: D1.1 (K), Q1.3 (D)
- new net: D1.2 (A), R2.1
- new net: D2.2 (A), Q2.3 (D)
- new net: D2.1 (K), R3.1
- no-connect marks 10 -> 17
Other:
- note added: "Power Good: Green LED On/Red LED Off\nPower Fault: Green LED Off/Red LED On"
- note added: "SRN6045TA-2R2Y"
- note removed: "SRN8040-2R2Y"
- moved on the sheet: C11, C13, C14, C16, C17, C18, C19, C20, C21, C22, C23, C24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

Commit message: Updated prez
Parts:
- J2: value 10118194-0001LF -> 10118192-0001LF; footprint croptop:USB_Micro-B_Molex_47346-0001 -> Connector_USB:USB_Micro-B_Molex_47346-0001
- U7: footprint (none) -> Package_TO_SOT_SMD:SOT-23-6
Changed lines of the file:
@@
 AR Path="/64809F0C/5CB340CB" Ref="J?"  Part="1"
 AR Path="/64807BBC/5CB340CB" Ref="J2"  Part="1"
-F 0 "J2" H 7975 2550 50  0000 R CNN
-F 1 "10118194-0001LF" H 8300 2450 50  0000 R CNN
-F 2 "croptop:USB_Micro-B_Molex_47346-0001" H 8100 2050 50  0001 C CNN
+F 0 "J2" H 8000 2550 50  0000 R CNN
+F 1 "10118192-0001LF" H 8300 2450 50  0000 R CNN
+F 2 "Connector_USB:USB_Micro-B_Molex_47346-0001" H 8100 2050 50  0001 C CNN
 F 3 "https://www.amphenol-icc.com/media/wysiwyg/files/drawing/10118194.pdf" H 8100 2050 50  0001 C CNN
 F 4 "microUSB B" H 200 0   50  0001 C CNN "Note"
@@
 F 0 "U7" H 13950 8526 50  0000 C CNN
 F 1 "TPD4E1U06DBV" H 13950 8435 50  0000 C CNN
-F 2 "" V 14200 8200 50  0001 C CNN
+F 2 "Package_TO_SOT_SMD:SOT-23-6" V 14200 8200 50  0001 C CNN
 F 3 "http://www.ti.com/lit/ds/symlink/tpd4e1u06.pdf" V 14200 8200 50  0001 C CNN
 	1    13950 8750

Commit message: Board almost done
Parts:
- removed C4: 0.1u, Capacitor_SMD:C_0402_1005Metric, symbol Device:C
- removed TP1, TP2, TP3: TestPoint, croptop:TestPoint, symbol Connector:TestPoint
- H1, H2, H3, H4: value 4mm Mounting Hole -> 3mm; footprint MountingHole:MountingHole_4mm_Pad -> MountingHole:MountingHole_3mm_Pad_Via
- J2: value 10118192-0001LF -> 0473460001
- J3: value 87583-3010RPALF -> 87583-2010BLF; footprint croptop:USB_A_Assmann_Horizontal -> croptop:87583-2010BLF
- U1: footprint digikey-footprints:TQFP-100_12x12mm -> Package_QFP:TQFP-100_12x12mm_P0.4mm
- U4: footprint (none) -> Package_TO_SOT_SMD:SOT-353_SC-70-5
- U6: footprint (none) -> Package_TO_SOT_SMD:SOT-23-5
- renumbered C19 to C18, C18 to C19, C26 to C25, C25 to C26, R13 to R12, R12 to R13, TP4 to TP1, TP5 to TP2, TP6 to TP3, TP7 to TP4, TP9 to TP5, TP8 to TP6, TP10 to TP7, TP11 to TP8, TP12 to TP9
Connections:
- net +3V3: no longer C18.1, U3.5 (IN)
- net +5V: now also C18.1, U3.5 (IN)
Other:
- note removed: "Pin 30"
- note removed: "Pin 31\n"
- moved on the sheet: C1, C2, C3

Commit message: Finished PCB
Parts:
- added C4, C90: 12.5p, Capacitor_SMD:C_0402_1005Metric, symbol Device:C
- added Y3: ABS07-32.768KHZ-1-T, croptop:ABLS_SEC, symbol Device:Crystal
Connections:
- net ADI_MISO: now also U1.52 (SDI3); no longer U1.9 (SDI1)
- net ADI_MOSI: now also U1.53 (SDO3); no longer U1.72 (SDO1)
- net ADI_SCLK: now also U1.48 (SCK3); no longer U1.70 (SCK1)
- net DGND: now also C4.2, C90.2
- net GPU_MISO: now also U1.9 (SDI1); no longer U1.11 (SDI2)
- net GPU_MOSI: now also U1.72 (SDO1); no longer U1.12 (SDO2)
- net GPU_SCLK: now also U1.70 (SCK1); no longer U1.10 (SCK2)
- net POTEN_ADC_1: now also U1.34 (AN10); no longer U1.33 (AN9)
- net POTEN_ADC_2: now also U1.33 (AN9); no longer U1.34 (AN10)
- net SD_MISO: now also U1.11 (SDI2); no longer U1.52 (SDI3)
- net SD_MOSI: now also U1.12 (SDO2); no longer U1.53 (SDO3)
- net SD_SCLK: now also U1.10 (SCK2); no longer U1.48 (SCK3)
- net ~ADI_CS: now also U1.51 (USBID); no longer U1.1 (RG15)
- net ~GPU_CS: now also U1.61 (RA5); no longer U1.4 (RE6)
- net ~PWR_FAULT: no longer U1.73 (SOSCI)
- net at U1.44 (CN12): now also D2.2 (A), Q2.3 (D)
- net at U1.74 (SOSCO): now also C90.1, Y3.2
- new net: C4.1, U1.73 (SOSCI), Y3.1
- no-connect marks 17 -> 14
Other:
- moved on the sheet: C11, C13, D1, D2, Q1, Q2, R1, R2, R3, R4, R5, R6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
