File: pcb1/croptop_io.sch (KiCad schematic (older format))
At the start: 57 parts, among them J5 Terminal Block, J6 DNP, J7 DNP, U10 AD7799, U11 74HCT125D, U17 DT6250-06MR-13, U18 PUSBM5V5X4, U8 74HCT125D, U9 DRV8872

Commit message: Updated prez
Parts:
- gave numbers to parts that had none: 1
Changed lines of the file:
@@
 P 1150 3550
 AR Path="/64809F0C/5C632DBE" Ref="TP?"  Part="1"
-AR Path="/669AB112/5C632DBE" Ref="TP?"  Part="1"
-F 0 "TP?" V 1150 3730 50  0000 L CNN
+AR Path="/669AB112/5C632DBE" Ref="TP4"  Part="1"
+F 0 "TP4" V 1150 3730 50  0000 L CNN
 F 1 "TestPoint_Alt" V 1185 3735 50  0001 L CNN
 F 2 "croptop:TestPoint" H 1350 3550 50  0001 C CNN
