File: PCB v3.0/croptop_io.sch (KiCad schematic (older format))
At the start: 139 parts, among them J10 1702474, J11 1702474, J12 1702474, J13 1702474, J14 1702474, J7 1702474, J8 1702474, J9 1702474, Q3 Q2319ADS-T1-GE3, U18 74HCT125D653, U19 AP22802AW5, U20 AD7799, U21 AP22802AW5, U22 TPD4E1U06DBV, U23 AP22802AW5, U24 TPD4E1U06DBV, U25 TPD4E1U06DBV, U26 TPD4E1U06DBV, U27 DRV8872, U28 DRV8825, U29 AP22802AW5

Commit message: Updated PCB dimensions for Nextion screen, deleted old files
- Updated PCB v3.0 to use the Nextion screen mounting and connectors
- Deleted old I2CDriver files from /Software/
- Deleted unused /Software/Readme
Parts:
- removed TP17, TP18, TP19, TP20, TP21, TP22, TP23, TP25, TP27, TP28, TP29, TP33, TP34, TP35, TP36, TP37, TP38, TP39, TP40, TP41, TP42, TP43, TP44, TP45, TP46, TP47, TP48, TP49, TP50, TP51, TP52, TP53, TP55, TP56, TP57: TestPoint, TestPoint:TestPoint_Pad_D1.0mm, symbol Connector:TestPoint
- J10, J11, J12, J13, J14, J7, J8, J9: MPN 277-2338-1-ND -> 1702474
